File: pcb/appleii/appleii.sch (EAGLE design)
At the start: 19 parts, among them J1 POWER_JACKPTH, J2 ATX24RH

Commit message: updated pcb
Parts:
- removed C4, C5: (no value), capacitor-wima:C5/2.5
- removed J2: ATX24RH, macse:ATX24RH
- removed J3, J7: (no value), atx_power_control:CONN_023.5MM-NO_SILK
- removed JP4: (no value), appleii:4PIN_FAN
- removed U$8: CAR_FUSE_HOLDER3IN1, atx_power_control:CAR_FUSE_HOLDER3IN1
- added JP3: (no value), appleii:4PIN_FAN
- added U$6: APPLEII, atx4vc:APPLEII
- C1, C2: device rcl:CPOL-USE5-10.5 -> capacitor-wima:C5/2.5
- J1: value POWER_JACKPTH -> ATX24RH; device appleii:POWER_JACKPTH -> macse:ATX24RH
- JP1: device appleii:4PIN_FAN -> pinhead:PINHD-1X2
- JP2: device pinhead:PINHD-1X2 -> pinhead:PINHD-1X3
- U$1: value M3_MOUNTING_HOLE -> CAR_FUSE_HOLDER3IN1; device a:M3_MOUNTING_HOLE -> atx_power_control:CAR_FUSE_HOLDER3IN1
- U$3: value M3_MOUNTING_HOLE -> ROCK_SW; device a:M3_MOUNTING_HOLE -> atx4vc:ROCK_SW
- U$4: value APPLEII -> M3_MOUNTING_HOLE; device atx4vc:APPLEII -> a:M3_MOUNTING_HOLE
- U$5: value ROCK_SW -> M3_MOUNTING_HOLE; device atx4vc:ROCK_SW -> a:M3_MOUNTING_HOLE
Connections:
- net +12V: now also JP2.3, U$6.P$4; no longer C1.+, JP1.2_VCC, U$4.P$4
- net +5V: now also JP2.1, U$1.A0, U$1.A1, U$6.P$3; no longer C2.+, JP4.2_VCC, U$4.P$3, U$8.A0, U$8.A1
- net -12V: now also J1.-12V, U$6.P$5; no longer J2.-12V, U$4.P$5
- net -5V: now also C3.1, U$6.P$6; no longer C5.1, U$4.P$6
- net GND: now also C1.2, C2.2, J1.GND@0, J1.GND@1, J1.GND@2, J1.GND@3, J1.GND@4, J1.GND@5, J1.GND@6, J1.GND@7, JP1.2, JP3.1_GND, U$3.P$1, U$3.P$3, U$6.P$1, U$6.P$2; no longer C1.-, C2.-, C4.2, C5.2, J1.GND, J1.GNDBREAK, J2.GND@0, J2.GND@1, J2.GND@2, J2.GND@3, J2.GND@4, J2.GND@5, J2.GND@6, J2.GND@7, J3.2, J7.2, JP1.1_GND, JP2.2, JP4.1_GND, U$4.P$1, U$4.P$2, U$5.P$1, U$5.P$3
- net N$1: now also JP2.2, JP3.2_VCC; no longer J1.PWR, J3.1
- net N$5: now also J1.PS_ON, JP1.1, U$3.P$2, U$3.P$4; no longer J2.PS_ON, J7.1, JP2.1, U$5.P$2, U$5.P$4
- net N$6: now also C1.1, J1.5V@1, J1.5V@2, J1.5V@3, J1.5V@4, U$1.B0, U$1.B1; no longer C4.1, J2.5V@1, J2.5V@2, J2.5V@3, J2.5V@4, U$8.B0, U$8.B1
- net N$8: now also C2.1, J1.12V@0, J1.12V@1; no longer C3.1, J2.12V@0, J2.12V@1
Other:
- moved on the sheet: C3
