File: pcb/appleii/appleii.brd (EAGLE design)
At the start: 75 x 45 mm, 21 parts, among them J1 ATX24RH

Commit message: updated IIGS design
Parts:
- added U$14, U$15, U$16, U$17, U$18, U$19, U$20: EDGEPAD, atx4vc:EDGEPAD
- moved U$9 1.42 mm to (8.93, 43.7), turned to 270 degrees
- moved JP1 0.51 mm to (4.70, 25.9)
- moved JP3 0.25 mm to (66.4, 3.43)
Connections:
- net GND: now also U$14.P$1, U$15.P$1, U$16.P$1, U$17.P$1, U$18.P$1, U$19.P$1, U$20.P$1
Routing:
- net +12V: track 52.4 -> 51.0 mm
- net +5V: track 38.0 -> 37.0 mm
