File: pcb/appleii/appleii_blanking_plate.sch (EAGLE design)
At the start: 21 parts, among them J1 ATX24RH

Commit message: updated IIGS design
Parts:
- removed C1, C2, C3: (no value), capacitor-wima:C5/2.5
- removed IC1: (no value), v-reg:79XXS
- removed J1: ATX24RH, macse:ATX24RH
- removed JP1: (no value), pinhead:PINHD-1X2
- removed JP2: (no value), pinhead:PINHD-1X3
- removed JP3: (no value), appleii:4PIN_FAN
- removed U$10, U$11, U$12, U$7, U$8, U$9: EDGEPAD, atx4vc:EDGEPAD
- removed U$6: APPLEII, atx4vc:APPLEII
- U$1: value CAR_FUSE_HOLDER3IN1 -> EDGEPADEDGEPAD_20MM; device atx_power_control:CAR_FUSE_HOLDER3IN1 -> atx4vc:EDGEPADEDGEPAD_20MM
- U$2: value CAR_FUSE_HOLDER3IN1 -> EDGEPAD; device atx_power_control:CAR_FUSE_HOLDER3IN1 -> atx4vc:EDGEPAD
- U$3: value ROCK_SW -> EDGEPAD; device atx4vc:ROCK_SW -> atx4vc:EDGEPAD
- U$4: value M3_MOUNTING_HOLE -> EDGEPAD; device a:M3_MOUNTING_HOLE -> atx4vc:EDGEPAD
- U$5: value M3_MOUNTING_HOLE -> EDGEPADEDGEPAD_20MM; device a:M3_MOUNTING_HOLE -> atx4vc:EDGEPADEDGEPAD_20MM
Connections:
- removed net +12V: JP2.3, U$2.B0, U$2.B1, U$6.P$4
- removed net +5V: JP2.1, U$1.A0, U$1.A1, U$6.P$3
- removed net -12V: IC1.IN, J1.-12V, U$6.P$5
- removed net -5V: C3.1, IC1.OUT, U$6.P$6
- removed net N$1: JP2.2, JP3.2_VCC
- removed net N$5: J1.PS_ON, JP1.1, U$3.P$2, U$3.P$4
- removed net N$6: C1.1, J1.5V@1, J1.5V@2, J1.5V@3, J1.5V@4, U$1.B0, U$1.B1
- removed net N$8: C2.1, J1.12V@0, J1.12V@1, U$2.A0, U$2.A1
- net GND: now also U$1.P$1, U$2.P$1, U$4.P$1, U$5.P$1; no longer C1.2, C2.2, C3.2, IC1.GND, J1.GND@0, J1.GND@1, J1.GND@2, J1.GND@3, J1.GND@4, J1.GND@5, J1.GND@6, J1.GND@7, JP1.2, JP3.1_GND, U$10.P$1, U$11.P$1, U$12.P$1, U$3.P$3, U$6.P$1, U$6.P$2, U$7.P$1, U$8.P$1, U$9.P$1
