File: pcb/mac_se_se30/mac_se_power_switch.sch (EAGLE design)
At the start: 5 parts

Commit message: updated pcb
Parts:
- removed J7: (no value), atx_power_control:CONN_023.5MM-NO_SILK
Connections:
- net N$2: no longer J7.2
- net N$3: no longer J7.1
Changed lines of the file:
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@@
 </classes>
 <parts>
-<part name="J7" library="atx_power_control" deviceset="CONN_02" device="3.5MM-NO_SILK"/>
 <part name="JP2" library="pinhead" library_urn="urn:adsk.eagle:library:325" deviceset="PINHD-1X2" device="/90" package3d_urn="urn:adsk.eagle:package:22437/2"/>
 <part name="U$2" library="a" deviceset="M3_MOUNTING_HOLE" device=""/>
@@
 </plain>
 <instances>
-<instance part="J7" gate="G$1" x="12.7" y="2.54" smashed="yes" rot="R180">
-<attribute name="VALUE" x="15.24" y="7.366" size="1.778" layer="96" font="vector" rot="R180"/>
-<attribute name="NAME" x="15.24" y="-3.048" size="1.778" layer="95" font="vector" rot="R180"/>
-</instance>
 <instance part="JP2" gate="G$1" x="27.94" y="0" smashed="yes">
 <attribute name="NAME" x="21.59" y="5.715" size="1.778" layer="95"/>
@@
 <pinref part="U$1" gate="G$1" pin="P$1"/>
 <wire x1="-40.64" y1="-10.16" x2="-33.02" y2="-10.16" width="0.1524" layer="91"/>
-<pinref part="J7" gate="G$1" pin="2"/>
 <pinref part="JP2" gate="G$1" pin="2"/>
 <wire x1="5.08" y1="0" x2="25.4" y2="0" width="0.1524" layer="91"/>
@@
 <wire x1="5.08" y1="-10.16" x2="5.08" y2="0" width="0.1524" layer="91"/>
 <junction x="-33.02" y="-10.16"/>
-<junction x="5.08" y="0"/>
 </segment>
 </net>
@@
 <pinref part="U$1" gate="G$1" pin="P$2"/>
 <wire x1="-40.64" y1="12.7" x2="-33.02" y2="12.7" width="0.1524" layer="91"/>
-<pinref part="J7" gate="G$1" pin="1"/>
 <pinref part="JP2" gate="G$1" pin="1"/>
 <wire x1="25.4" y1="2.54" x2="5.08" y2="2.54" width="0.1524" layer="91"/>
@@
 <wire x1="5.08" y1="12.7" x2="5.08" y2="2.54" width="0.1524" layer="91"/>
 <junction x="-33.02" y="12.7"/>
-<junction x="5.08" y="2.54"/>
 </segment>
 </net>
