File: pcb/mac_se_se30/macse.brd (EAGLE design)
At the start: 51 x 38 mm, 11 parts, among them J2 ATX24RH

Commit message: updated pcb
Parts:
- removed J7: (no value), atx_power_control:SCREWTERMINAL-3.5MM-2-NS
- removed JP1: (no value), atx_power_control:1X04
- added JP4: (no value), pinhead:1X03
- JP2: device pinhead:1X02 -> pinhead:1X02/90
- JP3: device atx_power_control:1X04 -> appleii:1X04
- moved JP3 16.6 mm to (44.3, 33.4), turned to 0 degrees
- moved C2 10.6 mm to (27.9, 35.4), flipped to the top, turned to 180 degrees
- moved C1 7.34 mm to (27.9, 30.9), turned to 180 degrees
- moved JP2 3.81 mm to (46.7, 25.0), turned to 270 degrees
Connections:
- new net N$2: JP3.2, JP4.2
- net +12V: now also JP4.1; no longer C2.1, JP1.3
- net +5V: now also C2.1, JP4.3; no longer JP3.3
- net GND: now also JP3.1; no longer J7.2, JP1.4, JP3.4
- net N$5: no longer J7.1
Routing:
- net -12V: track 48.9 -> 35.4 mm
- net +12V: track 72.8 -> 61.5 mm
- net N$2: track 0.00 -> 11.3 mm
- net +5V: track 38.5 -> 46.6 mm
- net N$5: track 15.3 -> 10.8 mm
Other:
- board text removed: "G"
