File: pcb/appleii/old/appleii.brd (EAGLE design)
At the start: 75 x 45 mm, 21 parts, among them J1 ATX24RH

Commit message: working on edgeplate
Parts:
- removed U$10, U$11, U$12, U$13, U$7, U$8, U$9: EDGEPAD, atx4vc:EDGEPAD
- moved JP1 22.5 mm to (3.05, 3.97), turned to 90 degrees
- moved C1 4.92 mm to (2.03, 11.6), turned to 90 degrees
- moved C2 3.79 mm to (4.95, 27.8)
- moved U$4 2.00 mm to (72.5, 20.0)
- moved U$5 2.00 mm to (2.50, 20.0)
- moved U$3 0.55 mm to (22.1, 23.7)
- moved J1 0.25 mm to (31.1, 9.26)
Connections:
- net GND: no longer U$10.P$1, U$11.P$1, U$12.P$1, U$13.P$1, U$7.P$1, U$8.P$1, U$9.P$1
Routing:
- net N$5: track 45.3 -> 72.2 mm
- net N$6: track 92.1 -> 93.2 mm
- net N$8: track 85.8 -> 84.8 mm
- net -12V: track 31.4 -> 30.8 mm
Other:
- outline, holes or cut-outs redrawn
- board text added: "PT1 dekuNukem DEC 2022"
- board text removed: "+12"
- board text removed: "+5"
- board text removed: "PD2 dekuNukem APR23"
