File: pcb/appleii/old/appleii.sch (EAGLE design)
At the start: 21 parts, among them J1 ATX24RH

Commit message: working on edgeplate
Parts:
- removed U$10, U$11, U$12, U$13, U$7, U$8, U$9: EDGEPAD, atx4vc:EDGEPAD
Connections:
- net GND: no longer U$10.P$1, U$11.P$1, U$12.P$1, U$13.P$1, U$7.P$1, U$8.P$1, U$9.P$1
Changed lines of the file:
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@@
 <part name="JP3" library="appleii" deviceset="4PIN_FAN" device=""/>
 <part name="JP2" library="pinhead" library_urn="urn:adsk.eagle:library:325" deviceset="PINHD-1X3" device="" package3d_urn="urn:adsk.eagle:package:22458/2"/>
-<part name="U$7" library="atx4vc" deviceset="EDGEPAD" device=""/>
-<part name="GND4" library="supply1" library_urn="urn:adsk.eagle:library:371" deviceset="GND" device=""/>
-<part name="U$8" library="atx4vc" deviceset="EDGEPAD" device=""/>
-<part name="GND6" library="supply1" library_urn="urn:adsk.eagle:library:371" deviceset="GND" device=""/>
-<part name="U$9" library="atx4vc" deviceset="EDGEPAD" device=""/>
-<part name="GND8" library="supply1" library_urn="urn:adsk.eagle:library:371" deviceset="GND" device=""/>
-<part name="U$10" library="atx4vc" deviceset="EDGEPAD" device=""/>
-<part name="GND12" library="supply1" library_urn="urn:adsk.eagle:library:371" deviceset="GND" device=""/>
-<part name="U$11" library="atx4vc" deviceset="EDGEPAD" device=""/>
-<part name="GND13" library="supply1" library_urn="urn:adsk.eagle:library:371" deviceset="GND" device=""/>
-<part name="U$12" library="atx4vc" deviceset="EDGEPAD" device=""/>
-<part name="GND14" library="supply1" library_urn="urn:adsk.eagle:library:371" deviceset="GND" device=""/>
-<part name="U$13" library="atx4vc" deviceset="EDGEPAD" device=""/>
-<part name="GND15" library="supply1" library_urn="urn:adsk.eagle:library:371" deviceset="GND" device=""/>
 </parts>
 <sheets>
@@
 <attribute name="VALUE" x="31.75" y="121.92" size="1.778" layer="96"/>
 </instance>
-<instance part="U$7" gate="G$1" x="-2.54" y="71.12" smashed="yes"/>
-<instance part="GND4" gate="1" x="-12.7" y="68.58" smashed="yes">
-<attribute name="VALUE" x="-15.24" y="66.04" size="1.778" layer="96"/>
-</instance>
-<instance part="U$8" gate="G$1" x="-2.54" y="58.42" smashed="yes"/>
-<instance part="GND6" gate="1" x="-12.7" y="55.88" smashed="yes">
-<attribute name="VALUE" x="-15.24" y="53.34" size="1.778" layer="96"/>
-</instance>
-<instance part="U$9" gate="G$1" x="-2.54" y="45.72" smashed="yes"/>
-<instance part="GND8" gate="1" x="-12.7" y="43.18" smashed="yes">
-<attribute name="VALUE" x="-15.24" y="40.64" size="1.778" layer="96"/>
-</instance>
-<instance part="U$10" gate="G$1" x="-2.54" y="33.02" smashed="yes"/>
-<instance part="GND12" gate="1" x="-12.7" y="30.48" smashed="yes">
-<attribute name="VALUE" x="-15.24" y="27.94" size="1.778" layer="96"/>
-</instance>
-<instance part="U$11" gate="G$1" x="83.82" y="53.34" smashed="yes"/>
-<instance part="GND13" gate="1" x="73.66" y="50.8" smashed="yes">
-<attribute name="VALUE" x="71.12" y="48.26" size="1.778" layer="96"/>
-</instance>
-<instance part="U$12" gate="G$1" x="83.82" y="40.64" smashed="yes"/>
-<instance part="GND14" gate="1" x="73.66" y="38.1" smashed="yes">
-<attribute name="VALUE" x="71.12" y="35.56" size="1.778" layer="96"/>
-</instance>
-<instance part="U$13" gate="G$1" x="83.82" y="27.94" smashed="yes"/>
-<instance part="GND15" gate="1" x="73.66" y="25.4" smashed="yes">
-<attribute name="VALUE" x="71.12" y="22.86" size="1.778" layer="96"/>
-</instance>
 </instances>
 <busses>
@@
 <wire x1="2.54" y1="134.62" x2="-15.24" y2="134.62" width="0.1524" layer="91"/>
 </segment>
-<segment>
-<pinref part="GND4" gate="1" pin="GND"/>
-<pinref part="U$7" gate="G$1" pin="P$1"/>
-<wire x1="-12.7" y1="71.12" x2="-7.62" y2="71.12" width="0.1524" layer="91"/>
-</segment>
-<segment>
-<pinref part="GND6" gate="1" pin="GND"/>
-<pinref part="U$8" gate="G$1" pin="P$1"/>
-<wire x1="-12.7" y1="58.42" x2="-7.62" y2="58.42" width="0.1524" layer="91"/>
-</segment>
-<segment>
-<pinref part="GND8" gate="1" pin="GND"/>
-<pinref part="U$9" gate="G$1" pin="P$1"/>
-<wire x1="-12.7" y1="45.72" x2="-7.62" y2="45.72" width="0.1524" layer="91"/>
-</segment>
-<segment>
-<pinref part="GND12" gate="1" pin="GND"/>
-<pinref part="U$10" gate="G$1" pin="P$1"/>
-<wire x1="-12.7" y1="33.02" x2="-7.62" y2="33.02" width="0.1524" layer="91"/>
-</segment>
-<segment>
-<pinref part="GND13" gate="1" pin="GND"/>
-<pinref part="U$11" gate="G$1" pin="P$1"/>
-<wire x1="73.66" y1="53.34" x2="78.74" y2="53.34" width="0.1524" layer="91"/>
-</segment>
-<segment>
-<pinref part="GND14" gate="1" pin="GND"/>
-<pinref part="U$12" gate="G$1" pin="P$1"/>
-<wire x1="73.66" y1="40.64" x2="78.74" y2="40.64" width="0.1524" layer="91"/>
-</segment>
-<segment>
-<pinref part="GND15" gate="1" pin="GND"/>
-<pinref part="U$13" gate="G$1" pin="P$1"/>
-<wire x1="73.66" y1="27.94" x2="78.74" y2="27.94" width="0.1524" layer="91"/>
-</segment>
 </net>
