File: pcb/bbc_micro/bbc.brd (EAGLE design)
At the start: 43 x 30 mm, 25 parts, among them U2 LM2776

Commit message: bbc run
Routing:
- net +5V: track 91.2 -> 70.0 mm
- added copper zone on layer 16, net +5V
Changed lines of the file:
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@@
 <?xml version="1.0" encoding="utf-8"?>
 <!DOCTYPE eagle SYSTEM "eagle.dtd">
-<eagle version="9.6.1">
+<eagle version="9.6.2">
 <drawing>
 <settings>
@@
 <text x="45.881" y="14.5442" size="1.9304" layer="25" distance="35" align="center">+5V</text>
 <text x="32.049" y="17.7138" size="1.9304" layer="25" distance="35" rot="R180" align="center">-5V</text>
-<rectangle x1="60.071" y1="31.371" x2="65.405" y2="42.293" layer="41"/>
 <text x="21.971" y="3.365" size="2.54" layer="25" distance="35" align="center">picoRC.com</text>
 <rectangle x1="7.239" y1="0.889" x2="12.573" y2="4.572" layer="41"/>
@@
 <vertex x="43.307" y="28.448"/>
 <vertex x="48.768" y="28.448"/>
-<vertex x="48.768" y="17.145"/>
-<vertex x="43.307" y="17.145"/>
+<vertex x="48.768" y="16.383"/>
+<vertex x="43.307" y="16.383"/>
 </polygon>
 <wire x1="29.271" y1="23.273" x2="28.356" y2="24.188" width="0.6096" layer="1"/>
@@
 <contactref element="C5" pad="1"/>
 <contactref element="U2" pad="4"/>
-<wire x1="44.644" y1="11.432" x2="47.304" y2="11.432" width="1.27" layer="16"/>
-<wire x1="47.304" y1="11.432" x2="47.304" y2="7.495" width="1.27" layer="16"/>
-<wire x1="47.304" y1="7.495" x2="47.304" y2="3.431" width="1.27" layer="16"/>
-<wire x1="47.304" y1="3.431" x2="44.644" y2="3.431" width="1.27" layer="16"/>
-<wire x1="44.644" y1="11.432" x2="44.644" y2="8.636" width="1.27" layer="16"/>
-<wire x1="44.644" y1="8.636" x2="44.644" y2="7.495" width="1.016" layer="16"/>
-<wire x1="44.644" y1="7.495" x2="44.644" y2="3.431" width="1.27" layer="16"/>
 <wire x1="37.973" y1="15.147" x2="37.973" y2="14.997" width="1.27" layer="1"/>
 <wire x1="37.973" y1="14.997" x2="40.005" y2="14.997" width="1.27" layer="1"/>
 <wire x1="40.005" y1="14.997" x2="42.037" y2="14.997" width="1.27" layer="1"/>
 <wire x1="44.644" y1="13.395" x2="44.644" y2="11.432" width="1.27" layer="1"/>
-<wire x1="44.644" y1="8.636" x2="39.779" y2="8.636" width="1.27" layer="16"/>
-<wire x1="39.271" y1="8.128" x2="39.779" y2="8.636" width="1.27" layer="16"/>
 <wire x1="42.037" y1="14.997" x2="43.042" y2="14.997" width="1.27" layer="1"/>
 <wire x1="43.042" y1="14.997" x2="44.644" y2="13.395" width="1.27" layer="1"/>
 <wire x1="39.271" y1="8.128" x2="38.1" y2="8.128" width="0.4064" layer="1"/>
 <wire x1="36.83" y1="6.858" x2="38.1" y2="8.128" width="0.4064" layer="1"/>
-<wire x1="34.605" y1="5.3039" x2="34.605" y2="5.03" width="0.4064" layer="1"/>
-<wire x1="34.605" y1="5.03" x2="36.079" y2="3.556" width="0.4064" layer="1"/>
-<wire x1="36.079" y1="3.556" x2="36.206" y2="3.683" width="0.4064" layer="1"/>
-<wire x1="36.206" y1="3.683" x2="36.576" y2="3.683" width="0.4064" layer="1"/>
-<wire x1="36.576" y1="3.683" x2="36.83" y2="3.937" width="0.4064" layer="1"/>
-<wire x1="36.83" y1="3.937" x2="36.83" y2="6.858" width="0.4064" layer="1"/>
+<wire x1="34.605" y1="5.3039" x2="34.7121" y2="5.3039" width="0.4064" layer="1"/>
+<wire x1="35.952" y1="4.064" x2="34.7121" y2="5.3039" width="0.4064" layer="1"/>
+<wire x1="35.952" y1="4.064" x2="35.952" y2="3.683" width="0.4064" layer="1"/>
+<wire x1="35.952" y1="3.683" x2="36.079" y2="3.556" width="0.4064" layer="1"/>
+<wire x1="36.83" y1="3.81" x2="36.576" y2="3.556" width="0.4064" layer="1"/>
+<wire x1="36.079" y1="3.556" x2="36.576" y2="3.556" width="0.4064" layer="1"/>
+<wire x1="36.83" y1="3.81" x2="36.83" y2="6.858" width="0.4064" layer="1"/>
 <wire x1="34.605" y1="5.3039" x2="34.605" y2="7.9041" width="0.4064" layer="1"/>
 <contactref element="C2" pad="+"/>
@@
 <wire x1="23.328" y1="17.272" x2="39.091" y2="17.272" width="1.27" layer="1"/>
 <wire x1="40.005" y1="14.997" x2="40.005" y2="18.186" width="1.27" layer="1"/>
+<wire x1="39.271" y1="8.128" x2="44.011" y2="8.128" width="1.778" layer="16"/>
+<wire x1="44.011" y1="8.128" x2="44.644" y2="7.495" width="1.778" layer="16"/>
+<polygon width="0.1524" layer="16" thermals="no">
+<vertex x="43.688" y="12.954"/>
+<vertex x="48.26" y="12.954"/>
+<vertex x="48.26" y="1.905"/>
+<vertex x="43.688" y="1.905"/>
+</polygon>
 </signal>
 <signal name="N$31">
