File: pcb/apriotpc/apricot.brd (EAGLE design)
At the start: 31 x 90 mm, 23 parts, among them J2 ATX24RH

Commit message: changed to smaller diameter caps
Parts:
- added C13: (no value), capacitor-wima:C5B2.5
- C11, C4, C9: device adafruit:E5-10,5 -> adafruit_changed:E3,5-8
- moved C1 7.55 mm to (26.1, 25.0)
- moved C7 5.89 mm to (25.9, 22.5)
- moved C12 5.64 mm to (25.9, 21.0)
- moved C11 5.37 mm to (25.9, 19.1)
- moved C8 4.87 mm to (25.9, 16.3)
- moved C5 2.29 mm to (27.3, 68.1)
- moved C3 1.91 mm to (26.7, 72.4)
- moved C10 1.78 mm to (26.7, 70.5)
- moved C9 1.53 mm to (26.7, 74.3)
- moved JP3 0.81 mm to (27.7, 84.7)
- moved C6 0.76 mm to (26.6, 77.0)
- moved JP1 0.38 mm to (25.7, 12.6)
- moved U$7 0.38 mm to (25.6, 5.10)
- moved U$3 0.28 mm to (2.67, 5.08)
- moved C4 0.25 mm to (4.32, 84.8)
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Connections:
- net +12V: now also C13.1
- net GND: now also C13.2
Routing:
- net GND: track 37.9 -> 30.6 mm
- net +12V: track 143.6 -> 148.0 mm
- net +5V: track 51.9 -> 56.1 mm
Other:
- board text added: "FAN"
- board text removed: "12\"
