File: pcb/ibmpc/ibm.brd (EAGLE design)
At the start: 104 x 76 mm, 33 parts, among them J2 ATX24RH

Commit message: working on new version
Parts:
- removed JP1: (no value), appleii:1X04
- added JP2: (no value), pinhead:1X04/90
- added U$1: ISA, blade:ISAPAD
- added U$11, U$14: 28FLAG, blade:2.8FLAG
- added U$12: CRT2P, blade:CRT2P
- U$3: value VH396_2P -> 28FLAG; device 396_conn:396_2P -> blade:2.8FLAG
- moved U$3 141.7 mm to (77.6, 51.7), turned to 90 degrees
- moved C1 111.4 mm to (35.3, 49.1)
- moved C4 111.4 mm to (35.7, 39.3)
- moved C5 111.4 mm to (36.1, 41.2)
- moved C7 111.4 mm to (36.1, 43.1)
- moved U$8 111.4 mm to (35.0, 59.9)
- moved C17 111.4 mm to (35.7, 36.3)
- moved C3 110.8 mm to (35.3, 45.4)
- moved C2 109.8 mm to (44.7, 39.2)
- moved C14 109.6 mm to (35.9, 21.0)
- moved C10 109.3 mm to (44.7, 43.1)
- moved C8 109.3 mm to (44.7, 41.2)
- moved IC1 109.2 mm to (36.4, 28.8)
- moved C16 109.1 mm to (44.8, 36.1)
- moved C9 108.7 mm to (44.0, 45.4)
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Connections:
- net +12V: now also JP2.3, U$12.2; no longer JP1.1, U$3.P$1
- net +5V: now also U$1.P$1, U$11.P$1, U$11.P$2
- net GND: now also JP2.4, U$12.1, U$3.P$1; no longer JP1.2
- net N$4: now also U$14.P$1, U$14.P$2
Other:
- board size 104 x 76 mm -> 104 x 75 mm

Commit message: working on new version
Parts:
- J2: device macse:ATX24_RIGHT_ANGLE -> blade:ATX24_RIGHT_ANGLE
- moved R2 91.5 mm to (19.1, 16.2), flipped to the top, turned to 180 degrees
- moved JP3 70.4 mm to (90.1, 68.3)
- moved C11 14.4 mm to (49.8, 13.8), turned to 270 degrees
- moved C14 12.2 mm to (45.8, 13.9), turned to 270 degrees
- moved LED1 5.00 mm to (90.0, 58.6), turned to 270 degrees
- moved U$4 4.11 mm to (89.5, 43.6)
- moved C6 4.06 mm to (43.6, 45.0)
- moved C10 3.86 mm to (43.6, 39.5)
- moved C16 3.81 mm to (44.8, 32.3)
- moved U$2 3.81 mm to (43.2, 56.1)
- moved C2 3.81 mm to (44.7, 35.4)
- moved C9 3.81 mm to (44.0, 41.6)
- moved C8 3.74 mm to (43.6, 37.7)
- moved R1 3.70 mm to (95.3, 53.4)
- moved IC1 3.57 mm to (36.1, 25.3)
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Routing:
- net +5V: track 0.00 -> 173.6 mm, vias 0 -> 2
- net N$3: track 0.00 -> 139.9 mm
- net +12V: track 0.00 -> 83.8 mm
- net N$4: track 0.00 -> 80.5 mm
- net N$8: track 0.00 -> 52.3 mm
- net -12V: track 0.00 -> 49.6 mm, vias 0 -> 1
- net -5V: track 0.00 -> 46.2 mm, vias 0 -> 1
- net N$6: track 0.00 -> 39.0 mm
- net GND: track 0.00 -> 35.9 mm, vias 0 -> 3
- net N$1: track 0.00 -> 15.4 mm
- net N$12: track 0.00 -> 4.07 mm
Other:
- board text added: "5155 kit: 2P PCB connector 2P cable"
- board text added: "external switch kit: long dupot cable (1m+) hooks or aligator clips maybe both?"

Commit message: working on new version
Parts:
- moved C11 3.43 mm to (46.4, 13.7)
- moved C14 3.31 mm to (42.5, 13.7)
- moved U$5 1.00 mm to (99.5, 69.6)
Routing:
- net +5V: track 173.6 -> 177.3 mm
- net -12V: track 49.6 -> 47.4 mm
- net N$8: track 52.3 -> 51.3 mm
- net N$6: track 39.0 -> 39.5 mm
Other:
- board size 104 x 75 mm -> 104 x 74 mm

Commit message: working on new version
Parts:
- added C12: (no value), adafruit_changed:E3,5-8
- added C13, C15: (no value), capacitor-wima:C5B2.5
- moved C17 1.78 mm to (35.7, 34.5)
- moved IC1 1.67 mm to (35.9, 23.6)
- moved C4 1.27 mm to (35.7, 38.1)
- moved JP2 1.00 mm to (53.1, 49.4)
- moved C16 0.76 mm to (44.8, 31.6)
- moved C1 0.51 mm to (35.0, 48.5)
- moved C10 0.51 mm to (43.6, 39.0)
- moved C2 0.51 mm to (44.7, 34.9)
- moved C5 0.51 mm to (35.1, 41.0)
- moved C9 0.51 mm to (44.0, 41.1)
- moved C3 0.51 mm to (35.3, 44.9)
- moved C6 0.51 mm to (43.6, 44.5)
- moved C7 0.51 mm to (35.1, 42.8)
- moved C8 0.51 mm to (43.6, 37.2)
- moved U$11 0.25 mm to (72.0, 51.9)
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Connections:
- net +12V: now also C12.+, C13.1, C15.1
- net GND: now also C12.-, C13.2, C15.2
Routing:
- net GND: track 35.9 -> 63.2 mm
- net +12V: track 83.8 -> 99.6 mm
- net +5V: track 177.3 -> 185.3 mm
- net N$3: track 139.9 -> 133.7 mm
Other:
- outline, holes or cut-outs redrawn
- board text added: "510"
- board text added: "FUSE 7.5A MAX"
- board text added: "PG"
- board text removed: "1"
- board text removed: "29"
- board text removed: "31"
- board text removed: "470"
- board text removed: "5"
- board text removed: "7"
- board text removed: "9"
- board text removed: "FUSE 5A MAX"
- board text removed: "ISA Bracket ------>"
- board text removed: "ISA Bracket <------"
- board text removed: "put a sticker on 7905 laying down footprint"

Commit message: working on new version
Parts:
- moved R2 0.51 mm to (19.1, 15.7)
- moved IC1 0.38 mm to (36.3, 23.6)
- moved JP2 0.13 mm to (53.0, 49.4)
Connections:
- net GND: now also U$14.P$1, U$14.P$2; no longer U$3.P$1, U$3.P$2
- net N$4: now also U$3.P$1, U$3.P$2; no longer U$14.P$1, U$14.P$2
Routing:
- net +5V: track 185.3 -> 176.9 mm
- net N$4: track 80.3 -> 82.5 mm
- net N$1: track 15.4 -> 15.9 mm
Other:
- board text added: "5155 kit: 2P PCB connector 2P cable additional caps"
- board text removed: "1 and 0 on ISA bracket? just cut out the outline"
- board text removed: "5155 kit: 2P PCB connector 2P cable"
