File: pcb/ibmpc/ibm.sch (EAGLE design)
At the start: 33 parts, among them J2 ATX24RH

Commit message: working on new version
Parts:
- removed JP1: (no value), appleii:4PIN_FAN
- added JP2: (no value), pinhead:PINHD-1X4/90
- added U$1: ISA, blade:ISA
- added U$11, U$14: 28FLAG, blade:28FLAG
- added U$12: CRT2P, blade:CRT2P
- U$3: value VH396_2P -> 28FLAG; device 396_conn:VH396_2P -> blade:28FLAG
Connections:
- net +12V: now also JP2.3, U$12.P$2; no longer JP1.1_GND, U$3.P$1
- net +5V: now also U$1.P$1, U$11.P$1
- net GND: now also JP2.4, U$12.P$1, U$3.P$1; no longer JP1.2_VCC, U$3.P$2
- net N$4: now also U$14.P$1
Changed lines of the file:
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@@
 <part name="C14" library="capacitor-wima" library_urn="urn:adsk.eagle:library:116" deviceset="C" device="5/2.5" package3d_urn="urn:adsk.eagle:package:5426/1"/>
 <part name="GND8" library="supply1" library_urn="urn:adsk.eagle:library:371" deviceset="GND" device=""/>
-<part name="JP1" library="appleii" deviceset="4PIN_FAN" device=""/>
-<part name="GND9" library="supply1" library_urn="urn:adsk.eagle:library:371" deviceset="GND" device=""/>
-<part name="P+7" library="supply1" library_urn="urn:adsk.eagle:library:371" deviceset="+12V" device=""/>
 <part name="U$4" library="apricot" deviceset="ROCKSW" device=""/>
 <part name="GND4" library="supply1" library_urn="urn:adsk.eagle:library:371" deviceset="GND" device=""/>
@@
 <part name="P-1" library="supply1" library_urn="urn:adsk.eagle:library:371" deviceset="-12V" device=""/>
 <part name="P-2" library="supply1" library_urn="urn:adsk.eagle:library:371" deviceset="-5V" device=""/>
-<part name="U$3" library="396_conn" deviceset="VH396_2P" device=""/>
 <part name="U$13" library="blade" deviceset="ISA" device=""/>
 <part name="U$15" library="blade" deviceset="ISA" device=""/>
@@
 <part name="R2" library="adafruit_changed" deviceset="R-US_" device="0411/15"/>
 <part name="GND15" library="supply1" library_urn="urn:adsk.eagle:library:371" deviceset="GND" device=""/>
+<part name="U$1" library="blade" deviceset="ISA" device=""/>
+<part name="U$11" library="blade" deviceset="28FLAG" device=""/>
+<part name="U$12" library="blade" deviceset="CRT2P" device=""/>
+<part name="U$3" library="blade" deviceset="28FLAG" device=""/>
+<part name="JP2" library="pinhead" library_urn="urn:adsk.eagle:library:325" deviceset="PINHD-1X4" device="/90" package3d_urn="urn:adsk.eagle:package:22404/2"/>
+<part name="P+4" library="supply1" library_urn="urn:adsk.eagle:library:371" deviceset="+12V" device=""/>
+<part name="GND17" library="supply1" library_urn="urn:adsk.eagle:library:371" deviceset="GND" device=""/>
+<part name="U$14" library="blade" deviceset="28FLAG" device=""/>
+<part name="P+6" library="supply1" library_urn="urn:adsk.eagle:library:371" deviceset="+5V" device=""/>
+<part name="GND9" library="supply1" library_urn="urn:adsk.eagle:library:371" deviceset="GND" device=""/>
 </parts>
 <sheets>
@@
 <attribute name="VALUE" x="203.2" y="223.52" size="1.778" layer="96"/>
 </instance>
-<instance part="JP1" gate="A" x="256.54" y="226.06" smashed="yes"/>
-<instance part="GND9" gate="1" x="279.4" y="226.06" smashed="yes">
-<attribute name="VALUE" x="276.86" y="223.52" size="1.778" layer="96"/>
-</instance>
-<instance part="P+7" gate="1" x="236.22" y="236.22" smashed="yes" rot="MR0">
-<attribute name="VALUE" x="238.76" y="231.14" size="1.778" layer="96" rot="MR90"/>
-</instance>
 <instance part="U$4" gate="G$1" x="226.06" y="134.62" smashed="yes"/>
 <instance part="GND4" gate="1" x="241.3" y="114.3" smashed="yes">
@@
 <attribute name="VALUE" x="284.48" y="185.42" size="1.778" layer="96"/>
 </instance>
-<instance part="GND13" gate="1" x="30.48" y="106.68" smashed="yes">
-<attribute name="VALUE" x="27.94" y="104.14" size="1.778" layer="96"/>
-</instance>
-<instance part="P+5" gate="1" x="30.48" y="114.3" smashed="yes" rot="MR0">
-<attribute name="VALUE" x="33.02" y="109.22" size="1.778" layer="96" rot="MR90"/>
+<instance part="GND13" gate="1" x="53.34" y="116.84" smashed="yes">
+<attribute name="VALUE" x="50.8" y="114.3" size="1.778" layer="96"/>
+</instance>
+<instance part="P+5" gate="1" x="53.34" y="127" smashed="yes" rot="MR0">
+<attribute name="VALUE" x="55.88" y="121.92" size="1.778" layer="96" rot="MR90"/>
 </instance>
 <instance part="IC1" gate="1" x="177.8" y="231.14" smashed="yes">
@@
 <attribute name="VALUE" x="190.5" y="218.44" size="1.778" layer="96" rot="R90"/>
 </instance>
-<instance part="U$3" gate="G$1" x="45.72" y="111.76" smashed="yes"/>
 <instance part="U$13" gate="G$1" x="45.72" y="50.8" smashed="yes"/>
 <instance part="U$15" gate="G$1" x="45.72" y="78.74" smashed="yes"/>
@@
 <instance part="GND15" gate="1" x="139.7" y="187.96" smashed="yes">
 <attribute name="VALUE" x="137.16" y="185.42" size="1.778" layer="96"/>
+</instance>
+<instance part="U$1" gate="G$1" x="45.72" y="101.6" smashed="yes"/>
+<instance part="U$11" gate="G$1" x="10.16" y="91.44" smashed="yes"/>
+<instance part="U$12" gate="G$1" x="38.1" y="119.38" smashed="yes" rot="R180"/>
+<instance part="U$3" gate="G$1" x="10.16" y="83.82" smashed="yes"/>
+<instance part="JP2" gate="A" x="302.26" y="226.06" smashed="yes">
+<attribute name="NAME" x="295.91" y="234.315" size="1.778" layer="95"/>
+<attribute name="VALUE" x="295.91" y="218.44" size="1.778" layer="96"/>
+</instance>
+<instance part="P+4" gate="1" x="312.42" y="228.6" smashed="yes" rot="MR0">
+<attribute name="VALUE" x="314.96" y="223.52" size="1.778" layer="96" rot="MR90"/>
+</instance>
+<instance part="GND17" gate="1" x="289.56" y="220.98" smashed="yes">
+<attribute name="VALUE" x="287.02" y="218.44" size="1.778" layer="96"/>
+</instance>
+<instance part="U$14" gate="G$1" x="266.7" y="180.34" smashed="yes"/>
+<instance part="P+6" gate="1" x="-7.62" y="93.98" smashed="yes">
+<attribute name="VALUE" x="-10.16" y="88.9" size="1.778" layer="96" rot="R90"/>
+</instance>
+<instance part="GND9" gate="1" x="-7.62" y="81.28" smashed="yes">
+<attribute name="VALUE" x="-10.16" y="78.74" size="1.778" layer="96"/>
 </instance>
 </instances>
@@
 </segment>
 <segment>
-<pinref part="JP1" gate="A" pin="2_VCC"/>
-<pinref part="GND9" gate="1" pin="GND"/>
-<wire x1="243.84" y1="228.6" x2="279.4" y2="228.6" width="0.1524" layer="91"/>
-</segment>
-<segment>
 <pinref part="U$4" gate="G$1" pin="PEG2"/>
 <pinref part="GND4" gate="1" pin="GND"/>
@@
 </segment>
 <segment>
-<pinref part="GND13" gate="1" pin="GND"/>
-<pinref part="U$3" gate="G$1" pin="P$2"/>
-<wire x1="30.48" y1="109.22" x2="40.64" y2="109.22" width="0.1524" layer="91"/>
-</segment>
-<segment>
 <pinref part="U$15" gate="G$1" pin="P$1"/>
 <pinref part="GND16" gate="1" pin="GND"/>
@@
 <pinref part="R2" gate="G$1" pin="2"/>
 <pinref part="GND15" gate="1" pin="GND"/>
+</segment>
+<segment>
+<pinref part="GND13" gate="1" pin="GND"/>
+<pinref part="U$12" gate="G$1" pin="P$1"/>
+<wire x1="48.26" y1="119.38" x2="53.34" y2="119.38" width="0.1524" layer="91"/>
+</segment>
+<segment>
+<pinref part="GND17" gate="1" pin="GND"/>
+<pinref part="JP2" gate="A" pin="4"/>
+<wire x1="289.56" y1="223.52" x2="299.72" y2="223.52" width="0.1524" layer="91"/>
+</segment>
+<segment>
+<pinref part="GND9" gate="1" pin="GND"/>
+<pinref part="U$3" gate="G$1" pin="P$1"/>
+<wire x1="-7.62" y1="83.82" x2="0" y2="83.82" width="0.1524" layer="91"/>
 </segment>
 </net>
@@
 <pinref part="U$16" gate="G$1" pin="P$1"/>
 <pinref part="P+11" gate="1" pin="+5V"/>
-<wire x1="58.42" y1="91.44" x2="68.58" y2="91.44" width="0.1524" layer="91"/>
+<wire x1="58.42" y1="91.44" x2="66.04" y2="91.44" width="0.1524" layer="91"/>
+<pinref part="U$1" gate="G$1" pin="P$1"/>
+<wire x1="66.04" y1="91.44" x2="68.58" y2="91.44" width="0.1524" layer="91"/>
+<wire x1="58.42" y1="101.6" x2="66.04" y2="101.6" width="0.1524" layer="91"/>
+<wire x1="66.04" y1="101.6" x2="66.04" y2="91.44" width="0.1524" layer="91"/>
+<junction x="66.04" y="91.44"/>
+</segment>
+<segment>
+<pinref part="P+6" gate="1" pin="+5V"/>
+<pinref part="U$11" gate="G$1" pin="P$1"/>
+<wire x1="-7.62" y1="91.44" x2="0" y2="91.44" width="0.1524" layer="91"/>
 </segment>
 </net>
@@
 </segment>
 <segment>
-<pinref part="P+7" gate="1" pin="+12V"/>
-<pinref part="JP1" gate="A" pin="1_GND"/>
-<wire x1="236.22" y1="233.68" x2="243.84" y2="233.68" width="0.1524" layer="91"/>
-</segment>
-<segment>
-<pinref part="P+5" gate="1" pin="+12V"/>
-<pinref part="U$3" gate="G$1" pin="P$1"/>
-<wire x1="30.48" y1="111.76" x2="40.64" y2="111.76" width="0.1524" layer="91"/>
-</segment>
-<segment>
 <pinref part="U$13" gate="G$1" pin="P$1"/>
 <pinref part="P+10" gate="1" pin="+12V"/>
 <wire x1="58.42" y1="50.8" x2="68.58" y2="50.8" width="0.1524" layer="91"/>
+</segment>
+<segment>
+<pinref part="P+5" gate="1" pin="+12V"/>
+<pinref part="U$12" gate="G$1" pin="P$2"/>
+<wire x1="48.26" y1="124.46" x2="53.34" y2="124.46" width="0.1524" layer="91"/>
+</segment>
+<segment>
+<pinref part="JP2" gate="A" pin="3"/>
+<pinref part="P+4" gate="1" pin="+12V"/>
+<wire x1="299.72" y1="226.06" x2="312.42" y2="226.06" width="0.1524" layer="91"/>
 </segment>
 </net>
@@
 <wire x1="190.5" y1="160.02" x2="190.5" y2="190.5" width="0.1524" layer="91"/>
 <pinref part="LED1" gate="G$1" pin="A"/>
-<wire x1="190.5" y1="190.5" x2="254" y2="190.5" width="0.1524" layer="91"/>
-</segment>
-</net>
+<wire x1="190.5" y1="190.5" x2="246.38" y2="190.5" width="0.1524" layer="91"/>
+<pinref part="U$14" gate="G$1" pin="P$1"/>
+<wire x1="246.38" y1="190.5" x2="254" y2="190.5" width="0.1524" layer="91"/>
+<wire x1="256.54" y1="180.34" x2="246.38" y2="180.34" width="0.1524" layer="91"/>
+<wire x1="246.38" y1="180.34" x2="246.38" y2="190.5" width="0.1524" layer="91"/>
+<junction x="246.38" y="190.5"/>
+</segment>
+</net>

Commit message: working on new version
Parts:
- J2: device macse:ATX24RH -> blade:ATX24RH
Changed lines of the file:
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@@
 <part name="U$2" library="atx_power_control" deviceset="CAR_FUSE_HOLDER" device="3IN1"/>
 <part name="P+3" library="supply1" library_urn="urn:adsk.eagle:library:371" deviceset="+5V" device=""/>
-<part name="J2" library="macse" deviceset="ATX24" device="RH"/>
+<part name="J2" library="blade" deviceset="ATX24" device="RH"/>
 <part name="C6" library="clock" deviceset="C-US" device="C1210" value="47uF"/>
 <part name="GND11" library="supply1" library_urn="urn:adsk.eagle:library:371" deviceset="GND" device=""/>

Commit message: working on new version
Parts:
- added C12: (no value), adafruit_changed:CPOL-USE3.5-8
- added C13, C15: (no value), capacitor-wima:C5/2.5
Connections:
- net +12V: now also C12.+, C13.1, C15.1
- net GND: now also C12.-, C13.2, C15.2
Changed lines of the file:
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@@
 <part name="P+6" library="supply1" library_urn="urn:adsk.eagle:library:371" deviceset="+5V" device=""/>
 <part name="GND9" library="supply1" library_urn="urn:adsk.eagle:library:371" deviceset="GND" device=""/>
+<part name="C12" library="adafruit_changed" deviceset="CPOL-US" device="E3.5-8"/>
+<part name="P+7" library="supply1" library_urn="urn:adsk.eagle:library:371" deviceset="+12V" device=""/>
+<part name="GND18" library="supply1" library_urn="urn:adsk.eagle:library:371" deviceset="GND" device=""/>
+<part name="C13" library="capacitor-wima" library_urn="urn:adsk.eagle:library:116" deviceset="C" device="5/2.5" package3d_urn="urn:adsk.eagle:package:5426/1"/>
+<part name="C15" library="capacitor-wima" library_urn="urn:adsk.eagle:library:116" deviceset="C" device="5/2.5" package3d_urn="urn:adsk.eagle:package:5426/1"/>
+<part name="P+9" library="supply1" library_urn="urn:adsk.eagle:library:371" deviceset="+12V" device=""/>
+<part name="GND19" library="supply1" library_urn="urn:adsk.eagle:library:371" deviceset="GND" device=""/>
 </parts>
 <sheets>
@@
 <instance part="U$11" gate="G$1" x="10.16" y="91.44" smashed="yes"/>
 <instance part="U$12" gate="G$1" x="38.1" y="119.38" smashed="yes" rot="R180"/>
-<instance part="U$3" gate="G$1" x="10.16" y="83.82" smashed="yes"/>
+<instance part="U$3" gate="G$1" x="266.7" y="172.72" smashed="yes"/>
 <instance part="JP2" gate="A" x="302.26" y="226.06" smashed="yes">
 <attribute name="NAME" x="295.91" y="234.315" size="1.778" layer="95"/>
@@
 <attribute name="VALUE" x="-10.16" y="88.9" size="1.778" layer="96" rot="R90"/>
 </instance>
-<instance part="GND9" gate="1" x="-7.62" y="81.28" smashed="yes">
-<attribute name="VALUE" x="-10.16" y="78.74" size="1.778" layer="96"/>
+<instance part="GND9" gate="1" x="248.92" y="170.18" smashed="yes">
+<attribute name="VALUE" x="246.38" y="167.64" size="1.778" layer="96"/>
+</instance>
+<instance part="C12" gate="G$1" x="101.6" y="68.58" smashed="yes">
+<attribute name="NAME" x="102.616" y="69.215" size="1.778" layer="95"/>
+<attribute name="VALUE" x="102.616" y="64.389" size="1.778" layer="96"/>
+</instance>
+<instance part="P+7" gate="1" x="101.6" y="73.66" smashed="yes" rot="MR0">
+<attribute name="VALUE" x="104.14" y="68.58" size="1.778" layer="96" rot="MR90"/>
+</instance>
+<instance part="GND18" gate="1" x="101.6" y="60.96" smashed="yes">
+<attribute name="VALUE" x="99.06" y="58.42" size="1.778" layer="96"/>
+</instance>
+<instance part="C13" gate="G$1" x="127" y="68.58" smashed="yes">
+<attribute name="NAME" x="128.524" y="68.961" size="1.778" layer="95"/>
+<attribute name="VALUE" x="128.524" y="63.881" size="1.778" layer="96"/>
+</instance>
+<instance part="C15" gate="G$1" x="134.62" y="68.58" smashed="yes">
+<attribute name="NAME" x="136.144" y="68.961" size="1.778" layer="95"/>
+<attribute name="VALUE" x="136.144" y="63.881" size="1.778" layer="96"/>
+</instance>
+<instance part="P+9" gate="1" x="129.54" y="76.2" smashed="yes" rot="MR0">
+<attribute name="VALUE" x="132.08" y="71.12" size="1.778" layer="96" rot="MR90"/>
+</instance>
+<instance part="GND19" gate="1" x="132.08" y="58.42" smashed="yes">
+<attribute name="VALUE" x="129.54" y="55.88" size="1.778" layer="96"/>
 </instance>
 </instances>
@@
 <pinref part="GND9" gate="1" pin="GND"/>
 <pinref part="U$3" gate="G$1" pin="P$1"/>
-<wire x1="-7.62" y1="83.82" x2="0" y2="83.82" width="0.1524" layer="91"/>
+<wire x1="248.92" y1="172.72" x2="256.54" y2="172.72" width="0.1524" layer="91"/>
+</segment>
+<segment>
+<pinref part="C12" gate="G$1" pin="-"/>
+<pinref part="GND18" gate="1" pin="GND"/>
+</segment>
+<segment>
+<pinref part="C13" gate="G$1" pin="2"/>
+<wire x1="127" y1="60.96" x2="127" y2="63.5" width="0.1524" layer="91"/>
+<pinref part="C15" gate="G$1" pin="2"/>
+<wire x1="127" y1="60.96" x2="132.08" y2="60.96" width="0.1524" layer="91"/>
+<wire x1="132.08" y1="60.96" x2="134.62" y2="60.96" width="0.1524" layer="91"/>
+<wire x1="134.62" y1="60.96" x2="134.62" y2="63.5" width="0.1524" layer="91"/>
+<pinref part="GND19" gate="1" pin="GND"/>
+<junction x="132.08" y="60.96"/>
 </segment>
 </net>
@@
 <wire x1="299.72" y1="226.06" x2="312.42" y2="226.06" width="0.1524" layer="91"/>
 </segment>
+<segment>
+<pinref part="C12" gate="G$1" pin="+"/>
+<pinref part="P+7" gate="1" pin="+12V"/>
+</segment>
+<segment>
+<pinref part="C13" gate="G$1" pin="1"/>
+<wire x1="127" y1="73.66" x2="127" y2="71.12" width="0.1524" layer="91"/>
+<pinref part="C15" gate="G$1" pin="1"/>
+<wire x1="127" y1="73.66" x2="129.54" y2="73.66" width="0.1524" layer="91"/>
+<wire x1="129.54" y1="73.66" x2="134.62" y2="73.66" width="0.1524" layer="91"/>
+<wire x1="134.62" y1="73.66" x2="134.62" y2="71.12" width="0.1524" layer="91"/>
+<pinref part="P+9" gate="1" pin="+12V"/>
+<junction x="129.54" y="73.66"/>
+</segment>
 </net>

Commit message: working on new version
Connections:
- net GND: now also U$14.P$1; no longer U$3.P$1
- net N$4: now also U$3.P$1; no longer U$14.P$1
Changed lines of the file:
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@@
 <attribute name="VALUE" x="-10.16" y="88.9" size="1.778" layer="96" rot="R90"/>
 </instance>
-<instance part="GND9" gate="1" x="248.92" y="170.18" smashed="yes">
-<attribute name="VALUE" x="246.38" y="167.64" size="1.778" layer="96"/>
+<instance part="GND9" gate="1" x="251.46" y="177.8" smashed="yes">
+<attribute name="VALUE" x="248.92" y="175.26" size="1.778" layer="96"/>
 </instance>
 <instance part="C12" gate="G$1" x="101.6" y="68.58" smashed="yes">
@@
 </segment>
 <segment>
-<pinref part="GND9" gate="1" pin="GND"/>
-<pinref part="U$3" gate="G$1" pin="P$1"/>
-<wire x1="248.92" y1="172.72" x2="256.54" y2="172.72" width="0.1524" layer="91"/>
-</segment>
-<segment>
 <pinref part="C12" gate="G$1" pin="-"/>
 <pinref part="GND18" gate="1" pin="GND"/>
@@
 <pinref part="GND19" gate="1" pin="GND"/>
 <junction x="132.08" y="60.96"/>
+</segment>
+<segment>
+<pinref part="GND9" gate="1" pin="GND"/>
+<pinref part="U$14" gate="G$1" pin="P$1"/>
+<wire x1="251.46" y1="180.34" x2="256.54" y2="180.34" width="0.1524" layer="91"/>
 </segment>
 </net>
@@
 <pinref part="LED1" gate="G$1" pin="A"/>
 <wire x1="190.5" y1="190.5" x2="246.38" y2="190.5" width="0.1524" layer="91"/>
-<pinref part="U$14" gate="G$1" pin="P$1"/>
 <wire x1="246.38" y1="190.5" x2="254" y2="190.5" width="0.1524" layer="91"/>
-<wire x1="256.54" y1="180.34" x2="246.38" y2="180.34" width="0.1524" layer="91"/>
-<wire x1="246.38" y1="180.34" x2="246.38" y2="190.5" width="0.1524" layer="91"/>
+<wire x1="246.38" y1="172.72" x2="246.38" y2="190.5" width="0.1524" layer="91"/>
 <junction x="246.38" y="190.5"/>
-</segment>
-</net>
+<pinref part="U$3" gate="G$1" pin="P$1"/>
+<wire x1="246.38" y1="172.72" x2="256.54" y2="172.72" width="0.1524" layer="91"/>
+</segment>
+</net>
