File: pcb/osborne_1/osborne1.brd (EAGLE design)
At the start: 40 x 97 mm, 20 parts, among them J2 ATX24RH

Commit message: added more caps to OS1
Parts:
- removed JP4: (no value), pinhead:1X03
- removed LED1, LED2: (no value), SparkFun-LED:LED_3MM
- removed R1, R2: (no value), adafruit:0207/2V
- added C3, C5: (no value), capacitor-wima:C5B2.5
- added C4, C6: (no value), adafruit_changed:E3,5-8
- moved TP2 1.02 mm to (35.8, 13.4)
- moved TP1 1.02 mm to (30.8, 13.4)
- moved C2 0.92 mm to (8.76, 60.5)
- moved C1 0.77 mm to (8.76, 69.7), turned to 270 degrees
Connections:
- removed net N$2: JP3.2, JP4.2
- removed net N$3: LED1.K, R2.1
- removed net N$4: LED2.K, R1.1
- net +12V: now also C3.1, C6.+, JP3.2; no longer JP4.1, LED2.A
- net +5V: now also C4.+, C5.1; no longer JP4.3, LED1.A
- net GND: now also C3.2, C4.-, C5.2, C6.-; no longer R1.2, R2.2
Routing:
- net +5V: track 72.6 -> 83.8 mm
- net +12V: track 48.9 -> 58.3 mm
- net N$2: track 4.56 -> 0.00 mm
- net N$4: track 4.31 -> 0.00 mm
- net N$3: track 3.08 -> 0.00 mm
Other:
- board text added: "PD2 dekuNukem JUL 2023"
- board text removed: "12"
- board text removed: "5"
- board text removed: "PD1 dekuNukem APR 2023"

Commit message: working on new version
Changed lines of the file:
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@@
 <text x="8.001" y="5.207" size="2.1844" layer="25" distance="35" align="center">FUSE
 5A MAX</text>
-<hole x="35.433" y="24.13" drill="8.25"/>
+<hole x="35.306" y="24.13" drill="8.25"/>
 <wire x1="45" y1="10" x2="-5" y2="10" width="0.1524" layer="51"/>
 <wire x1="0" y1="87" x2="87" y2="87" width="0.1524" layer="51"/>

Commit message: working on new version
Parts:
- moved C5 11.9 mm to (4.45, 81.5), turned to 90 degrees
- moved C1 11.8 mm to (7.87, 81.5), turned to 90 degrees
- moved C3 11.4 mm to (6.73, 49.1), turned to 225 degrees
- moved C4 10.3 mm to (5.97, 70.4), turned to 270 degrees
- moved C6 9.53 mm to (5.97, 61.5), turned to 135 degrees
- moved C2 6.83 mm to (6.60, 54.0), turned to 225 degrees
Routing:
- net +5V: track 83.8 -> 81.7 mm
- net +12V: track 58.3 -> 57.5 mm
- net N$1: track 60.2 -> 59.5 mm
