File: pcb/apple_iigs/iigs.sch (EAGLE design)
At the start: 15 parts, among them J1 ATX24RH

Commit message: removed fan voltage selector
Parts:
- removed JP2: (no value), pinhead:PINHD-1X3
Connections:
- removed net N$1: JP2.2, JP4.2_VCC
- net +12V: now also JP4.2_VCC; no longer JP2.3
- net +5V: no longer JP2.1
Changed lines of the file:
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@@
 <part name="P-7" library="supply1" library_urn="urn:adsk.eagle:library:371" deviceset="-12V" device=""/>
 <part name="JP4" library="appleii" deviceset="4PIN_FAN" device=""/>
-<part name="JP2" library="pinhead" library_urn="urn:adsk.eagle:library:325" deviceset="PINHD-1X3" device="" package3d_urn="urn:adsk.eagle:package:22458/2"/>
 <part name="GND1" library="supply1" library_urn="urn:adsk.eagle:library:371" deviceset="GND" device=""/>
-<part name="P+1" library="supply1" library_urn="urn:adsk.eagle:library:371" deviceset="+5V" device=""/>
 <part name="P+4" library="supply1" library_urn="urn:adsk.eagle:library:371" deviceset="+12V" device=""/>
 <part name="C11" library="clock" deviceset="C-US" device="C1210" value="47uF"/>
@@
 </instance>
 <instance part="JP4" gate="A" x="-17.78" y="175.26" smashed="yes"/>
-<instance part="JP2" gate="A" x="0" y="177.8" smashed="yes">
-<attribute name="NAME" x="-6.35" y="183.515" size="1.778" layer="95"/>
-<attribute name="VALUE" x="-6.35" y="170.18" size="1.778" layer="96"/>
-</instance>
 <instance part="GND1" gate="1" x="-43.18" y="180.34" smashed="yes">
 <attribute name="VALUE" x="-45.72" y="177.8" size="1.778" layer="96"/>
 </instance>
-<instance part="P+1" gate="1" x="7.62" y="182.88" smashed="yes">
-<attribute name="VALUE" x="5.08" y="177.8" size="1.778" layer="96" rot="R90"/>
-</instance>
-<instance part="P+4" gate="1" x="20.32" y="177.8" smashed="yes" rot="MR0">
-<attribute name="VALUE" x="22.86" y="172.72" size="1.778" layer="96" rot="MR90"/>
+<instance part="P+4" gate="1" x="-2.54" y="180.34" smashed="yes" rot="MR0">
+<attribute name="VALUE" x="0" y="175.26" size="1.778" layer="96" rot="MR90"/>
 </instance>
 <instance part="C11" gate="G$1" x="0" y="137.16" smashed="yes">
@@
 </segment>
 <segment>
-<pinref part="JP2" gate="A" pin="1"/>
-<pinref part="P+1" gate="1" pin="+5V"/>
-<wire x1="-2.54" y1="180.34" x2="7.62" y2="180.34" width="0.1524" layer="91"/>
-</segment>
-<segment>
 <pinref part="C11" gate="G$1" pin="1"/>
 <pinref part="C13" gate="G$1" pin="2"/>
@@
 </segment>
 <segment>
-<pinref part="JP2" gate="A" pin="3"/>
 <pinref part="P+4" gate="1" pin="+12V"/>
-<wire x1="-2.54" y1="175.26" x2="20.32" y2="175.26" width="0.1524" layer="91"/>
+<pinref part="JP4" gate="A" pin="2_VCC"/>
+<wire x1="-30.48" y1="177.8" x2="-2.54" y2="177.8" width="0.1524" layer="91"/>
 </segment>
 <segment>
@@
 </segment>
 </net>
-<net name="N$1" class="0">
-<segment>
-<pinref part="JP4" gate="A" pin="2_VCC"/>
-<pinref part="JP2" gate="A" pin="2"/>
-<wire x1="-30.48" y1="177.8" x2="-2.54" y2="177.8" width="0.1524" layer="91"/>
-</segment>
-</net>
