File: pcb/ibmpc/at/ibm.brd (EAGLE design)
At the start: 104 x 76 mm, 33 parts, among them J2 ATX24RH

Commit message: working on new version
Parts:
- added U$1: 20PEDGE, apricot:20P_EDGE
- added U$11: M3_MOUNTING_HOLE, apricot:M3_MOUNTING_HOLE_PACK
- moved U$3 121.8 mm to (40.8, 15.2)
- moved C14 114.3 mm to (25.7, 6.87)
- moved C1 111.5 mm to (25.2, 34.2)
- moved C10 111.5 mm to (37.0, 28.2)
- moved C16 111.5 mm to (37.4, 21.3)
- moved C17 111.5 mm to (25.6, 21.3)
- moved C2 111.5 mm to (36.5, 24.4)
- moved C3 111.5 mm to (25.8, 30.4)
- moved C4 111.5 mm to (25.6, 24.4)
- moved C5 111.5 mm to (26.0, 26.3)
- moved C6 111.5 mm to (36.9, 34.3)
- moved C7 111.5 mm to (26.0, 28.2)
- moved C8 111.5 mm to (37.0, 26.3)
- moved C9 111.5 mm to (36.9, 30.4)
- moved U$2 111.5 mm to (37.0, 45.0)
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Connections:
- new net N$5: J2.9, U$1.P$9
- net +12V: now also U$1.P$10
- net +5V: now also U$1.P$19, U$1.P$20, U$1.P$4, U$1.P$6
- net -12V: now also U$1.P$12
- net -5V: now also U$1.P$18
- net GND: now also U$1.P$13, U$1.P$15, U$1.P$16, U$1.P$17, U$1.P$3, U$1.P$5, U$1.P$7, U$11.P$1, U$11.P$2
- net N$3: now also U$1.P$14
- net N$4: now also U$1.P$8
Routing:
- net N$4: track 0.00 -> 185.6 mm, vias 0 -> 1
- net +5V: track 0.00 -> 137.2 mm, vias 0 -> 4
- net N$3: track 0.00 -> 134.1 mm, vias 0 -> 2
- net +12V: track 0.00 -> 113.2 mm, vias 0 -> 1
- net N$5: track 0.00 -> 101.4 mm
- net -5V: track 0.00 -> 100.8 mm, vias 0 -> 1
- net -12V: track 0.00 -> 97.8 mm, vias 0 -> 1
- net N$8: track 0.00 -> 93.3 mm
- net GND: track 0.00 -> 91.8 mm, vias 0 -> 3
- net N$6: track 0.00 -> 32.8 mm
- net N$1: track 0.00 -> 14.0 mm
- net N$12: track 0.00 -> 6.26 mm
Other:
- board size 104 x 76 mm -> 123 x 64.6 mm

Commit message: working on improvements
Parts:
- removed JP1: (no value), appleii:1X04
- removed U$11: M3_MOUNTING_HOLE, apricot:M3_MOUNTING_HOLE_PACK
- removed U$3: VH396_2P, 396_conn:396_2P
- added JP2: (no value), pinhead:1X04/90
- moved JP3 91.3 mm to (14.7, 61.3)
- moved C11 12.5 mm to (38.2, 4.04)
- moved C14 11.8 mm to (37.5, 6.74)
- moved IC1 10.6 mm to (37.5, 14.1)
- moved U$8 9.50 mm to (34.3, 45.0)
- moved C1 9.05 mm to (34.2, 33.9)
- moved J2 9.00 mm to (17.7, 29.6)
- moved C3 8.50 mm to (34.3, 30.4)
- moved C4 8.38 mm to (34.0, 24.4)
- moved C5 8.29 mm to (34.2, 26.7)
- moved C7 8.29 mm to (34.2, 28.5)
- moved C17 8.25 mm to (33.8, 21.3)
- moved R2 8.24 mm to (17.7, 2.67), turned to 180 degrees
- moved C2 6.75 mm to (43.2, 24.4)
- moved U$2 6.50 mm to (43.5, 45.0)
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Connections:
- net +12V: no longer JP1.1, U$3.P$1
- net GND: no longer JP1.2, U$11.P$1, U$11.P$2, U$3.P$2
Routing:
- net N$3: track 134.1 -> 63.0 mm
- net N$8: track 93.3 -> 42.8 mm
- net -12V: track 97.8 -> 47.7 mm
- net +12V: track 113.2 -> 70.0 mm
- net +5V: track 137.2 -> 96.3 mm
- net -5V: track 100.8 -> 60.7 mm
- net GND: track 91.8 -> 79.1 mm
- net N$5: track 101.4 -> 92.2 mm
- net N$4: track 185.6 -> 176.9 mm
- net N$1: track 14.0 -> 9.70 mm
- net N$6: track 32.8 -> 33.8 mm
Other:
- board size 123 x 64.6 mm -> 114 x 65.6 mm
- board text added: "120mil for 7.5A"
- board text removed: "5V"
- board text removed: "ISA Bracket ------>"
- board text removed: "ISA Bracket <------"

Commit message: working on improvements
Parts:
- added U$3: ISA, blade:ISAPAD
- moved JP3 99.2 mm to (112.0, 41.9)
- moved JP2 5.59 mm to (103.9, 41.9)
- moved J2 0.50 mm to (18.2, 29.6)
- moved R2 0.13 mm to (17.6, 2.67)
Connections:
- net +5V: now also U$3.P$1
Routing:
- net N$6: track 33.8 -> 33.3 mm
- net N$5: track 92.2 -> 91.7 mm
- net N$4: track 176.9 -> 176.4 mm

Commit message: working on improvements
Parts:
- moved JP3 94.8 mm to (19.2, 61.3)
- moved JP2 59.2 mm to (47.9, 61.3)
- moved R2 46.1 mm to (-22.2, 25.9), turned to 270 degrees
- moved C1 6.00 mm to (40.2, 33.9)
- moved C10 6.00 mm to (49.0, 28.2)
- moved C11 6.00 mm to (44.2, 4.04)
- moved C14 6.00 mm to (43.5, 6.74)
- moved C16 6.00 mm to (49.3, 21.3)
- moved C17 6.00 mm to (39.8, 21.3)
- moved C2 6.00 mm to (49.2, 24.4)
- moved C3 6.00 mm to (40.3, 30.4)
- moved C4 6.00 mm to (40.0, 24.4)
- moved C5 6.00 mm to (40.2, 26.7)
- moved C6 6.00 mm to (48.9, 34.3)
- moved C7 6.00 mm to (40.2, 28.5)
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Routing:
- net N$8: track 42.6 -> 18.0 mm
- net N$4: track 176.4 -> 170.1 mm
- net N$12: track 6.26 -> 0.00 mm
- net N$3: track 63.0 -> 57.0 mm
- net +5V: track 96.2 -> 99.7 mm
- net +12V: track 70.0 -> 73.2 mm
- net -5V: track 60.7 -> 63.6 mm
- net GND: track 79.1 -> 76.3 mm
- net -12V: track 47.7 -> 50.2 mm
- net N$5: track 91.7 -> 91.1 mm
Other:
- board size 114 x 65.6 mm -> 108 x 69.6 mm
- board text added: "5A FUSE"
- board text removed: "FUSE 5A MAX"
- board text removed: "put a sticker on 7905 laying down footprint"

Commit message: working on improvements
Parts:
- added U$11: M3_MOUNTING_HOLE, apricot:M3_MOUNTING_HOLE_PACK
- moved R1 30.1 mm to (91.9, 13.6), turned to 0 degrees
- moved C1 16.8 mm to (25.2, 41.5)
- moved C10 16.8 mm to (34.0, 35.8)
- moved C11 16.8 mm to (29.2, 11.7)
- moved C16 16.8 mm to (34.3, 28.9)
- moved C17 16.8 mm to (24.8, 28.9)
- moved C5 16.8 mm to (25.2, 34.3)
- moved C7 16.8 mm to (25.2, 36.1)
- moved C8 16.8 mm to (34.0, 33.9)
- moved C9 16.8 mm to (33.9, 38.0)
- moved JP2 16.8 mm to (32.9, 68.9)
- moved JP3 16.8 mm to (4.19, 68.9)
- moved U$1 16.8 mm to (64.0, 23.6)
- moved U$10 16.8 mm to (67.3, 3.91)
- moved U$15 16.8 mm to (6.39, 3.91)
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Routing:
- net GND: track 76.3 -> 55.7 mm
- net N$8: track 18.0 -> 7.70 mm
- net N$4: track 170.1 -> 169.1 mm
Other:
- board size 108 x 69.6 mm -> 108 x 75 mm
- board text added: "5V and 12V right angle blade down here?"
- board text added: "GND and PG right angle blade here?"
- board text added: "extend PCB right to here"
