File: pcb/ibmpc/at/ibm.sch (EAGLE design)
At the start: 33 parts, among them J2 ATX24RH

Commit message: working on new version
Parts:
- added U$1: 20PEDGE, apricot:20PEDGE
- added U$11: M3_MOUNTING_HOLE, apricot:M3_MOUNTING_HOLE
Connections:
- new net N$5: J2.5V_STDBY, U$1.5VSB
- net +12V: now also U$1.12V
- net +5V: now also U$1.5V
- net -12V: now also U$1.-12V
- net -5V: now also U$1.-5V
- net GND: now also U$1.GND, U$11.P$1, U$11.P$2
- net N$3: now also U$1.PS_ON
- net N$4: now also U$1.PWR_OK
Changed lines of the file:
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@@
 <part name="U$6" library="apricot" deviceset="M3_MOUNTING_HOLE" device=""/>
 <part name="GND6" library="supply1" library_urn="urn:adsk.eagle:library:371" deviceset="GND" device=""/>
+<part name="U$1" library="apricot" deviceset="20PEDGE" device=""/>
 <part name="C9" library="adafruit_changed" deviceset="CPOL-US" device="E3.5-8"/>
 <part name="C2" library="capacitor-wima" library_urn="urn:adsk.eagle:library:116" deviceset="C" device="5/2.5" package3d_urn="urn:adsk.eagle:package:5426/1"/>
@@
 <part name="C10" library="clock" deviceset="CAP" device="0805" value="100nF"/>
 <part name="GND5" library="supply1" library_urn="urn:adsk.eagle:library:371" deviceset="GND" device=""/>
+<part name="P+4" library="supply1" library_urn="urn:adsk.eagle:library:371" deviceset="+5V" device=""/>
+<part name="P+6" library="supply1" library_urn="urn:adsk.eagle:library:371" deviceset="+12V" device=""/>
 <part name="GND7" library="supply1" library_urn="urn:adsk.eagle:library:371" deviceset="GND" device=""/>
 <part name="C14" library="capacitor-wima" library_urn="urn:adsk.eagle:library:116" deviceset="C" device="5/2.5" package3d_urn="urn:adsk.eagle:package:5426/1"/>
@@
 <part name="P-2" library="supply1" library_urn="urn:adsk.eagle:library:371" deviceset="-5V" device=""/>
 <part name="U$3" library="396_conn" deviceset="VH396_2P" device=""/>
+<part name="U$11" library="apricot" deviceset="M3_MOUNTING_HOLE" device=""/>
 <part name="U$13" library="blade" deviceset="ISA" device=""/>
 <part name="U$15" library="blade" deviceset="ISA" device=""/>
@@
 <attribute name="VALUE" x="-10.16" y="162.56" size="1.778" layer="96"/>
 </instance>
+<instance part="U$1" gate="G$1" x="101.6" y="254" smashed="yes"/>
 <instance part="C9" gate="G$1" x="109.22" y="104.14" smashed="yes">
 <attribute name="NAME" x="110.236" y="104.775" size="1.778" layer="95"/>
@@
 <instance part="GND5" gate="1" x="129.54" y="231.14" smashed="yes">
 <attribute name="VALUE" x="127" y="228.6" size="1.778" layer="96"/>
+</instance>
+<instance part="P+4" gate="1" x="139.7" y="261.62" smashed="yes">
+<attribute name="VALUE" x="137.16" y="256.54" size="1.778" layer="96" rot="R90"/>
+</instance>
+<instance part="P+6" gate="1" x="142.24" y="266.7" smashed="yes" rot="MR0">
+<attribute name="VALUE" x="144.78" y="261.62" size="1.778" layer="96" rot="MR90"/>
 </instance>
 <instance part="GND7" gate="1" x="177.8" y="243.84" smashed="yes" rot="R180">
@@
 </instance>
 <instance part="U$3" gate="G$1" x="45.72" y="111.76" smashed="yes"/>
+<instance part="U$11" gate="G$1" x="-35.56" y="205.74" smashed="yes"/>
 <instance part="U$13" gate="G$1" x="45.72" y="50.8" smashed="yes"/>
 <instance part="U$15" gate="G$1" x="45.72" y="78.74" smashed="yes"/>
@@
 <wire x1="-12.7" y1="167.64" x2="-7.62" y2="167.64" width="0.1524" layer="91"/>
 <junction x="-7.62" y="167.64"/>
+<pinref part="U$11" gate="G$1" pin="P$1"/>
+<wire x1="-12.7" y1="210.82" x2="-7.62" y2="210.82" width="0.1524" layer="91"/>
+<wire x1="-7.62" y1="210.82" x2="-7.62" y2="203.2" width="0.1524" layer="91"/>
+<junction x="-7.62" y="193.04"/>
+<pinref part="U$11" gate="G$1" pin="P$2"/>
+<wire x1="-7.62" y1="203.2" x2="-7.62" y2="193.04" width="0.1524" layer="91"/>
+<wire x1="-12.7" y1="203.2" x2="-7.62" y2="203.2" width="0.1524" layer="91"/>
+<junction x="-7.62" y="203.2"/>
 </segment>
 <segment>
@@
 </segment>
 <segment>
+<pinref part="U$1" gate="G$1" pin="GND"/>
 <pinref part="GND5" gate="1" pin="GND"/>
 <wire x1="114.3" y1="233.68" x2="129.54" y2="233.68" width="0.1524" layer="91"/>
@@
 </segment>
 <segment>
+<pinref part="P+4" gate="1" pin="+5V"/>
+<pinref part="U$1" gate="G$1" pin="5V"/>
+<wire x1="139.7" y1="259.08" x2="114.3" y2="259.08" width="0.1524" layer="91"/>
+</segment>
+<segment>
 <pinref part="U$16" gate="G$1" pin="P$1"/>
 <pinref part="P+11" gate="1" pin="+5V"/>
@@
 </segment>
 <segment>
+<pinref part="U$1" gate="G$1" pin="12V"/>
+<pinref part="P+6" gate="1" pin="+12V"/>
+<wire x1="114.3" y1="264.16" x2="142.24" y2="264.16" width="0.1524" layer="91"/>
+</segment>
+<segment>
 <pinref part="P+7" gate="1" pin="+12V"/>
 <pinref part="JP1" gate="A" pin="1_GND"/>
@@
 <wire x1="109.22" y1="167.64" x2="215.9" y2="167.64" width="0.1524" layer="91"/>
 <wire x1="215.9" y1="167.64" x2="215.9" y2="248.92" width="0.1524" layer="91"/>
+<pinref part="U$1" gate="G$1" pin="-12V"/>
 <wire x1="215.9" y1="248.92" x2="203.2" y2="248.92" width="0.1524" layer="91"/>
 <wire x1="203.2" y1="248.92" x2="162.56" y2="248.92" width="0.1524" layer="91"/>
@@
 <segment>
 <pinref part="J2" gate="G$1" pin="PS_ON"/>
-<wire x1="109.22" y1="162.56" x2="231.14" y2="162.56" width="0.1524" layer="91"/>
+<wire x1="109.22" y1="162.56" x2="195.58" y2="162.56" width="0.1524" layer="91"/>
+<wire x1="195.58" y1="162.56" x2="195.58" y2="205.74" width="0.1524" layer="91"/>
+<wire x1="195.58" y1="205.74" x2="60.96" y2="205.74" width="0.1524" layer="91"/>
+<wire x1="60.96" y1="205.74" x2="60.96" y2="233.68" width="0.1524" layer="91"/>
+<pinref part="U$1" gate="G$1" pin="PS_ON"/>
+<wire x1="60.96" y1="233.68" x2="78.74" y2="233.68" width="0.1524" layer="91"/>
 <pinref part="JP3" gate="G$1" pin="1"/>
+<wire x1="195.58" y1="162.56" x2="231.14" y2="162.56" width="0.1524" layer="91"/>
+<junction x="195.58" y="162.56"/>
 <wire x1="231.14" y1="162.56" x2="251.46" y2="162.56" width="0.1524" layer="91"/>
 <wire x1="251.46" y1="162.56" x2="251.46" y2="134.62" width="0.1524" layer="91"/>
@@
 <wire x1="109.22" y1="160.02" x2="190.5" y2="160.02" width="0.1524" layer="91"/>
 <wire x1="190.5" y1="160.02" x2="190.5" y2="190.5" width="0.1524" layer="91"/>
+<wire x1="190.5" y1="190.5" x2="190.5" y2="203.2" width="0.1524" layer="91"/>
+<wire x1="190.5" y1="203.2" x2="63.5" y2="203.2" width="0.1524" layer="91"/>
+<wire x1="63.5" y1="203.2" x2="63.5" y2="228.6" width="0.1524" layer="91"/>
+<pinref part="U$1" gate="G$1" pin="PWR_OK"/>
+<wire x1="63.5" y1="228.6" x2="78.74" y2="228.6" width="0.1524" layer="91"/>
 <pinref part="LED1" gate="G$1" pin="A"/>
 <wire x1="190.5" y1="190.5" x2="254" y2="190.5" width="0.1524" layer="91"/>
+<junction x="190.5" y="190.5"/>
+</segment>
+</net>
+<net name="N$5" class="0">
+<segment>
+<pinref part="J2" gate="G$1" pin="5V_STDBY"/>
+<wire x1="81.28" y1="177.8" x2="5.08" y2="177.8" width="0.1524" layer="91"/>
+<wire x1="5.08" y1="177.8" x2="5.08" y2="238.76" width="0.1524" layer="91"/>
+<pinref part="U$1" gate="G$1" pin="5VSB"/>
+<wire x1="5.08" y1="238.76" x2="114.3" y2="238.76" width="0.1524" layer="91"/>
 </segment>
 </net>
@@
 <wire x1="193.04" y1="223.52" x2="149.86" y2="223.52" width="0.1524" layer="91"/>
 <wire x1="149.86" y1="223.52" x2="149.86" y2="243.84" width="0.1524" layer="91"/>
+<pinref part="U$1" gate="G$1" pin="-5V"/>
 <pinref part="C14" gate="G$1" pin="1"/>
 <wire x1="149.86" y1="243.84" x2="114.3" y2="243.84" width="0.1524" layer="91"/>

Commit message: working on improvements
Parts:
- removed JP1: (no value), appleii:4PIN_FAN
- removed U$11: M3_MOUNTING_HOLE, apricot:M3_MOUNTING_HOLE
- removed U$3: VH396_2P, 396_conn:VH396_2P
- added JP2: (no value), pinhead:PINHD-1X4/90
Connections:
- net +12V: no longer JP1.1_GND, U$3.P$1
- net GND: no longer JP1.2_VCC, U$11.P$1, U$11.P$2, U$3.P$2
Changed lines of the file:
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@@
 <part name="C14" library="capacitor-wima" library_urn="urn:adsk.eagle:library:116" deviceset="C" device="5/2.5" package3d_urn="urn:adsk.eagle:package:5426/1"/>
 <part name="GND8" library="supply1" library_urn="urn:adsk.eagle:library:371" deviceset="GND" device=""/>
-<part name="JP1" library="appleii" deviceset="4PIN_FAN" device=""/>
-<part name="GND9" library="supply1" library_urn="urn:adsk.eagle:library:371" deviceset="GND" device=""/>
-<part name="P+7" library="supply1" library_urn="urn:adsk.eagle:library:371" deviceset="+12V" device=""/>
 <part name="U$4" library="apricot" deviceset="ROCKSW" device=""/>
 <part name="GND4" library="supply1" library_urn="urn:adsk.eagle:library:371" deviceset="GND" device=""/>
@@
 <part name="R1" library="adafruit" deviceset="R-US_" device="0207/10" value="470"/>
 <part name="GND12" library="supply1" library_urn="urn:adsk.eagle:library:371" deviceset="GND" device=""/>
-<part name="GND13" library="supply1" library_urn="urn:adsk.eagle:library:371" deviceset="GND" device=""/>
-<part name="P+5" library="supply1" library_urn="urn:adsk.eagle:library:371" deviceset="+12V" device=""/>
 <part name="IC1" library="v-reg" library_urn="urn:adsk.eagle:library:409" deviceset="79XXS" device="" package3d_urn="urn:adsk.eagle:package:30343/1"/>
 <part name="C16" library="capacitor-wima" library_urn="urn:adsk.eagle:library:116" deviceset="C" device="5/2.5" package3d_urn="urn:adsk.eagle:package:5426/1"/>
@@
 <part name="P-1" library="supply1" library_urn="urn:adsk.eagle:library:371" deviceset="-12V" device=""/>
 <part name="P-2" library="supply1" library_urn="urn:adsk.eagle:library:371" deviceset="-5V" device=""/>
-<part name="U$3" library="396_conn" deviceset="VH396_2P" device=""/>
-<part name="U$11" library="apricot" deviceset="M3_MOUNTING_HOLE" device=""/>
 <part name="U$13" library="blade" deviceset="ISA" device=""/>
 <part name="U$15" library="blade" deviceset="ISA" device=""/>
@@
 <part name="R2" library="adafruit_changed" deviceset="R-US_" device="0411/15"/>
 <part name="GND15" library="supply1" library_urn="urn:adsk.eagle:library:371" deviceset="GND" device=""/>
+<part name="JP2" library="pinhead" library_urn="urn:adsk.eagle:library:325" deviceset="PINHD-1X4" device="/90" package3d_urn="urn:adsk.eagle:package:22404/2"/>
 </parts>
 <sheets>
@@
 <attribute name="VALUE" x="203.2" y="223.52" size="1.778" layer="96"/>
 </instance>
-<instance part="JP1" gate="A" x="256.54" y="226.06" smashed="yes"/>
-<instance part="GND9" gate="1" x="279.4" y="226.06" smashed="yes">
-<attribute name="VALUE" x="276.86" y="223.52" size="1.778" layer="96"/>
-</instance>
-<instance part="P+7" gate="1" x="236.22" y="236.22" smashed="yes" rot="MR0">
-<attribute name="VALUE" x="238.76" y="231.14" size="1.778" layer="96" rot="MR90"/>
-</instance>
 <instance part="U$4" gate="G$1" x="226.06" y="134.62" smashed="yes"/>
 <instance part="GND4" gate="1" x="241.3" y="114.3" smashed="yes">
@@
 <instance part="GND12" gate="1" x="287.02" y="187.96" smashed="yes">
 <attribute name="VALUE" x="284.48" y="185.42" size="1.778" layer="96"/>
-</instance>
-<instance part="GND13" gate="1" x="30.48" y="106.68" smashed="yes">
-<attribute name="VALUE" x="27.94" y="104.14" size="1.778" layer="96"/>
-</instance>
-<instance part="P+5" gate="1" x="30.48" y="114.3" smashed="yes" rot="MR0">
-<attribute name="VALUE" x="33.02" y="109.22" size="1.778" layer="96" rot="MR90"/>
 </instance>
 <instance part="IC1" gate="1" x="177.8" y="231.14" smashed="yes">
@@
 <attribute name="VALUE" x="190.5" y="218.44" size="1.778" layer="96" rot="R90"/>
 </instance>
-<instance part="U$3" gate="G$1" x="45.72" y="111.76" smashed="yes"/>
-<instance part="U$11" gate="G$1" x="-35.56" y="205.74" smashed="yes"/>
 <instance part="U$13" gate="G$1" x="45.72" y="50.8" smashed="yes"/>
 <instance part="U$15" gate="G$1" x="45.72" y="78.74" smashed="yes"/>
@@
 <instance part="GND15" gate="1" x="139.7" y="187.96" smashed="yes">
 <attribute name="VALUE" x="137.16" y="185.42" size="1.778" layer="96"/>
+</instance>
+<instance part="JP2" gate="A" x="-15.24" y="220.98" smashed="yes">
+<attribute name="NAME" x="-21.59" y="229.235" size="1.778" layer="95"/>
+<attribute name="VALUE" x="-21.59" y="213.36" size="1.778" layer="96"/>
 </instance>
 </instances>
@@
 <wire x1="-12.7" y1="167.64" x2="-7.62" y2="167.64" width="0.1524" layer="91"/>
 <junction x="-7.62" y="167.64"/>
-<pinref part="U$11" gate="G$1" pin="P$1"/>
-<wire x1="-12.7" y1="210.82" x2="-7.62" y2="210.82" width="0.1524" layer="91"/>
-<wire x1="-7.62" y1="210.82" x2="-7.62" y2="203.2" width="0.1524" layer="91"/>
-<junction x="-7.62" y="193.04"/>
-<pinref part="U$11" gate="G$1" pin="P$2"/>
-<wire x1="-7.62" y1="203.2" x2="-7.62" y2="193.04" width="0.1524" layer="91"/>
-<wire x1="-12.7" y1="203.2" x2="-7.62" y2="203.2" width="0.1524" layer="91"/>
-<junction x="-7.62" y="203.2"/>
 </segment>
 <segment>
@@
 </segment>
 <segment>
-<pinref part="JP1" gate="A" pin="2_VCC"/>
-<pinref part="GND9" gate="1" pin="GND"/>
-<wire x1="243.84" y1="228.6" x2="279.4" y2="228.6" width="0.1524" layer="91"/>
-</segment>
-<segment>
 <pinref part="U$4" gate="G$1" pin="PEG2"/>
 <pinref part="GND4" gate="1" pin="GND"/>
@@
 <pinref part="C11" gate="G$1" pin="2"/>
 <pinref part="GND3" gate="1" pin="GND"/>
-</segment>
-<segment>
-<pinref part="GND13" gate="1" pin="GND"/>
-<pinref part="U$3" gate="G$1" pin="P$2"/>
-<wire x1="30.48" y1="109.22" x2="40.64" y2="109.22" width="0.1524" layer="91"/>
 </segment>
 <segment>
@@
 </segment>
 <segment>
-<pinref part="P+7" gate="1" pin="+12V"/>
-<pinref part="JP1" gate="A" pin="1_GND"/>
-<wire x1="236.22" y1="233.68" x2="243.84" y2="233.68" width="0.1524" layer="91"/>
-</segment>
-<segment>
-<pinref part="P+5" gate="1" pin="+12V"/>
-<pinref part="U$3" gate="G$1" pin="P$1"/>
-<wire x1="30.48" y1="111.76" x2="40.64" y2="111.76" width="0.1524" layer="91"/>
-</segment>
-<segment>

Commit message: working on improvements
Parts:
- added U$3: ISA, blade:ISA
Connections:
- net +5V: now also U$3.P$1
Changed lines of the file:
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@@
 <part name="GND15" library="supply1" library_urn="urn:adsk.eagle:library:371" deviceset="GND" device=""/>
 <part name="JP2" library="pinhead" library_urn="urn:adsk.eagle:library:325" deviceset="PINHD-1X4" device="/90" package3d_urn="urn:adsk.eagle:package:22404/2"/>
+<part name="U$3" library="blade" deviceset="ISA" device=""/>
+<part name="P+5" library="supply1" library_urn="urn:adsk.eagle:library:371" deviceset="+5V" device=""/>
 </parts>
 <sheets>
@@
 <attribute name="NAME" x="-21.59" y="229.235" size="1.778" layer="95"/>
 <attribute name="VALUE" x="-21.59" y="213.36" size="1.778" layer="96"/>
+</instance>
+<instance part="U$3" gate="G$1" x="45.72" y="106.68" smashed="yes"/>
+<instance part="P+5" gate="1" x="68.58" y="109.22" smashed="yes">
+<attribute name="VALUE" x="66.04" y="104.14" size="1.778" layer="96" rot="R90"/>
 </instance>
 </instances>
@@
 <wire x1="58.42" y1="91.44" x2="68.58" y2="91.44" width="0.1524" layer="91"/>
 </segment>
+<segment>
+<pinref part="U$3" gate="G$1" pin="P$1"/>
+<pinref part="P+5" gate="1" pin="+5V"/>
+<wire x1="58.42" y1="106.68" x2="68.58" y2="106.68" width="0.1524" layer="91"/>
+</segment>
 </net>

Commit message: working on improvements
Parts:
- added U$11: M3_MOUNTING_HOLE, apricot:M3_MOUNTING_HOLE
Changed lines of the file:
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@@
 <part name="U$3" library="blade" deviceset="ISA" device=""/>
 <part name="P+5" library="supply1" library_urn="urn:adsk.eagle:library:371" deviceset="+5V" device=""/>
+<part name="U$11" library="apricot" deviceset="M3_MOUNTING_HOLE" device=""/>
 </parts>
 <sheets>
@@
 <attribute name="VALUE" x="66.04" y="104.14" size="1.778" layer="96" rot="R90"/>
 </instance>
+<instance part="U$11" gate="G$1" x="-30.48" y="142.24" smashed="yes"/>
 </instances>
 <busses>
