File: pcb/macplus/macplus.sch (EAGLE design)
At the start: 11 parts, among them J1 ATX24RH

Commit message: updated with more caps
Parts:
- removed J7: (no value), atx_power_control:CONN_023.5MM-NO_SILK
- removed JP4: (no value), atx_power_control:PINHD-1X4
- added C1: (no value), capacitor-wima:C5/2.5
- added C12, C5, C6, C7: 100nF, clock:CAP0805
- added C3: (no value), adafruit_changed:CPOL-USE3.5-8
- added C4, C8: 47uF, clock:C-USC1210
- JP1: device pinhead:PINHD-1X3 -> appleii:4PIN_FAN
Connections:
- removed net N$7: JP1.2, JP4.3
- net +12V: now also C1.1, C3.+, JP1.2_VCC; no longer JP1.3
- net +5V: no longer JP1.1
- net GND: now also C1.2, C12.1, C3.-, C4.2, C5.1, C6.1, C7.1, C8.2, JP1.1_GND; no longer J7.2, JP4.4
- net N$5: no longer J7.1
- net N$6: now also C12.2, C7.2, C8.1
- net N$8: now also C4.1, C5.2, C6.2
