File: pcb/trs80_model2/trs80_m2.brd (EAGLE design)
At the start: 240 x 148 mm, 2 parts

Commit message: trs80m2 done
Parts:
- added C1, C5, C8: (no value), adafruit_changed:E3,5-8
- added C2, C3, C4, C6, C7: (no value), capacitor-wima:C5B2.5
- added J1: 350760-4, con-amp:350760-4
- added JP1, JP4: (no value), appleii:1X04
- added U$3: TE_3X5, os1:TRS80M2_3X5
- added U$4, U$5, U$6, U$7, U$8: M3_HOLE_PLATED, os1:M3_HOLE_PLATED
- added U$9: CAR_FUSE_HOLDER3IN1, atx_power_control:FUSE_HOLDER_3IN1
- moved U$1 4.00 mm to (27.0, 50.0)
Connections:
- new net +12V: C4.1, C5.+, C6.1, JP1.2, JP4.2, U$1.P$3, U$3.P$14, U$3.P$15
- new net +24V: C7.1, C8.+, U$1.P$4, U$3.P$13
- new net +5V: U$1.P$2, U$9.A0, U$9.A1
- new net -12V: U$1.P$5, U$3.P$1, U$3.P$2
- new net GND: C1.-, C2.2, C3.2, C4.2, C5.-, C6.2, C7.2, C8.-, J1.2, JP1.1, JP4.1, U$1.P$1, U$1.P$6, U$3.P$10, U$3.P$3, U$3.P$4, U$3.P$5, U$3.P$6, U$3.P$7, U$4.P$1, U$5.P$1, U$6.P$1, U$7.P$1, U$8.P$1
- new net LIVE: J1.3, U$1.P$8
- new net N$2: C1.+, C2.1, C3.1, U$3.P$11, U$3.P$12, U$3.P$8, U$3.P$9, U$9.B0, U$9.B1
- new net NEUTRAL: J1.1, U$1.P$7
Routing:
- net +12V: track 0.00 -> 179.4 mm
- net -12V: track 0.00 -> 167.6 mm
- net GND: track 0.00 -> 100.4 mm
- net +5V: track 0.00 -> 71.7 mm
- net +24V: track 0.00 -> 61.4 mm
- net N$2: track 0.00 -> 58.8 mm
- net NEUTRAL: track 0.00 -> 41.3 mm
- net LIVE: track 0.00 -> 31.7 mm
- added copper zone on layer 1, net GND
Other:
- outline, holes or cut-outs redrawn
- board text added: "+24 +12 +12 GND +5 +5 GND +5 +5 GND GND GND -12 -12 GND"
- board text added: "1"
- board text added: "13"
- board text added: "15"
- board text added: "3"
- board text added: "4"
- board text added: "5V 7.5A"
- board text added: "6"
- board text added: "E"
- board text added: "L"
- board text added: "N"
- board text added: "PC FAN"
- board text added: "TRS-80 Model II picoRC.com"
- board text removed: "FAN"
- board text removed: "GND"
- board text removed: "NC"
- board text removed: "ORANGE"
- board text removed: "OS1 POWER"
- board text removed: "RED"
- board text removed: "VCC"
- board text removed: "YELO"

Commit message: isolated pe and gnd
Parts:
- moved U$5 1.00 mm to (232.5, 12.8)
- moved U$8 1.00 mm to (232.5, 141.8)
- moved U$6 0.50 mm to (119.5, 141.8)
Connections:
- new net PE: J1.2, U$1.P$6, U$4.P$1, U$5.P$1, U$6.P$1, U$7.P$1, U$8.P$1
- net GND: no longer J1.2, U$1.P$6, U$4.P$1, U$5.P$1, U$6.P$1, U$7.P$1, U$8.P$1
Routing:
- net PE: track 0.00 -> 524.1 mm
- net GND: track 100.4 -> 105.0 mm
- net +12V: track 179.4 -> 178.0 mm
Other:
- board size 240 x 148 mm -> 239 x 148 mm
- board text added: "+"

Commit message: reworking trs80m2
Parts:
- removed C4, C6, C7: (no value), capacitor-wima:C5B2.5
- removed U$1: TERM_8.25_8P, os1:TERMINAL_8.25MM_8P
- added TP1, TP2, TP3, TP4, TP5, TP6, TP7, TP8: TPPAD1-20Y, testpad:P1-20Y
- added U$10, U$11: M3_HOLE_PLATED, os1:M3_HOLE_PLATED
- moved U$3 122.2 mm to (82.0, 127.0)
- moved C8 97.1 mm to (-12.0, 171.0)
- moved C5 94.3 mm to (-34.0, 145.5)
- moved JP1 52.0 mm to (85.5, 187.5)
- moved JP4 47.4 mm to (61.5, 182.5)
- moved C1 44.1 mm to (45.5, -29.0)
- moved C2 44.1 mm to (37.5, -29.0)
- moved C3 44.1 mm to (33.5, -29.0)
- moved U$9 44.1 mm to (62.0, -29.0)
- moved U$2 33.3 mm to (12.0, 8.00)
- moved J1 8.60 mm to (16.0, 123.5)
Connections:
- net +12V: now also TP6.TP; no longer C4.1, C6.1, U$1.P$3
- net +24V: now also TP5.TP; no longer C7.1, U$1.P$4
- net +5V: now also TP8.TP; no longer U$1.P$2
- net -12V: now also TP4.TP; no longer U$1.P$5
- net GND: now also TP7.TP; no longer C4.2, C6.2, C7.2, U$1.P$1
- net LIVE: now also TP1.TP; no longer U$1.P$8
- net NEUTRAL: now also TP2.TP; no longer U$1.P$7
- net PE: now also TP3.TP; no longer U$1.P$6
Routing:
- net PE: track 524.1 -> 0.00 mm
- net +12V: track 178.0 -> 0.00 mm
- net -12V: track 167.6 -> 0.00 mm
- net GND: track 105.0 -> 0.00 mm
- net +5V: track 71.7 -> 0.00 mm
- net +24V: track 61.4 -> 0.00 mm
- net N$2: track 58.8 -> 0.00 mm
- net NEUTRAL: track 41.3 -> 0.00 mm
- net LIVE: track 31.7 -> 0.00 mm
Other:
- board size 239 x 148 mm -> 239 x 179.2 mm
- board text added: "25 OCT 2025 todo: earth via PSU metal case, make meanwell mounting hole plated through, ensure contact, in guide ask to confirm continuity of earth terminal and chassis, if no continuity use ground lug"
