File: pcb/sirius1/sirius1.brd (EAGLE design)
At the start: 211 x 189.7 mm, 12 parts

Commit message: 396 sirius1
Parts:
- added C1: (no value), adafruit_changed:E3,5-8
- added U$6: 396_SIRIUS1, 396_conn:396_SIRIUS1
- moved JP4 179.0 mm to (5.99, 13.0)
- moved U$5 141.0 mm to (-0.50, 114.0), flipped to the bottom
- moved U$1 140.0 mm to (140.0, 0.00), flipped to the bottom
- moved U$2 140.0 mm to (0.00, 0.00), flipped to the bottom
- moved U$4 140.0 mm to (140.0, 114.0), flipped to the bottom
Connections:
- new net +5V: U$6.P$2, U$6.P$3
- new net -12V: U$6.P$8
- net +12V: now also C1.+, U$6.P$1, U$6.P$7
- net GND: now also C1.-, U$6.P$4, U$6.P$5
Routing:
- net +12V: track 99.1 -> 0.00 mm
- net NEUTRAL: track 13.0 -> 0.00 mm
- net LIVE: track 5.00 -> 0.00 mm
Other:
- board size 211 x 189.7 mm -> 156 x 184.7 mm
- board text removed: "NC"
- board text removed: "NC RED ORANGE YELLOW"
- board text removed: "OG"
- board text removed: "RD"
- board text removed: "YL"
Changed lines of the file:
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@@
 <setting verticaltext="up"/>
 </settings>
-<grid distance="10" unitdist="mm" unit="mm" style="lines" multiple="1" display="no" altdistance="1" altunitdist="mil" altunit="mil"/>
+<grid distance="1" unitdist="mm" unit="mm" style="lines" multiple="1" display="no" altdistance="1" altunitdist="mil" altunit="mil"/>
 <layers>
 <layer number="1" name="Top" color="4" fill="1" visible="yes" active="yes"/>
@@
 <board>
 <plain>
-<wire x1="-23" y1="-9" x2="188" y2="-9" width="0" layer="20"/>
-<wire x1="188" y1="-9" x2="188" y2="120" width="0" layer="20"/>
-<wire x1="188" y1="120" x2="-23" y2="120" width="0" layer="20"/>
-<wire x1="-23" y1="120" x2="-23" y2="-9" width="0" layer="20"/>
-<text x="35.886" y="172.529" size="1.778" layer="25" rot="R90" align="center">YL</text>
-<text x="33.346" y="172.501" size="1.6764" layer="25" rot="R90" align="center">OG</text>
-<text x="30.806" y="172.533" size="1.6764" layer="25" rot="R90" align="center">RD</text>
-<text x="28.266" y="172.422" size="1.6764" layer="25" rot="R90" align="center">NC</text>
-<text x="112.804" y="179.808" size="2.54" layer="25" rot="R270" align="center">GND</text>
+<wire x1="-8" y1="-4" x2="148" y2="-4" width="0" layer="20"/>
+<wire x1="148" y1="-4" x2="148" y2="120" width="0" layer="20"/>
+<wire x1="148" y1="120" x2="-8" y2="120" width="0" layer="20"/>
+<wire x1="-8" y1="120" x2="-8" y2="-4" width="0" layer="20"/>
 <text x="98.164" y="175.858" size="2.54" layer="25" rot="R90" align="center">LIVE</text>
 <text x="80.18" y="177.89" size="2.54" layer="25" rot="R90" align="center">NEUTRAL</text>
-<text x="68.92" y="172.148" size="1.778" layer="25" rot="R90" align="center">YL</text>
-<text x="66.38" y="172.12" size="1.6764" layer="25" rot="R90" align="center">OG</text>
-<text x="63.84" y="172.152" size="1.6764" layer="25" rot="R90" align="center">RD</text>
-<text x="61.3" y="172.041" size="1.6764" layer="25" rot="R90" align="center">NC</text>
 <text x="92.996" y="144.362" size="3.81" layer="25" rot="SR270" align="center">5V
 5A</text>
@@
 <text x="45.676" y="160.402" size="5.08" layer="26" rot="MR270" align="center-left">GND</text>
 <text x="36.676" y="160.402" size="5.08" layer="26" rot="MR270" align="center-left">+5V</text>
-<text x="52.537" y="172.402" size="1.778" layer="25" rot="R90" align="center">YL</text>
-<text x="49.997" y="172.374" size="1.6764" layer="25" rot="R90" align="center">OG</text>
-<text x="47.457" y="172.406" size="1.6764" layer="25" rot="R90" align="center">RD</text>
-<text x="44.917" y="172.295" size="1.6764" layer="25" rot="R90" align="center">NC</text>
-<text x="32.344" y="178.502" size="1.4224" layer="26" distance="80" rot="MR270" align="center-right">NC
-RED
-ORANGE
-YELLOW</text>
-<text x="48.854" y="178.502" size="1.4224" layer="26" distance="80" rot="MR270" align="center-right">NC
-RED
-ORANGE
-YELLOW</text>
-<text x="65.364" y="178.502" size="1.4224" layer="26" distance="80" rot="MR270" align="center-right">NC
-RED
-ORANGE
-YELLOW</text>
-<text x="0.022" y="8.374" size="5.08" layer="25" rot="SR0" align="center">E</text>
+<text x="139.978" y="8.374" size="5.08" layer="25" rot="SR0" align="center">E</text>
 </plain>
 <attributes>
@@
 <attribute name="VALUE" x="142.548" y="130.076" size="1.27" layer="27" ratio="10"/>
 </element>
-<element name="JP4" library="appleii" package="1X04" value="" x="110.99" y="157.98" smashed="yes" rot="R270"/>
+<element name="JP4" library="appleii" package="1X04" value="" x="5.99" y="12.98" smashed="yes" rot="R270"/>
 <element name="U$14" library="blade" package="2.8FLAG" value="28FLAG" x="84.74" y="175.73" smashed="yes" rot="R90"/>
 <element name="U$3" library="blade" package="2.8FLAG" value="28FLAG" x="93.74" y="175.73" smashed="yes" rot="R90"/>
@@
 <attribute name="VALUE" x="-36.323" y="143.0374" size="1.27" layer="27" ratio="10" rot="R270"/>
 </element>
-<element name="U$1" library="os1" package="M3_HOLE_PLATED" value="M3_HOLE_PLATEDM3" x="0" y="0" smashed="yes"/>
-<element name="U$2" library="os1" package="M2.5_HOLE_PLATED" value="M3_HOLE_PLATEDM2,5" x="140" y="0" smashed="yes"/>
-<element name="U$4" library="os1" package="M2.5_HOLE_PLATED" value="M3_HOLE_PLATEDM2,5" x="0" y="114" smashed="yes"/>
-<element name="U$5" library="os1" package="M2.5_HOLE_PLATED" value="M3_HOLE_PLATEDM2,5" x="140.5" y="114" smashed="yes"/>
+<element name="U$1" library="os1" package="M3_HOLE_PLATED" value="M3_HOLE_PLATEDM3" x="140" y="0" smashed="yes" rot="MR0"/>
+<element name="U$2" library="os1" package="M2.5_HOLE_PLATED" value="M3_HOLE_PLATEDM2,5" x="0" y="0" smashed="yes" rot="MR0"/>
+<element name="U$4" library="os1" package="M2.5_HOLE_PLATED" value="M3_HOLE_PLATEDM2,5" x="140" y="114" smashed="yes" rot="MR0"/>
+<element name="U$5" library="os1" package="M2.5_HOLE_PLATED" value="M3_HOLE_PLATEDM2,5" x="-0.5" y="114" smashed="yes" rot="MR0"/>
+<element name="C1" library="adafruit_changed" package="E3,5-8" value="" x="99" y="95" smashed="yes">
+<attribute name="NAME" x="102.302" y="97.794" size="1.27" layer="25" ratio="10"/>
+<attribute name="VALUE" x="96.714" y="91.952" size="1.27" layer="27" ratio="10"/>
+</element>
+<element name="U$6" library="396_conn" package="396_SIRIUS1" value="396_SIRIUS1" x="119" y="112" smashed="yes"/>
 </elements>
 <signals>
@@
 <contactref element="C5" pad="-"/>
 <polygon width="0.254" layer="1" isolate="0.8128">
-<vertex x="-11.5" y="116"/>
-<vertex x="-11.5" y="-11"/>
-<vertex x="185" y="-11"/>
-<vertex x="185" y="116"/>
+<vertex x="-81.5" y="186"/>
+<vertex x="-81.5" y="-41"/>
+<vertex x="275" y="-41"/>
+<vertex x="275" y="186"/>
 </polygon>
 <contactref element="JP4" pad="1"/>
-<wire x1="147.12" y1="132.87" x2="167.44" y2="133.83" width="0" layer="19" extent="1-1"/>
-<wire x1="113.9327625" y1="155.217234375" x2="147.12" y2="132.87" width="0" layer="19" extent="1-1"/>
-<wire x1="110.99" y1="161.79" x2="113.9327625" y2="155.217234375" width="0" layer="19" extent="1-1"/>
+<contactref element="C1" pad="-"/>
+<contactref element="U$6" pad="P$4"/>
+<contactref element="U$6" pad="P$5"/>
+<wire x1="120.98" y1="112" x2="147.12" y2="132.87" width="0" layer="19" extent="1-1"/>
 </signal>
 <signal name="+12V">
 <contactref element="JP4" pad="2"/>
-<wire x1="31" y1="170.73" x2="30.92" y2="170.81" width="1.27" layer="16"/>
-<wire x1="67.2" y1="170.73" x2="69.99" y2="167.94" width="1.27" layer="16"/>
-<wire x1="31" y1="170.73" x2="67.2" y2="170.73" width="1.27" layer="16"/>
-<wire x1="69.99" y1="167.94" x2="69.99" y2="159.68" width="1.27" layer="16"/>
-<wire x1="69.99" y1="159.68" x2="81.72" y2="147.95" width="1.27" layer="16"/>
-<wire x1="81.72" y1="147.95" x2="97.468" y2="147.95" width="1.27" layer="16"/>
-<wire x1="97.468" y1="147.95" x2="108.768" y2="159.25" width="1.27" layer="16"/>
-<wire x1="108.768" y1="159.25" x2="110.99" y2="159.25" width="1.27" layer="16"/>
+<contactref element="U$6" pad="P$7"/>
+<contactref element="C1" pad="+"/>
+<contactref element="U$6" pad="P$1"/>
+<wire x1="105.14" y1="112" x2="128.9" y2="112" width="0" layer="19" extent="1-1"/>
+<wire x1="97.222" y1="95" x2="105.14" y2="112" width="0" layer="19" extent="1-1"/>
+<wire x1="5.99" y1="14.25" x2="97.222" y2="95" width="0" layer="19" extent="1-1"/>
 </signal>
 <signal name="NEUTRAL">
 <contactref element="U$14" pad="P$2"/>
 <contactref element="U$14" pad="P$1"/>
-<wire x1="84.74" y1="178.23" x2="84.74" y2="173.23" width="2.54" layer="16"/>
-<wire x1="84.74" y1="173.23" x2="84.74" y2="165.23" width="2.54" layer="16"/>
+<wire x1="84.74" y1="173.23" x2="84.74" y2="178.23" width="0" layer="19" extent="1-1"/>
 </signal>
 <signal name="LIVE">
 <contactref element="U$3" pad="P$2"/>
 <contactref element="U$3" pad="P$1"/>
-<wire x1="93.74" y1="178.23" x2="93.74" y2="173.23" width="2.54" layer="16"/>
+<wire x1="93.74" y1="173.23" x2="93.74" y2="178.23" width="0" layer="19" extent="1-1"/>
+</signal>
+<signal name="+5V">
+<contactref element="U$6" pad="P$2"/>
+<contactref element="U$6" pad="P$3"/>
+<wire x1="109.1" y1="112" x2="113.06" y2="112" width="0" layer="19" extent="1-1"/>
+</signal>
+<signal name="-12V">
+<contactref element="U$6" pad="P$8"/>
 </signal>
 </signals>

Commit message: sirius 1 done
Parts:
- removed R2: (no value), adafruit_changed:0411/15
- removed U$14, U$3: 28FLAG, blade:2.8FLAG
- added C2: (no value), adafruit_changed:E3,5-8
- added C27, C7: 47uF, clock:C1210
- added C3: 470uF, rcl:SMC_D
- added U$10: INDUCTOR_PTH_8MM, 396_conn:INDUCTOR_PTH_8MM
- added U$7: MEANWELL_RT65, os1:MEANWELL_RT65
- added U$8: CAR_FUSE_HOLDER3IN1, atx_power_control:FUSE_HOLDER_3IN1
- moved U$9 155.4 mm to (135.0, 93.0), flipped to the top, turned to 0 degrees
- moved C4 69.6 mm to (98.5, 113.0), turned to 270 degrees
- moved C5 61.0 mm to (70.0, 113.0), turned to 270 degrees
- moved C6 53.9 mm to (94.5, 113.0), turned to 270 degrees
- moved C1 26.9 mm to (79.0, 113.0), turned to 270 degrees
- moved JP4 15.2 mm to (12.0, -1.01), turned to 0 degrees
- moved U$6 1.41 mm to (118.0, 113.0)
Connections:
- removed net LIVE: U$3.P$1, U$3.P$2
- removed net NEUTRAL: U$14.P$1, U$14.P$2
- new net N$1: C1.+, C2.+, C4.1, C5.+, C6.1, U$10.P$2, U$6.P$1
- new net N$2: U$7.+5V, U$8.B0, U$8.B1
- new net N$4: U$7.+12V, U$9.B0, U$9.B1
- net +12V: now also U$10.P$1, U$9.A0, U$9.A1; no longer C1.+, U$6.P$1
- net +5V: now also C27.1, C3.+, C7.1, U$8.A0, U$8.A1
- net -12V: now also U$7.-12V
- net GND: now also C2.-, C27.2, C3.-, C7.2, U$1.P$1, U$2.P$1, U$4.P$1, U$5.P$1, U$7.EARTH, U$7.GND, U$7.GND2, U$7.GND3
Routing:
- net +12V: track 0.00 -> 251.7 mm
- net -12V: track 0.00 -> 59.8 mm
- net N$1: track 0.00 -> 51.4 mm
- net +5V: track 0.00 -> 40.5 mm
- net N$4: track 0.00 -> 34.4 mm
- net N$2: track 0.00 -> 24.8 mm
- net GND: track 0.00 -> 20.2 mm
Other:
- board size 156 x 184.7 mm -> 154 x 123 mm
- board text added: "+"
- board text added: "+12"
- board text added: "+12 CRT"
- board text added: "+5"
- board text added: "-12"
- board text added: "-12V"
- board text added: "12V 3A"
- board text added: "Sirius 1 / Victor 9000"
- board text added: "dekuNukem 2026"
- board text removed: "LIVE"
- board text removed: "NEUTRAL"
- board text removed: "Osborne 1 picoRC.com"
