File: pcb/sirius1/sirius1.sch (EAGLE design)
At the start: 12 parts

Commit message: 396 sirius1
Parts:
- added C1: (no value), adafruit_changed:CPOL-USE3.5-8
- added U$6: 396_SIRIUS1, 396_conn:396_SIRIUS1
Connections:
- new net +5V: U$6.+5V1, U$6.+5V2
- new net -12V: U$6.-12V
- net +12V: now also C1.+, U$6.+12V1, U$6.+12V2
- net GND: now also C1.-, U$6.GND1, U$6.GND2
Changed lines of the file:
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@@
 <part name="U$4" library="os1" deviceset="M3_HOLE_PLATED" device="M2,5"/>
 <part name="U$5" library="os1" deviceset="M3_HOLE_PLATED" device="M2,5"/>
+<part name="P+1" library="supply1" library_urn="urn:adsk.eagle:library:371" deviceset="+12V" device=""/>
+<part name="P+4" library="supply1" library_urn="urn:adsk.eagle:library:371" deviceset="+5V" device=""/>
+<part name="P-1" library="supply1" library_urn="urn:adsk.eagle:library:371" deviceset="-12V" device=""/>
+<part name="GND1" library="supply1" library_urn="urn:adsk.eagle:library:371" deviceset="GND" device=""/>
+<part name="P+5" library="supply1" library_urn="urn:adsk.eagle:library:371" deviceset="+12V" device=""/>
+<part name="C1" library="adafruit_changed" deviceset="CPOL-US" device="E3.5-8"/>
+<part name="GND2" library="supply1" library_urn="urn:adsk.eagle:library:371" deviceset="GND" device=""/>
+<part name="U$6" library="396_conn" deviceset="396_SIRIUS1" device=""/>
 </parts>
 <sheets>
@@
 <instance part="U$4" gate="G$1" x="43.18" y="93.98" smashed="yes"/>
 <instance part="U$5" gate="G$1" x="43.18" y="86.36" smashed="yes"/>
+<instance part="P+1" gate="1" x="91.44" y="86.36" smashed="yes" rot="MR0">
+<attribute name="VALUE" x="93.98" y="81.28" size="1.778" layer="96" rot="MR90"/>
+</instance>
+<instance part="P+4" gate="1" x="63.5" y="60.96" smashed="yes" rot="MR0">
+<attribute name="VALUE" x="63.5" y="63.5" size="1.778" layer="96" rot="MR90"/>
+</instance>
+<instance part="P-1" gate="1" x="76.2" y="35.56" smashed="yes">
+<attribute name="VALUE" x="73.66" y="33.02" size="1.778" layer="96" rot="R90"/>
+</instance>
+<instance part="GND1" gate="1" x="111.76" y="48.26" smashed="yes" rot="MR0">
+<attribute name="VALUE" x="114.3" y="45.72" size="1.778" layer="96" rot="MR0"/>
+</instance>
+<instance part="P+5" gate="1" x="66.04" y="45.72" smashed="yes" rot="MR0">
+<attribute name="VALUE" x="68.58" y="40.64" size="1.778" layer="96" rot="MR90"/>
+</instance>
+<instance part="C1" gate="G$1" x="91.44" y="76.2" smashed="yes">
+<attribute name="NAME" x="92.456" y="76.835" size="1.778" layer="95"/>
+<attribute name="VALUE" x="92.456" y="72.009" size="1.778" layer="96"/>
+</instance>
+<instance part="GND2" gate="1" x="91.44" y="66.04" smashed="yes" rot="MR0">
+<attribute name="VALUE" x="93.98" y="63.5" size="1.778" layer="96" rot="MR0"/>
+</instance>
+<instance part="U$6" gate="G$1" x="96.52" y="50.8" smashed="yes"/>
 </instances>
 <busses>
@@
 <wire x1="160.02" y1="27.94" x2="172.72" y2="27.94" width="0.1524" layer="91"/>
 </segment>
+<segment>
+<pinref part="GND1" gate="1" pin="GND"/>
+<wire x1="83.82" y1="50.8" x2="88.9" y2="50.8" width="0.1524" layer="91"/>
+<wire x1="83.82" y1="48.26" x2="83.82" y2="50.8" width="0.1524" layer="91"/>
+<wire x1="88.9" y1="48.26" x2="83.82" y2="48.26" width="0.1524" layer="91"/>
+<pinref part="U$6" gate="G$1" pin="GND1"/>
+<pinref part="U$6" gate="G$1" pin="GND2"/>
+</segment>
+<segment>
+<pinref part="GND2" gate="1" pin="GND"/>
+<pinref part="C1" gate="G$1" pin="-"/>
+<wire x1="91.44" y1="68.58" x2="91.44" y2="71.12" width="0.1524" layer="91"/>
+</segment>
 </net>
 <net name="+12V" class="0">
@@
 <pinref part="JP4" gate="A" pin="2_VCC"/>
 <wire x1="172.72" y1="22.86" x2="200.66" y2="22.86" width="0.1524" layer="91"/>
+</segment>
+<segment>
+<pinref part="P+5" gate="1" pin="+12V"/>
+<wire x1="88.9" y1="43.18" x2="66.04" y2="43.18" width="0.1524" layer="91"/>
+<pinref part="U$6" gate="G$1" pin="+12V1"/>
+</segment>
+<segment>
+<pinref part="C1" gate="G$1" pin="+"/>
+<pinref part="P+1" gate="1" pin="+12V"/>
+<wire x1="91.44" y1="83.82" x2="91.44" y2="81.28" width="0.1524" layer="91"/>
+<wire x1="91.44" y1="81.28" x2="91.44" y2="78.74" width="0.1524" layer="91"/>
+<wire x1="91.44" y1="81.28" x2="71.12" y2="81.28" width="0.1524" layer="91"/>
+<junction x="91.44" y="81.28"/>
+<pinref part="U$6" gate="G$1" pin="+12V2"/>
+<wire x1="71.12" y1="81.28" x2="71.12" y2="58.42" width="0.1524" layer="91"/>
+<wire x1="71.12" y1="58.42" x2="88.9" y2="58.42" width="0.1524" layer="91"/>
 </segment>
 </net>
@@
 </segment>
 </net>
+<net name="+5V" class="0">
+<segment>
+<pinref part="P+4" gate="1" pin="+5V"/>
+<wire x1="63.5" y1="58.42" x2="63.5" y2="55.88" width="0.1524" layer="91"/>
+<wire x1="63.5" y1="55.88" x2="88.9" y2="55.88" width="0.1524" layer="91"/>
+<wire x1="88.9" y1="53.34" x2="63.5" y2="53.34" width="0.1524" layer="91"/>
+<wire x1="63.5" y1="53.34" x2="63.5" y2="55.88" width="0.1524" layer="91"/>
+<junction x="63.5" y="55.88"/>
+<pinref part="U$6" gate="G$1" pin="+5V1"/>
+<pinref part="U$6" gate="G$1" pin="+5V2"/>
+</segment>
+</net>
+<net name="-12V" class="0">
+<segment>
+<pinref part="P-1" gate="1" pin="-12V"/>
+<wire x1="76.2" y1="38.1" x2="76.2" y2="40.64" width="0.1524" layer="91"/>
+<wire x1="76.2" y1="40.64" x2="88.9" y2="40.64" width="0.1524" layer="91"/>
+<pinref part="U$6" gate="G$1" pin="-12V"/>
+</segment>
+</net>

Commit message: sirius 1 done
Parts:
- removed R2: (no value), adafruit_changed:R-US_0411/15
- removed U$14, U$3: 28FLAG, blade:28FLAG
- added C2: (no value), adafruit_changed:CPOL-USE3.5-8
- added C27, C7: 47uF, clock:C-USC1210
- added C3: 470uF, rcl:CPOL-USSMCD
- added U$10: INDUCTOR_PTH_8MM, 396_conn:INDUCTOR_PTH_8MM
- added U$7: MEANWELL_RT65, os1:MEANWELL_RT65
- added U$8: CAR_FUSE_HOLDER3IN1, atx_power_control:CAR_FUSE_HOLDER3IN1
Connections:
- removed net LIVE: U$3.P$1
- removed net NEUTRAL: U$14.P$1
- new net N$1: C1.+, C2.+, C4.1, C5.+, C6.1, U$10.P$2, U$6.+12V_CRT
- new net N$2: U$7.5V, U$8.B0, U$8.B1
- new net N$4: U$7.12V, U$9.B0, U$9.B1
- net +12V: now also U$10.P$1, U$6.+12V, U$9.A0, U$9.A1; no longer C1.+, U$6.+12V1, U$6.+12V2
- net +5V: now also C27.1, C3.+, C7.1, U$8.A0, U$8.A1
- net -12V: now also U$7.-12V
- net GND: now also C2.-, C27.2, C3.-, C7.2, U$1.P$1, U$2.P$1, U$4.P$1, U$5.P$1, U$7.EARTH, U$7.GND
Other:
- moved on the sheet: C1, C4, C5, C6
