File: pcb/sirius1/sirius1.sch (EAGLE design)
At the start: 18 parts

Commit message: m3 holes, moved PSU down slighly, thicker 12V trace
Parts:
- U$2, U$4, U$5: value M3_HOLE_PLATEDM2,5 -> M3_HOLE_PLATEDM3; device os1:M3_HOLE_PLATEDM2,5 -> os1:M3_HOLE_PLATEDM3
Changed lines of the file:
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@@
 <part name="P+10" library="supply1" library_urn="urn:adsk.eagle:library:371" deviceset="+12V" device=""/>
 <part name="U$1" library="os1" deviceset="M3_HOLE_PLATED" device="M3"/>
-<part name="U$2" library="os1" deviceset="M3_HOLE_PLATED" device="M2,5"/>
-<part name="U$4" library="os1" deviceset="M3_HOLE_PLATED" device="M2,5"/>
-<part name="U$5" library="os1" deviceset="M3_HOLE_PLATED" device="M2,5"/>
+<part name="U$2" library="os1" deviceset="M3_HOLE_PLATED" device="M3" value="M3_HOLE_PLATEDM3"/>
+<part name="U$4" library="os1" deviceset="M3_HOLE_PLATED" device="M3" value="M3_HOLE_PLATEDM3"/>
+<part name="U$5" library="os1" deviceset="M3_HOLE_PLATED" device="M3" value="M3_HOLE_PLATEDM3"/>
 <part name="P+1" library="supply1" library_urn="urn:adsk.eagle:library:371" deviceset="+12V" device=""/>
 <part name="P+4" library="supply1" library_urn="urn:adsk.eagle:library:371" deviceset="+5V" device=""/>
