File: pcb/os1_mw/osborne1.brd (EAGLE design)
At the start: 160 x 100 mm, 2 parts

Commit message: added docs
Parts:
- added JP1, JP2, JP3: (no value), pinhead:1X04/90
- added U$3: VH396_3P, 396_conn:396_3P
- moved U$2 5.10 mm to (138.0, 79.0)
- moved U$1 1.00 mm to (123.0, 100.0)
Changed lines of the file:
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@@
 </autorouter>
 <elements>
-<element name="U$1" library="apricot" package="MEANWELL_RD50" value="MEANWELL_RD50" x="123" y="99" smashed="yes" rot="R180"/>
-<element name="U$2" library="os1" package="TERMINAL9500" value="TERM9.5" x="143" y="78" smashed="yes" rot="R270"/>
+<element name="U$1" library="apricot" package="MEANWELL_RD50" value="MEANWELL_RD50" x="123" y="100" smashed="yes" rot="R180"/>
+<element name="U$2" library="os1" package="TERMINAL9500" value="TERM9.5" x="138" y="79" smashed="yes" rot="R270"/>
+<element name="U$3" library="396_conn" package="396_3P" value="VH396_3P" x="151" y="22" smashed="yes" rot="R90"/>
+<element name="JP2" library="pinhead" library_urn="urn:adsk.eagle:library:325" package="1X04/90" package3d_urn="urn:adsk.eagle:package:22404/2" value="" x="153" y="45" smashed="yes" rot="R270">
+<attribute name="NAME" x="149.19" y="50.715" size="1.27" layer="25" ratio="10"/>
+<attribute name="POPULARITY" value="9" x="153" y="45" size="1.778" layer="27" rot="R270" display="off"/>
+<attribute name="VALUE" x="148.555" y="38.015" size="1.27" layer="27"/>
+</element>
+<element name="JP1" library="pinhead" library_urn="urn:adsk.eagle:library:325" package="1X04/90" package3d_urn="urn:adsk.eagle:package:22404/2" value="" x="153" y="75" smashed="yes" rot="R270">
+<attribute name="NAME" x="149.19" y="80.715" size="1.27" layer="25" ratio="10"/>
+<attribute name="POPULARITY" value="9" x="153" y="75" size="1.778" layer="27" rot="R270" display="off"/>
+<attribute name="VALUE" x="148.555" y="68.015" size="1.27" layer="27"/>
+</element>
+<element name="JP3" library="pinhead" library_urn="urn:adsk.eagle:library:325" package="1X04/90" package3d_urn="urn:adsk.eagle:package:22404/2" value="" x="153" y="60" smashed="yes" rot="R270">
+<attribute name="NAME" x="149.19" y="65.715" size="1.27" layer="25" ratio="10"/>
+<attribute name="POPULARITY" value="9" x="153" y="60" size="1.778" layer="27" rot="R270" display="off"/>
+<attribute name="VALUE" x="148.555" y="53.015" size="1.27" layer="27"/>
+</element>
 </elements>
 <signals>
@@
 which will not be processed correctly with this version.
 </note>
+<note version="8.2" severity="warning">
+Since Version 8.2, EAGLE supports online libraries. The ids
+of those online libraries will not be understood (or retained)
+with this version.
+</note>
+<note version="8.3" severity="warning">
+Since Version 8.3, EAGLE supports URNs for individual library
+assets (packages, symbols, and devices). The URNs of those assets
+will not be understood (or retained) with this version.
+</note>
+<note version="8.3" severity="warning">
+Since Version 8.3, EAGLE supports the association of 3D packages
+with devices in libraries, schematics, and board files. Those 3D
+packages will not be understood (or retained) with this version.
+</note>
 </compatibility>

Commit message: new os1 pcb done
Parts:
- removed U$3: VH396_3P, 396_conn:396_3P
- added C4, C6: (no value), capacitor-wima:C5B2.5
- added C5: (no value), adafruit_changed:E3,5-8
- added JP4: (no value), appleii:1X04
- added TP1, TP2: PTR1PAD1-17, testpad:P1-17
- added U$4, U$5, U$6, U$8: M3_HOLE_PLATED, os1:M3_HOLE_PLATED
- added U$7: 396_2P_LIVE, 396_conn:396_2P_LIVE
- added U$9: CAR_FUSE_HOLDER3IN1, atx_power_control:FUSE_HOLDER_3IN1
- moved U$1 2.00 mm to (123.0, 102.0)
- moved U$2 1.00 mm to (138.0, 78.0)
Connections:
- new net +12V: JP1.2, JP2.2, JP3.2, JP4.2, U$2.P$3
- new net +5V: C4.1, C5.+, C6.1, JP1.4, JP2.4, JP3.4, U$9.A0, U$9.A1
- new net GND: C4.2, C5.-, C6.2, JP1.3, JP2.3, JP3.3, JP4.1, TP1.TP, TP2.TP, U$2.P$2, U$2.P$4, U$2.P$5, U$4.P$1, U$5.P$1, U$6.P$1, U$8.P$1
- new net LIVE: U$2.P$7, U$7.P$1
- new net N$2: U$2.P$1, U$9.B0, U$9.B1
- new net NEUTRAL: U$2.P$6, U$7.P$2
Routing:
- net +5V: track 0.00 -> 230.7 mm
- net +12V: track 0.00 -> 156.5 mm
- net N$2: track 0.00 -> 133.1 mm
- net GND: track 0.00 -> 90.8 mm
- net NEUTRAL: track 0.00 -> 16.0 mm
- net LIVE: track 0.00 -> 15.3 mm
- added copper zone on layer 1, net GND
Other:
- outline, holes or cut-outs redrawn
- board text added: "5V 5A"
- board text added: "LIVE"
- board text added: "NEUTRAL"
- board text added: "OG"
- board text added: "Osborne 1 picoRC.com"
- board text added: "PC FAN"
- board text added: "RD"
- board text added: "YL"
- board text removed: "FAN"
- board text removed: "ORANGE"
- board text removed: "OS1 POWER"
- board text removed: "RED"
- board text removed: "VCC"
- board text removed: "YELO"

Commit message: isolated pe and gnd
Parts:
- moved U$9 1.02 mm to (8.02, 86.0)
Connections:
- new net PE: U$2.P$5, U$4.P$1, U$5.P$1, U$6.P$1, U$8.P$1
- net GND: no longer U$2.P$5, U$4.P$1, U$5.P$1, U$6.P$1, U$8.P$1
Routing:
- net PE: track 0.00 -> 354.3 mm
- net GND: track 90.8 -> 44.8 mm
- net N$2: track 133.1 -> 132.1 mm
- net +5V: track 230.7 -> 229.7 mm
Other:
- board text added: "NOT FINISHED YET! CHECK REAL HARDWARE! IS GND AND PE CONNECTED?"
Changed lines of the file:
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@@
 <setting verticaltext="up"/>
 </settings>
-<grid distance="0.25" unitdist="mm" unit="mm" style="lines" multiple="1" display="no" altdistance="1" altunitdist="mil" altunit="mil"/>
+<grid distance="10" unitdist="mil" unit="mil" style="lines" multiple="1" display="no" altdistance="1" altunitdist="mil" altunit="mil"/>
 <layers>
 <layer number="1" name="Top" color="4" fill="1" visible="yes" active="yes"/>
@@
 <vertex x="108" y="32.25"/>
 </polygon>
-<text x="13.436" y="82.422" size="3.81" layer="25" rot="R90" align="center">5V 5A</text>
+<text x="8.002" y="72.364" size="3.81" layer="25" rot="R180" align="center">5V 5A</text>
 <text x="11.064" y="37.328" size="5.08" layer="25" rot="R270" align="center">Osborne 1
 picoRC.com</text>
 <text x="130.328" y="9.186" size="2.54" layer="25" rot="R180" align="center">PC FAN</text>
+<polygon width="1.27" layer="41">
+<vertex x="20.25" y="108.75"/>
+<vertex x="127" y="108.75"/>
+<vertex x="127" y="-5.5"/>
+<vertex x="20.25" y="-5.5"/>
+</polygon>
+<text x="204.992" y="57.232" size="2.54" layer="25" align="center">NOT FINISHED YET!
+CHECK REAL HARDWARE!
+IS GND AND PE CONNECTED?</text>
 </plain>
 <attributes>
@@
 <element name="U$6" library="os1" package="M3_HOLE_PLATED" value="M3_HOLE_PLATED" x="19" y="90" smashed="yes"/>
 <element name="U$8" library="os1" package="M3_HOLE_PLATED" value="M3_HOLE_PLATED" x="141" y="90" smashed="yes"/>
-<element name="U$9" library="atx_power_control" package="FUSE_HOLDER_3IN1" value="CAR_FUSE_HOLDER3IN1" x="7" y="86" smashed="yes" rot="R270"/>
+<element name="U$9" library="atx_power_control" package="FUSE_HOLDER_3IN1" value="CAR_FUSE_HOLDER3IN1" x="8.016" y="86" smashed="yes" rot="R270"/>
 <element name="C4" library="capacitor-wima" library_urn="urn:adsk.eagle:library:116" package="C5B2.5" package3d_urn="urn:adsk.eagle:package:5426/1" value="" x="152" y="94" smashed="yes">
 <attribute name="NAME" x="149.968" y="95.524" size="1.27" layer="25" ratio="10"/>
@@
 <signals>
 <signal name="GND">
-<contactref element="U$8" pad="P$1"/>
-<contactref element="U$6" pad="P$1"/>
-<contactref element="U$4" pad="P$1"/>
-<contactref element="U$5" pad="P$1"/>
 <contactref element="C6" pad="2"/>
 <contactref element="C4" pad="2"/>
 <contactref element="C5" pad="-"/>
-<contactref element="U$2" pad="P$5"/>
 <contactref element="U$2" pad="P$4"/>
 <contactref element="U$2" pad="P$2"/>
@@
 <contactref element="JP3" pad="3"/>
 <contactref element="JP2" pad="3"/>
-<polygon width="0.254" layer="1" isolate="0.8128" thermals="no">
+<polygon width="0.254" layer="1" isolate="0.8128">
 <vertex x="-11.5" y="116"/>
 <vertex x="-11.5" y="-11"/>
@@
 <wire x1="144.25" y1="73.73" x2="144.25" y2="58.73" width="1.27" layer="1"/>
 <wire x1="144.25" y1="58.73" x2="144.25" y2="43.73" width="1.27" layer="1"/>
-<wire x1="149.19" y1="43.73" x2="154.5" y2="43.73" width="1.27" layer="1"/>
-<wire x1="154.5" y1="43.73" x2="154.5" y2="58.73" width="1.27" layer="1"/>
-<wire x1="154.5" y1="58.73" x2="154.5" y2="73.75" width="1.27" layer="1"/>
-<wire x1="154.5" y1="73.75" x2="149.19" y2="73.75" width="1.27" layer="1"/>
 <wire x1="149.19" y1="73.75" x2="149.19" y2="73.73" width="1.27" layer="1"/>
 <wire x1="149.19" y1="58.73" x2="144.25" y2="58.73" width="1.27" layer="1"/>
-<wire x1="149.19" y1="58.73" x2="154.5" y2="58.73" width="1.27" layer="1"/>
 <contactref element="JP4" pad="1"/>
+<wire x1="149.19" y1="43.73" x2="150.5" y2="5" width="0" layer="19" extent="1-1"/>
 </signal>
 <signal name="+12V">
@@
 <contactref element="U$9" pad="B0"/>
 <contactref element="U$2" pad="P$1"/>
-<wire x1="138" y1="78" x2="9.7" y2="78" width="2.54" layer="16"/>
-<wire x1="9.7" y1="78" x2="8.75" y2="78.95" width="2.54" layer="16"/>
-<wire x1="8.75" y1="78.95" x2="5.25" y2="78.95" width="2.54" layer="16"/>
+<wire x1="138" y1="78" x2="10.716" y2="78" width="2.54" layer="16"/>
+<wire x1="10.716" y1="78" x2="9.766" y2="78.95" width="2.54" layer="16"/>
+<wire x1="9.766" y1="78.95" x2="6.266" y2="78.95" width="2.54" layer="16"/>
 </signal>
 <signal name="+5V">
@@
 <contactref element="JP1" pad="4"/>
 <contactref element="JP2" pad="4"/>
-<wire x1="5.25" y1="93.05" x2="8.75" y2="93.05" width="2.54" layer="16"/>
-<wire x1="8.75" y1="93.05" x2="13.7" y2="98" width="2.54" layer="16"/>
-<wire x1="13.7" y1="98" x2="103" y2="98" width="2.54" layer="16"/>
+<wire x1="6.266" y1="93.05" x2="9.766" y2="93.05" width="2.54" layer="16"/>
+<wire x1="9.766" y1="93.05" x2="14.716" y2="98" width="2.54" layer="16"/>
+<wire x1="14.716" y1="98" x2="103" y2="98" width="2.54" layer="16"/>
 <wire x1="103" y1="98" x2="112" y2="89" width="2.54" layer="16"/>
 <wire x1="146.46" y1="97" x2="149.46" y2="94" width="2.54" layer="16"/>
@@
 <wire x1="150.06" y1="41.19" x2="150.5" y2="40.75" width="1.016" layer="16"/>
 </signal>
+<signal name="PE">
+<contactref element="U$2" pad="P$5"/>
+<contactref element="U$8" pad="P$1"/>
+<contactref element="U$6" pad="P$1"/>
+<contactref element="U$4" pad="P$1"/>
+<contactref element="U$5" pad="P$1"/>
+<wire x1="141" y1="90" x2="134.566" y2="83.566" width="1.27" layer="16"/>
+<wire x1="25.434" y1="83.566" x2="19" y2="90" width="1.27" layer="16"/>
+<wire x1="134.566" y1="83.566" x2="25.434" y2="83.566" width="1.27" layer="16"/>
+<wire x1="19" y1="90" x2="16.63" y2="87.63" width="1.27" layer="16"/>
+<wire x1="16.63" y1="87.63" x2="5.08" y2="87.63" width="1.27" layer="16"/>
+<wire x1="5.08" y1="87.63" x2="2.032" y2="84.582" width="1.27" layer="16"/>
+<wire x1="2.032" y1="26.968" x2="19" y2="10" width="1.27" layer="16"/>
+<wire x1="2.032" y1="84.582" x2="2.032" y2="26.968" width="1.27" layer="16"/>
+<wire x1="138" y1="40" x2="132.71" y2="40" width="1.27" layer="16"/>
+<wire x1="132.71" y1="40" x2="127" y2="34.29" width="1.27" layer="16"/>
+<wire x1="127" y1="34.29" x2="127" y2="21.968" width="1.27" layer="16"/>
+<wire x1="138.968" y1="10" x2="141" y2="10" width="1.27" layer="16"/>
+<wire x1="138.968" y1="10" x2="127" y2="21.968" width="1.27" layer="16"/>
+<wire x1="141" y1="90" x2="146.926" y2="84.074" width="1.27" layer="1"/>
+<wire x1="156.972" y1="38.862" x2="155.702" y2="37.592" width="1.27" layer="1"/>
+<wire x1="155.702" y1="37.592" x2="140.408" y2="37.592" width="1.27" layer="1"/>
+<wire x1="140.408" y1="37.592" x2="138" y2="40" width="1.27" layer="1"/>
+<wire x1="146.926" y1="84.074" x2="152.4" y2="84.074" width="1.27" layer="1"/>
+<wire x1="152.4" y1="84.074" x2="156.972" y2="79.502" width="1.27" layer="1"/>
+<wire x1="156.972" y1="79.502" x2="156.972" y2="38.862" width="1.27" layer="1"/>
+</signal>
 </signals>

Commit message: adjust pcb
Parts:
- removed U$7: 396_2P_LIVE, 396_conn:396_2P_LIVE
- added R1, R2: (no value), adafruit_changed:0411/15
- added U$14, U$3: 28FLAG, blade:2.8FLAG
- moved JP2 19.0 mm to (141.0, 59.7)
- moved JP3 17.3 mm to (141.0, 72.4)
- moved JP1 15.7 mm to (141.0, 85.1)
- moved C6 13.3 mm to (139.5, 93.5)
- moved U$9 13.2 mm to (6.02, 73.0)
- moved C4 12.9 mm to (139.5, 97.0)
- moved C5 12.0 mm to (119.0, 93.0)
- moved JP4 12.0 mm to (119.2, 3.75)
- moved TP1 12.0 mm to (138.5, 5.00)
- moved TP2 12.0 mm to (143.5, 5.00)
- moved U$1 12.0 mm to (111.0, 102.0)
- moved U$2 12.0 mm to (126.0, 78.0)
- moved U$4 12.0 mm to (7.00, 10.0)
- moved U$5 12.0 mm to (129.0, 10.0)
- moved U$6 12.0 mm to (7.00, 90.0)
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Connections:
- removed net PE: U$2.P$5, U$4.P$1, U$5.P$1, U$6.P$1, U$8.P$1
- net +12V: now also R1.2
- net GND: now also R1.1, R2.2, U$2.P$5, U$4.P$1, U$5.P$1, U$6.P$1, U$8.P$1
- net LIVE: now also U$3.P$1, U$3.P$2; no longer U$7.P$1
- net N$2: now also R2.1
- net NEUTRAL: now also U$14.P$1, U$14.P$2; no longer U$7.P$2
Routing:
- net PE: track 354.3 -> 0.00 mm
- net GND: track 44.8 -> 0.00 mm
- net +5V: track 229.7 -> 201.9 mm
- net +12V: track 156.5 -> 178.7 mm
- net N$2: track 132.1 -> 138.2 mm
- net NEUTRAL: track 16.0 -> 13.7 mm
- net LIVE: track 15.3 -> 13.5 mm
Other:
- board size 160 x 100 mm -> 148 x 100 mm
- board text added: "+12V"
- board text added: "+5V"
- board text added: "EARTH"
- board text added: "picoRC.com"
- board text removed: "NOT FINISHED YET! CHECK REAL HARDWARE! IS GND AND PE CONNECTED?"

Commit message: working on os1
Parts:
- removed R1: (no value), adafruit_changed:0411/15
- moved JP2 10.2 mm to (141.0, 49.5)
- moved JP3 6.35 mm to (141.0, 66.0)
- moved JP1 2.54 mm to (141.0, 82.5)
- moved R2 1.80 mm to (6.22, 46.7)
- flipped U$9 to the bottom
Connections:
- net +12V: no longer R1.2
- net GND: no longer R1.1
Routing:
- net +12V: track 178.7 -> 159.9 mm
- net +5V: track 201.9 -> 212.8 mm
- net N$2: track 138.2 -> 138.9 mm
Other:
- board text added: "NC RED ORANGE YELLOW"

Commit message: working on os1
Routing:
- net +12V: track 159.9 -> 120.5 mm
Changed lines of the file:
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@@
 <layer number="19" name="Unrouted" color="6" fill="1" visible="yes" active="yes"/>
 <layer number="20" name="Dimension" color="24" fill="1" visible="yes" active="yes"/>
-<layer number="21" name="tPlace" color="7" fill="1" visible="no" active="yes"/>
+<layer number="21" name="tPlace" color="7" fill="1" visible="yes" active="yes"/>
 <layer number="22" name="bPlace" color="7" fill="1" visible="yes" active="yes"/>
-<layer number="23" name="tOrigins" color="15" fill="1" visible="no" active="yes"/>
+<layer number="23" name="tOrigins" color="15" fill="1" visible="yes" active="yes"/>
 <layer number="24" name="bOrigins" color="15" fill="1" visible="yes" active="yes"/>
-<layer number="25" name="tNames" color="7" fill="1" visible="no" active="yes"/>
+<layer number="25" name="tNames" color="7" fill="1" visible="yes" active="yes"/>
 <layer number="26" name="bNames" color="7" fill="1" visible="yes" active="yes"/>
-<layer number="27" name="tValues" color="7" fill="1" visible="no" active="yes"/>
-<layer number="28" name="bValues" color="7" fill="1" visible="no" active="yes"/>
+<layer number="27" name="tValues" color="7" fill="1" visible="yes" active="yes"/>
+<layer number="28" name="bValues" color="7" fill="1" visible="yes" active="yes"/>
 <layer number="29" name="tStop" color="7" fill="3" visible="no" active="yes"/>
 <layer number="30" name="bStop" color="7" fill="6" visible="no" active="yes"/>
@@
 <layer number="37" name="tTest" color="7" fill="1" visible="no" active="yes"/>
 <layer number="38" name="bTest" color="7" fill="1" visible="no" active="yes"/>
-<layer number="39" name="tKeepout" color="4" fill="11" visible="no" active="yes"/>
+<layer number="39" name="tKeepout" color="4" fill="11" visible="yes" active="yes"/>
 <layer number="40" name="bKeepout" color="1" fill="11" visible="yes" active="yes"/>
-<layer number="41" name="tRestrict" color="4" fill="10" visible="no" active="yes"/>
+<layer number="41" name="tRestrict" color="4" fill="10" visible="yes" active="yes"/>
 <layer number="42" name="bRestrict" color="1" fill="10" visible="yes" active="yes"/>
 <layer number="43" name="vRestrict" color="2" fill="10" visible="no" active="yes"/>
@@
 <layer number="49" name="Reference" color="7" fill="1" visible="no" active="yes"/>
 <layer number="50" name="dxf" color="7" fill="1" visible="no" active="no"/>
-<layer number="51" name="tDocu" color="7" fill="1" visible="no" active="yes"/>
+<layer number="51" name="tDocu" color="7" fill="1" visible="yes" active="yes"/>
 <layer number="52" name="bDocu" color="7" fill="1" visible="yes" active="yes"/>
 <layer number="53" name="tGND_GNDA" color="7" fill="1" visible="no" active="no"/>
@@
 <text x="133.311" y="53.44" size="1.6764" layer="25" align="center">NC</text>
 <polygon width="1.27" layer="41">
-<vertex x="99.25" y="35.5"/>
+<vertex x="115.76" y="35.5"/>
 <vertex x="150.25" y="35.5"/>
 <vertex x="150.25" y="15.5"/>
-<vertex x="99.75" y="15.5"/>
-<vertex x="96" y="19.25"/>
-<vertex x="96" y="32.25"/>
+<vertex x="116.26" y="15.5"/>
+<vertex x="112.51" y="19.25"/>
+<vertex x="112.51" y="32.25"/>
 </polygon>
 <text x="6.636" y="58.002" size="3.81" layer="25" rot="SR270" align="center">5V
@@
 <wire x1="132" y1="83.74" x2="132.08" y2="83.82" width="1.27" layer="16"/>
 <wire x1="137.16" y1="67.31" x2="132" y2="67.31" width="1.27" layer="16"/>
-<wire x1="132" y1="46.27" x2="130.48" y2="44.75" width="1.27" layer="16"/>
+<wire x1="132" y1="47.54" x2="129.21" y2="44.75" width="1.27" layer="16"/>
 <wire x1="132" y1="67.31" x2="132" y2="59" width="1.27" layer="16"/>
 <wire x1="132" y1="59" x2="132" y2="50.8" width="1.27" layer="16"/>
-<wire x1="132" y1="50.8" x2="132" y2="46.27" width="1.27" layer="16"/>
+<wire x1="132" y1="50.8" x2="132" y2="47.54" width="1.27" layer="16"/>
 <wire x1="137.16" y1="50.8" x2="132" y2="50.8" width="1.27" layer="16"/>
 <wire x1="126" y1="59" x2="132" y2="59" width="1.27" layer="16"/>
-<wire x1="130.48" y1="44.75" x2="96.82" y2="44.75" width="1.27" layer="16"/>
-<wire x1="96.82" y1="44.75" x2="92.71" y2="40.64" width="1.27" layer="16"/>
-<wire x1="92.71" y1="40.64" x2="92.71" y2="17.78" width="1.27" layer="16"/>
-<wire x1="92.71" y1="17.78" x2="97.282" y2="13.208" width="1.27" layer="16"/>
-<wire x1="97.282" y1="13.208" x2="115.824" y2="13.208" width="1.27" layer="16"/>
-<wire x1="120.52" y1="8.512" x2="120.52" y2="3.75" width="1.27" layer="16"/>
-<wire x1="115.824" y1="13.208" x2="120.52" y2="8.512" width="1.27" layer="16"/>
+<wire x1="129.21" y1="44.75" x2="120.95" y2="44.75" width="1.27" layer="16"/>
+<wire x1="120.95" y1="44.75" x2="109.22" y2="33.02" width="1.27" layer="16"/>
+<wire x1="109.22" y1="33.02" x2="109.22" y2="17.272" width="1.27" layer="16"/>
+<wire x1="109.22" y1="17.272" x2="120.52" y2="5.972" width="1.27" layer="16"/>
+<wire x1="120.52" y1="5.972" x2="120.52" y2="3.75" width="1.27" layer="16"/>
 </signal>
 <signal name="NEUTRAL">

Commit message: mw os1
Parts:
- removed U$14, U$3: 28FLAG, blade:2.8FLAG
- U$1: device apricot:MEANWELL_RD50 -> os1:MEANWELL_RD50
- U$2: value TERM9.5 -> TERM_RD50; device os1:TERMINAL9500 -> os1:TERMINAL9500_NOMAINS
- moved TP1 92.5 mm to (138.0, 97.5)
- moved TP2 92.5 mm to (143.0, 97.5)
- moved C4 4.12 mm to (140.5, 93.0)
- moved C6 4.12 mm to (140.5, 89.5)
- moved JP1 2.00 mm to (141.0, 80.5)
- moved JP2 2.00 mm to (141.0, 47.5)
- moved JP3 2.00 mm to (141.0, 64.0)
Connections:
- removed net LIVE: U$2.P$7, U$3.P$1, U$3.P$2
- removed net NEUTRAL: U$14.P$1, U$14.P$2, U$2.P$6
- net GND: now also U$1.P$1, U$1.P$2
Routing:
- net GND: track 0.00 -> 134.0 mm
- net NEUTRAL: track 13.7 -> 0.00 mm
- net LIVE: track 13.5 -> 0.00 mm
- net +12V: track 120.5 -> 109.5 mm
- net +5V: track 212.8 -> 211.0 mm
Other:
- board size 148 x 100 mm -> 147.1 x 100 mm
- board text added: "PE"
