File: pcb/os1_mw/osborne1.brd (EAGLE design)
At the start: 147.1 x 100 mm, 17 parts

Commit message: updated osborne 1 pcb
Parts:
- added U$3: TERM_RD50_MAINS, os1:TERMINAL9500_MAINS
- added U$7: CAR_FUSE_HOLDER3IN1, atx_power_control:FUSE_HOLDER_3IN1
- U$2: value TERM_RD50 -> 396_2P_LIVE; device os1:TERMINAL9500_NOMAINS -> 396_conn:396_2P_LIVE
- moved U$2 59.4 mm to (139.0, 20.0), turned to 90 degrees
- moved JP3 12.0 mm to (141.0, 52.0)
- moved JP1 12.0 mm to (141.0, 68.5)
- moved JP2 12.0 mm to (141.0, 35.5)
- moved R2 4.26 mm to (6.00, 51.0)
Connections:
- new net N$1: U$3.P$3, U$7.B0, U$7.B1
- new net N$3: U$2.P$2, U$3.P$6
- new net N$4: U$2.P$1, U$3.P$7
- net +12V: now also U$7.A0, U$7.A1; no longer U$2.P$3
- net GND: now also U$3.P$2, U$3.P$4, U$3.P$5; no longer U$2.P$2, U$2.P$4, U$2.P$5
- net N$2: now also U$3.P$1; no longer U$2.P$1
Routing:
- net GND: track 134.0 -> 0.00 mm
- net N$1: track 0.00 -> 130.8 mm
- net +12V: track 109.5 -> 207.7 mm
- net N$3: track 0.00 -> 15.7 mm
- net N$4: track 0.00 -> 15.1 mm
- net +5V: track 211.0 -> 222.7 mm
- net N$2: track 138.9 -> 134.8 mm
Other:
- outline, holes or cut-outs redrawn
- board text added: "12V 3A"

Commit message: adjust pcb
Parts:
- moved U$2 1.00 mm to (139.0, 19.0)
Other:
- outline, holes or cut-outs redrawn
- board text added: "L"
- board text added: "N"
- board text removed: "LIVE"
- board text removed: "NEUTRAL"
Changed lines of the file:
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@@
 <setting verticaltext="up"/>
 </settings>
-<grid distance="1" unitdist="mm" unit="mm" style="lines" multiple="1" display="no" altdistance="1" altunitdist="mil" altunit="mil"/>
+<grid distance="0.5" unitdist="mm" unit="mm" style="lines" multiple="1" display="no" altdistance="1" altunitdist="mil" altunit="mil"/>
 <layers>
-<layer number="1" name="Top" color="4" fill="1" visible="no" active="yes"/>
+<layer number="1" name="Top" color="4" fill="1" visible="yes" active="yes"/>
 <layer number="2" name="Route2" color="16" fill="1" visible="no" active="no"/>
 <layer number="3" name="Route3" color="17" fill="1" visible="no" active="no"/>
@@
 <layer number="19" name="Unrouted" color="6" fill="1" visible="yes" active="yes"/>
 <layer number="20" name="Dimension" color="24" fill="1" visible="yes" active="yes"/>
-<layer number="21" name="tPlace" color="7" fill="1" visible="no" active="yes"/>
+<layer number="21" name="tPlace" color="7" fill="1" visible="yes" active="yes"/>
 <layer number="22" name="bPlace" color="7" fill="1" visible="yes" active="yes"/>
-<layer number="23" name="tOrigins" color="15" fill="1" visible="no" active="yes"/>
+<layer number="23" name="tOrigins" color="15" fill="1" visible="yes" active="yes"/>
 <layer number="24" name="bOrigins" color="15" fill="1" visible="yes" active="yes"/>
-<layer number="25" name="tNames" color="7" fill="1" visible="no" active="yes"/>
+<layer number="25" name="tNames" color="7" fill="1" visible="yes" active="yes"/>
 <layer number="26" name="bNames" color="7" fill="1" visible="yes" active="yes"/>
-<layer number="27" name="tValues" color="7" fill="1" visible="no" active="yes"/>
-<layer number="28" name="bValues" color="7" fill="1" visible="no" active="yes"/>
+<layer number="27" name="tValues" color="7" fill="1" visible="yes" active="yes"/>
+<layer number="28" name="bValues" color="7" fill="1" visible="yes" active="yes"/>
 <layer number="29" name="tStop" color="7" fill="3" visible="no" active="yes"/>
 <layer number="30" name="bStop" color="7" fill="6" visible="no" active="yes"/>
@@
 <layer number="37" name="tTest" color="7" fill="1" visible="no" active="yes"/>
 <layer number="38" name="bTest" color="7" fill="1" visible="no" active="yes"/>
-<layer number="39" name="tKeepout" color="4" fill="11" visible="no" active="yes"/>
+<layer number="39" name="tKeepout" color="4" fill="11" visible="yes" active="yes"/>
 <layer number="40" name="bKeepout" color="1" fill="11" visible="yes" active="yes"/>
-<layer number="41" name="tRestrict" color="4" fill="10" visible="no" active="yes"/>
+<layer number="41" name="tRestrict" color="4" fill="10" visible="yes" active="yes"/>
 <layer number="42" name="bRestrict" color="1" fill="10" visible="yes" active="yes"/>
 <layer number="43" name="vRestrict" color="2" fill="10" visible="no" active="yes"/>
@@
 <layer number="49" name="Reference" color="7" fill="1" visible="no" active="yes"/>
 <layer number="50" name="dxf" color="7" fill="1" visible="no" active="no"/>
-<layer number="51" name="tDocu" color="7" fill="1" visible="no" active="yes"/>
+<layer number="51" name="tDocu" color="7" fill="1" visible="yes" active="yes"/>
 <layer number="52" name="bDocu" color="7" fill="1" visible="yes" active="yes"/>
 <layer number="53" name="tGND_GNDA" color="7" fill="1" visible="no" active="no"/>
@@
 <wire x1="5" y1="0" x2="143" y2="0" width="0" layer="20"/>
 <wire x1="143" y1="0" x2="147" y2="6" width="0" layer="20" curve="90"/>
-<text x="133.799" y="76.854" size="1.778" layer="25" align="center">YL</text>
-<text x="133.771" y="79.394" size="1.6764" layer="25" align="center">OG</text>
-<text x="133.803" y="81.934" size="1.6764" layer="25" align="center">RD</text>
-<text x="133.692" y="84.474" size="1.6764" layer="25" align="center">NC</text>
+<text x="132.799" y="64.854" size="1.778" layer="25" align="center">YL</text>
+<text x="132.771" y="67.394" size="1.6764" layer="25" align="center">OG</text>
+<text x="132.803" y="69.934" size="1.6764" layer="25" align="center">RD</text>
+<text x="132.692" y="72.474" size="1.6764" layer="25" align="center">NC</text>
 <text x="133.578" y="97.436" size="2.54" layer="25" rot="R180" align="center">PE</text>
-<text x="113.5" y="20.5" size="3.81" layer="25" align="center-left">LIVE</text>
-<text x="113.5" y="30" size="3.81" layer="25" align="center-left">NEUTRAL</text>
-<text x="133.418" y="43.82" size="1.778" layer="25" align="center">YL</text>
-<text x="133.39" y="46.36" size="1.6764" layer="25" align="center">OG</text>
-<text x="133.422" y="48.9" size="1.6764" layer="25" align="center">RD</text>
-<text x="133.311" y="51.44" size="1.6764" layer="25" align="center">NC</text>
+<text x="113.5" y="20.5" size="3.81" layer="25" align="center-left">L</text>
+<text x="113.5" y="31" size="3.81" layer="25" align="center-left">N</text>
+<text x="133.918" y="31.82" size="1.778" layer="25" align="center">YL</text>
+<text x="133.89" y="34.36" size="1.6764" layer="25" align="center">OG</text>
+<text x="133.922" y="36.9" size="1.6764" layer="25" align="center">RD</text>
+<text x="133.811" y="39.44" size="1.6764" layer="25" align="center">NC</text>
 <text x="-16.936" y="29.328" size="3.81" layer="25" rot="SR270" align="center">picoRC.com</text>
 <text x="130.828" y="2.686" size="2.54" layer="25" rot="R180" align="center">PC FAN</text>
@@
 <text x="121.672" y="69.064" size="5.08" layer="26" rot="MR0" align="center-left">GND</text>
 <text x="121.672" y="78.064" size="5.08" layer="26" rot="MR0" align="center-left">+5V</text>
-<text x="133.672" y="60.203" size="1.778" layer="25" align="center">YL</text>
-<text x="133.644" y="62.743" size="1.6764" layer="25" align="center">OG</text>
-<text x="133.676" y="65.283" size="1.6764" layer="25" align="center">RD</text>
-<text x="133.565" y="67.823" size="1.6764" layer="25" align="center">NC</text>
+<text x="132.672" y="48.203" size="1.778" layer="25" align="center">YL</text>
+<text x="132.644" y="50.743" size="1.6764" layer="25" align="center">OG</text>
+<text x="132.676" y="53.283" size="1.6764" layer="25" align="center">RD</text>
+<text x="132.565" y="55.823" size="1.6764" layer="25" align="center">NC</text>
 <text x="139.772" y="68.396" size="1.4224" layer="26" distance="80" rot="MR0" align="center-right">NC
 RED
@@
 <vertex x="132.75" y="31.5"/>
 <vertex x="145.25" y="31.5"/>
-<vertex x="145.25" y="13.5"/>
-<vertex x="132.75" y="13.5"/>
+<vertex x="145.25" y="12.5"/>
+<vertex x="132.75" y="12.5"/>
 </polygon>
-<rectangle x1="135" y1="19" x2="143" y2="21" layer="46"/>
+<rectangle x1="135" y1="18" x2="143" y2="20" layer="46"/>
 <rectangle x1="121" y1="24.5" x2="131" y2="26.5" layer="46"/>
 <text x="12.096" y="30.002" size="3.81" layer="26" rot="MR90" align="center">12V 3A</text>
+<text x="144.5" y="24" size="3.81" layer="25" align="center-left">N</text>
+<text x="144.5" y="14.5" size="3.81" layer="25" align="center-left">L</text>
 </plain>
 <attributes>
@@
 </element>
 <element name="U$3" library="os1" package="TERMINAL9500_MAINS" value="TERM_RD50_MAINS" x="126" y="78" smashed="yes" rot="R270"/>
-<element name="U$2" library="396_conn" package="396_2P_LIVE" value="396_2P_LIVE" x="139" y="20" smashed="yes" rot="R90"/>
+<element name="U$2" library="396_conn" package="396_2P_LIVE" value="396_2P_LIVE" x="139" y="19" smashed="yes" rot="R90"/>
 <element name="U$7" library="atx_power_control" package="FUSE_HOLDER_3IN1" value="CAR_FUSE_HOLDER3IN1" x="6" y="30" smashed="yes" rot="MR90"/>
 </elements>
@@
 <contactref element="U$3" pad="P$6"/>
 <contactref element="U$2" pad="P$2"/>
-<wire x1="139" y1="23.96" x2="135.04" y2="23.96" width="1.27" layer="16"/>
-<wire x1="128.5" y1="30.5" x2="126" y2="30.5" width="1.27" layer="16"/>
-<wire x1="135.04" y1="23.96" x2="128.5" y2="30.5" width="1.27" layer="16"/>
+<wire x1="139" y1="22.96" x2="137.04" y2="22.96" width="1.27" layer="16"/>
+<wire x1="129.5" y1="30.5" x2="126" y2="30.5" width="1.27" layer="16"/>
+<wire x1="137.04" y1="22.96" x2="129.5" y2="30.5" width="1.27" layer="16"/>
 </signal>
 <signal name="N$4">
 <contactref element="U$2" pad="P$1"/>
 <contactref element="U$3" pad="P$7"/>
-<wire x1="139" y1="16.04" x2="134.46" y2="16.04" width="1.27" layer="16"/>
-<wire x1="134.46" y1="16.04" x2="129.5" y2="21" width="1.27" layer="16"/>
+<wire x1="139" y1="15.04" x2="135.46" y2="15.04" width="1.27" layer="16"/>
+<wire x1="135.46" y1="15.04" x2="129.5" y2="21" width="1.27" layer="16"/>
 <wire x1="129.5" y1="21" x2="126" y2="21" width="1.27" layer="16"/>
 </signal>

Commit message: updated osborne 1 pcb
Parts:
- moved C4 3.00 mm to (140.5, 90.0)
- moved C6 3.00 mm to (140.5, 86.5)
Routing:
- net +5V: track 222.7 -> 221.6 mm
Other:
- board size 147.1 x 100 mm -> 147 x 100 mm
- board text added: "LIVE"
- board text added: "NEUTRAL"
Changed lines of the file:
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@@
 <setting verticaltext="up"/>
 </settings>
-<grid distance="0.5" unitdist="mm" unit="mm" style="lines" multiple="1" display="no" altdistance="1" altunitdist="mil" altunit="mil"/>
+<grid distance="1" unitdist="mm" unit="mm" style="lines" multiple="1" display="no" altdistance="1" altunitdist="mil" altunit="mil"/>
 <layers>
-<layer number="1" name="Top" color="4" fill="1" visible="yes" active="yes"/>
+<layer number="1" name="Top" color="4" fill="1" visible="no" active="yes"/>
 <layer number="2" name="Route2" color="16" fill="1" visible="no" active="no"/>
 <layer number="3" name="Route3" color="17" fill="1" visible="no" active="no"/>
@@
 <layer number="19" name="Unrouted" color="6" fill="1" visible="yes" active="yes"/>
 <layer number="20" name="Dimension" color="24" fill="1" visible="yes" active="yes"/>
-<layer number="21" name="tPlace" color="7" fill="1" visible="yes" active="yes"/>
+<layer number="21" name="tPlace" color="7" fill="1" visible="no" active="yes"/>
 <layer number="22" name="bPlace" color="7" fill="1" visible="yes" active="yes"/>
-<layer number="23" name="tOrigins" color="15" fill="1" visible="yes" active="yes"/>
+<layer number="23" name="tOrigins" color="15" fill="1" visible="no" active="yes"/>
 <layer number="24" name="bOrigins" color="15" fill="1" visible="yes" active="yes"/>
-<layer number="25" name="tNames" color="7" fill="1" visible="yes" active="yes"/>
+<layer number="25" name="tNames" color="7" fill="1" visible="no" active="yes"/>
 <layer number="26" name="bNames" color="7" fill="1" visible="yes" active="yes"/>
-<layer number="27" name="tValues" color="7" fill="1" visible="yes" active="yes"/>
-<layer number="28" name="bValues" color="7" fill="1" visible="yes" active="yes"/>
+<layer number="27" name="tValues" color="7" fill="1" visible="no" active="yes"/>
+<layer number="28" name="bValues" color="7" fill="1" visible="no" active="yes"/>
 <layer number="29" name="tStop" color="7" fill="3" visible="no" active="yes"/>
 <layer number="30" name="bStop" color="7" fill="6" visible="no" active="yes"/>
@@
 <layer number="37" name="tTest" color="7" fill="1" visible="no" active="yes"/>
 <layer number="38" name="bTest" color="7" fill="1" visible="no" active="yes"/>
-<layer number="39" name="tKeepout" color="4" fill="11" visible="yes" active="yes"/>
+<layer number="39" name="tKeepout" color="4" fill="11" visible="no" active="yes"/>
 <layer number="40" name="bKeepout" color="1" fill="11" visible="yes" active="yes"/>
-<layer number="41" name="tRestrict" color="4" fill="10" visible="yes" active="yes"/>
+<layer number="41" name="tRestrict" color="4" fill="10" visible="no" active="yes"/>
 <layer number="42" name="bRestrict" color="1" fill="10" visible="yes" active="yes"/>
 <layer number="43" name="vRestrict" color="2" fill="10" visible="no" active="yes"/>
@@
 <layer number="49" name="Reference" color="7" fill="1" visible="no" active="yes"/>
 <layer number="50" name="dxf" color="7" fill="1" visible="no" active="no"/>
-<layer number="51" name="tDocu" color="7" fill="1" visible="yes" active="yes"/>
+<layer number="51" name="tDocu" color="7" fill="1" visible="no" active="yes"/>
 <layer number="52" name="bDocu" color="7" fill="1" visible="yes" active="yes"/>
 <layer number="53" name="tGND_GNDA" color="7" fill="1" visible="no" active="no"/>
@@
 <board>
 <plain>
-<wire x1="147" y1="6" x2="147" y2="96" width="0" layer="20"/>
+<wire x1="5" y1="0" x2="142" y2="0" width="0" layer="20"/>
+<wire x1="142" y1="0" x2="147" y2="5" width="0" layer="20" curve="90"/>
+<wire x1="147" y1="5" x2="147" y2="96" width="0" layer="20"/>
 <wire x1="147" y1="96" x2="143" y2="100" width="0" layer="20" curve="90"/>
 <wire x1="143" y1="100" x2="5" y2="100" width="0" layer="20"/>
@@
 <wire x1="0" y1="95" x2="0" y2="5" width="0" layer="20"/>
 <wire x1="0" y1="5" x2="5" y2="0" width="0" layer="20" curve="90"/>
-<wire x1="5" y1="0" x2="143" y2="0" width="0" layer="20"/>
-<wire x1="143" y1="0" x2="147" y2="6" width="0" layer="20" curve="90"/>
 <text x="132.799" y="64.854" size="1.778" layer="25" align="center">YL</text>
 <text x="132.771" y="67.394" size="1.6764" layer="25" align="center">OG</text>
@@
 <text x="144.5" y="24" size="3.81" layer="25" align="center-left">N</text>
 <text x="144.5" y="14.5" size="3.81" layer="25" align="center-left">L</text>
+<text x="120.672" y="21.064" size="5.08" layer="26" rot="MR0" align="center-left">LIVE</text>
+<text x="120.672" y="31.064" size="5.08" layer="26" rot="MR0" align="center-left">NEUTRAL</text>
+<wire x1="132" y1="33" x2="123" y2="33" width="0.508" layer="22"/>
+<wire x1="123" y1="33" x2="122" y2="32" width="0.508" layer="22"/>
+<wire x1="122" y1="32" x2="122" y2="19" width="0.508" layer="22"/>
+<wire x1="122" y1="19" x2="123" y2="18" width="0.508" layer="22"/>
+<wire x1="123" y1="18" x2="128" y2="18" width="0.508" layer="22"/>
+<wire x1="128" y1="18" x2="135" y2="11" width="0.508" layer="22"/>
+<wire x1="135" y1="11" x2="142" y2="11" width="0.508" layer="22"/>
+<wire x1="142" y1="11" x2="143" y2="12" width="0.508" layer="22"/>
+<wire x1="143" y1="12" x2="143" y2="24" width="0.508" layer="22"/>
+<wire x1="143" y1="24" x2="141" y2="26" width="0.508" layer="22"/>
+<wire x1="141" y1="26" x2="139" y2="26" width="0.508" layer="22"/>
+<wire x1="139" y1="26" x2="132" y2="33" width="0.508" layer="22"/>
 </plain>
 <attributes>
@@
 <element name="U$8" library="os1" package="M3_HOLE_PLATED" value="M3_HOLE_PLATED" x="129" y="90" smashed="yes"/>
 <element name="U$9" library="atx_power_control" package="FUSE_HOLDER_3IN1" value="CAR_FUSE_HOLDER3IN1" x="6" y="73" smashed="yes" rot="MR270"/>
-<element name="C4" library="capacitor-wima" library_urn="urn:adsk.eagle:library:116" package="C5B2.5" package3d_urn="urn:adsk.eagle:package:5426/1" value="" x="140.5" y="93" smashed="yes">
-<attribute name="NAME" x="144.968" y="92.524" size="1.27" layer="25" ratio="10"/>
-<attribute name="POPULARITY" value="10" x="140.5" y="103" size="1.778" layer="27" display="off"/>
-<attribute name="VALUE" x="138.468" y="90.206" size="1.27" layer="27" ratio="10"/>
+<element name="C4" library="capacitor-wima" library_urn="urn:adsk.eagle:library:116" package="C5B2.5" package3d_urn="urn:adsk.eagle:package:5426/1" value="" x="140.5" y="90" smashed="yes">
+<attribute name="NAME" x="144.968" y="89.524" size="1.27" layer="25" ratio="10"/>
+<attribute name="POPULARITY" value="10" x="140.5" y="100" size="1.778" layer="27" display="off"/>
+<attribute name="VALUE" x="138.468" y="87.206" size="1.27" layer="27" ratio="10"/>
 </element>
 <element name="C5" library="adafruit_changed" package="E3,5-8" value="" x="119" y="93" smashed="yes" rot="R135">
@@
 <attribute name="VALUE" x="122.77170625" y="93.538815625" size="1.27" layer="27" ratio="10" rot="R135"/>
 </element>
-<element name="C6" library="capacitor-wima" library_urn="urn:adsk.eagle:library:116" package="C5B2.5" package3d_urn="urn:adsk.eagle:package:5426/1" value="" x="140.5" y="89.5" smashed="yes">
-<attribute name="NAME" x="144.968" y="89.024" size="1.27" layer="25" ratio="10"/>
-<attribute name="POPULARITY" value="10" x="140.5" y="90.5" size="1.778" layer="27" display="off"/>
-<attribute name="VALUE" x="138.468" y="86.706" size="1.27" layer="27" ratio="10"/>
+<element name="C6" library="capacitor-wima" library_urn="urn:adsk.eagle:library:116" package="C5B2.5" package3d_urn="urn:adsk.eagle:package:5426/1" value="" x="140.5" y="86.5" smashed="yes">
+<attribute name="NAME" x="144.968" y="86.024" size="1.27" layer="25" ratio="10"/>
+<attribute name="POPULARITY" value="10" x="140.5" y="87.5" size="1.778" layer="27" display="off"/>
+<attribute name="VALUE" x="138.468" y="83.706" size="1.27" layer="27" ratio="10"/>
 </element>
 <element name="TP1" library="testpad" library_urn="urn:adsk.eagle:library:385" package="P1-17" package3d_urn="urn:adsk.eagle:package:27949/1" value="PTR1PAD1-17" x="138" y="97.5" smashed="yes" rot="R90">
@@
 <wire x1="14.116" y1="80.05" x2="7.75" y2="80.05" width="2.54" layer="16"/>
 <wire x1="7.75" y1="80.05" x2="4.25" y2="80.05" width="2.54" layer="16"/>
-<wire x1="137.96" y1="93" x2="136" y2="93" width="2.54" layer="16"/>
+<wire x1="137.96" y1="90" x2="137.96" y2="91.04" width="2.54" layer="16"/>
 <wire x1="132" y1="97" x2="125.514471875" y2="97" width="2.54" layer="16"/>
-<wire x1="136" y1="93" x2="132" y2="97" width="2.54" layer="16"/>
-<wire x1="137.96" y1="93" x2="137.96" y2="89.5" width="2.54" layer="16"/>
-<wire x1="137.96" y1="89.5" x2="137.96" y2="86.04" width="2.54" layer="16"/>
+<wire x1="137.96" y1="91.04" x2="132" y2="97" width="2.54" layer="16"/>
+<wire x1="137.96" y1="90" x2="137.96" y2="86.5" width="2.54" layer="16"/>
+<wire x1="137.96" y1="86.5" x2="137.96" y2="86.04" width="2.54" layer="16"/>
 <wire x1="143" y1="33" x2="143" y2="48" width="2.54" layer="16"/>
 <wire x1="143" y1="48" x2="143" y2="65" width="2.54" layer="16"/>
