File: pcb/os1_mw/osborne1.sch (EAGLE design)
At the start: 17 parts

Commit message: adjust pcb
Parts:
- removed U$7: 396_2P_LIVE, 396_conn:396_2P_LIVE
- added R1, R2: (no value), adafruit_changed:R-US_0411/15
- added U$14, U$3: 28FLAG, blade:28FLAG
Connections:
- removed net PE: U$2.P$5, U$4.P$1, U$5.P$1, U$6.P$1, U$8.P$1
- net +12V: now also R1.2
- net GND: now also R1.1, R2.2, U$2.P$5, U$4.P$1, U$5.P$1, U$6.P$1, U$8.P$1
- net LIVE: now also U$3.P$1; no longer U$7.P$1
- net N$2: now also R2.1
- net NEUTRAL: now also U$14.P$1; no longer U$7.P$2
Changed lines of the file:
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@@
 <part name="P+3" library="supply1" library_urn="urn:adsk.eagle:library:371" deviceset="+12V" device=""/>
 <part name="GND4" library="supply1" library_urn="urn:adsk.eagle:library:371" deviceset="GND" device=""/>
-<part name="U$7" library="396_conn" deviceset="396_2P_LIVE" device=""/>
 <part name="P+1" library="supply1" library_urn="urn:adsk.eagle:library:371" deviceset="+5V" device=""/>
 <part name="P+4" library="supply1" library_urn="urn:adsk.eagle:library:371" deviceset="+12V" device=""/>
@@
 <part name="GND13" library="supply1" library_urn="urn:adsk.eagle:library:371" deviceset="GND" device=""/>
 <part name="P+10" library="supply1" library_urn="urn:adsk.eagle:library:371" deviceset="+12V" device=""/>
-<part name="PE1" library="supply1" library_urn="urn:adsk.eagle:library:371" deviceset="PE" device=""/>
-<part name="PE2" library="supply1" library_urn="urn:adsk.eagle:library:371" deviceset="PE" device=""/>
+<part name="GND1" library="supply1" library_urn="urn:adsk.eagle:library:371" deviceset="GND" device=""/>
+<part name="U$14" library="blade" deviceset="28FLAG" device=""/>
+<part name="U$3" library="blade" deviceset="28FLAG" device=""/>
+<part name="R2" library="adafruit_changed" deviceset="R-US_" device="0411/15"/>
+<part name="GND3" library="supply1" library_urn="urn:adsk.eagle:library:371" deviceset="GND" device=""/>
+<part name="R1" library="adafruit_changed" deviceset="R-US_" device="0411/15"/>
+<part name="GND5" library="supply1" library_urn="urn:adsk.eagle:library:371" deviceset="GND" device=""/>
 </parts>
 <sheets>
@@
 <attribute name="VALUE" x="58.42" y="-33.02" size="1.778" layer="96" rot="MR0"/>
 </instance>
-<instance part="U$7" gate="G$1" x="10.16" y="-68.58" smashed="yes" rot="R180"/>
 <instance part="P+1" gate="1" x="139.7" y="-20.32" smashed="yes" rot="MR270">
 <attribute name="VALUE" x="137.16" y="-20.32" size="1.778" layer="96" rot="MR0"/>
@@
 <attribute name="VALUE" x="203.2" y="20.32" size="1.778" layer="96" rot="MR90"/>
 </instance>
-<instance part="PE1" gate="M" x="45.72" y="-35.56" smashed="yes">
-<attribute name="VALUE" x="43.18" y="-38.1" size="1.778" layer="96" rot="R90"/>
-</instance>
-<instance part="PE2" gate="M" x="27.94" y="96.52" smashed="yes">
-<attribute name="VALUE" x="25.4" y="93.98" size="1.778" layer="96" rot="R90"/>
+<instance part="GND1" gate="1" x="27.94" y="99.06" smashed="yes" rot="MR0">
+<attribute name="VALUE" x="30.48" y="96.52" size="1.778" layer="96" rot="MR0"/>
+</instance>
+<instance part="U$14" gate="G$1" x="53.34" y="-38.1" smashed="yes"/>
+<instance part="U$3" gate="G$1" x="53.34" y="-43.18" smashed="yes"/>
+<instance part="R2" gate="G$1" x="20.32" y="2.54" smashed="yes">
+<attribute name="NAME" x="16.51" y="4.0386" size="1.778" layer="95"/>
+<attribute name="VALUE" x="16.51" y="-0.762" size="1.778" layer="96"/>
+</instance>
+<instance part="GND3" gate="1" x="35.56" y="0" smashed="yes" rot="MR0">
+<attribute name="VALUE" x="38.1" y="-2.54" size="1.778" layer="96" rot="MR0"/>
+</instance>
+<instance part="R1" gate="G$1" x="-15.24" y="-27.94" smashed="yes">
+<attribute name="NAME" x="-19.05" y="-26.4414" size="1.778" layer="95"/>
+<attribute name="VALUE" x="-19.05" y="-31.242" size="1.778" layer="96"/>
+</instance>
+<instance part="GND5" gate="1" x="-25.4" y="-30.48" smashed="yes" rot="MR0">
+<attribute name="VALUE" x="-22.86" y="-33.02" size="1.778" layer="96" rot="MR0"/>
 </instance>
 </instances>
@@
 <wire x1="48.26" y1="-17.78" x2="48.26" y2="-27.94" width="0.1524" layer="91"/>
 <junction x="48.26" y="-27.94"/>
+<wire x1="15.24" y1="-27.94" x2="5.08" y2="-27.94" width="0.1524" layer="91"/>
+<wire x1="5.08" y1="-27.94" x2="5.08" y2="-33.02" width="0.1524" layer="91"/>
+<junction x="15.24" y="-27.94"/>
+<pinref part="U$2" gate="G$1" pin="P$5"/>
+<wire x1="5.08" y1="-33.02" x2="15.24" y2="-33.02" width="0.1524" layer="91"/>
 </segment>
 <segment>
@@
 <wire x1="160.02" y1="27.94" x2="172.72" y2="27.94" width="0.1524" layer="91"/>
 </segment>
+<segment>
+<pinref part="U$6" gate="G$1" pin="P$1"/>
+<pinref part="GND1" gate="1" pin="GND"/>
+<wire x1="38.1" y1="101.6" x2="27.94" y2="101.6" width="0.1524" layer="91"/>
+<pinref part="U$8" gate="G$1" pin="P$1"/>
+<wire x1="27.94" y1="101.6" x2="27.94" y2="109.22" width="0.1524" layer="91"/>
+<wire x1="27.94" y1="109.22" x2="27.94" y2="116.84" width="0.1524" layer="91"/>
+<wire x1="27.94" y1="116.84" x2="27.94" y2="124.46" width="0.1524" layer="91"/>
+<wire x1="27.94" y1="124.46" x2="38.1" y2="124.46" width="0.1524" layer="91"/>
+<junction x="27.94" y="101.6"/>
+<pinref part="U$4" gate="G$1" pin="P$1"/>
+<wire x1="38.1" y1="116.84" x2="27.94" y2="116.84" width="0.1524" layer="91"/>
+<junction x="27.94" y="116.84"/>
+<pinref part="U$5" gate="G$1" pin="P$1"/>
+<wire x1="38.1" y1="109.22" x2="27.94" y2="109.22" width="0.1524" layer="91"/>
+<junction x="27.94" y="109.22"/>
+</segment>
+<segment>
+<pinref part="GND3" gate="1" pin="GND"/>
+<pinref part="R2" gate="G$1" pin="2"/>
+<wire x1="35.56" y1="2.54" x2="25.4" y2="2.54" width="0.1524" layer="91"/>
+</segment>
+<segment>
+<pinref part="GND5" gate="1" pin="GND"/>
+<pinref part="R1" gate="G$1" pin="1"/>
+<wire x1="-25.4" y1="-27.94" x2="-20.32" y2="-27.94" width="0.1524" layer="91"/>
+</segment>
 </net>
 <net name="+12V" class="0">
@@
 <pinref part="U$2" gate="G$1" pin="P$3"/>
 <pinref part="P+3" gate="1" pin="+12V"/>
-<wire x1="15.24" y1="-22.86" x2="-5.08" y2="-22.86" width="0.1524" layer="91"/>
+<wire x1="15.24" y1="-22.86" x2="0" y2="-22.86" width="0.1524" layer="91"/>
+<pinref part="R1" gate="G$1" pin="2"/>
+<wire x1="0" y1="-22.86" x2="-5.08" y2="-22.86" width="0.1524" layer="91"/>
+<wire x1="-10.16" y1="-27.94" x2="0" y2="-27.94" width="0.1524" layer="91"/>
+<wire x1="0" y1="-27.94" x2="0" y2="-22.86" width="0.1524" layer="91"/>
+<junction x="0" y="-22.86"/>
 </segment>
 <segment>
@@
 <label x="2.54" y="-38.1" size="1.778" layer="95" rot="MR0" xref="yes"/>
 <pinref part="U$2" gate="G$1" pin="P$6"/>
-</segment>
-<segment>
-<wire x1="15.24" y1="-66.04" x2="27.94" y2="-66.04" width="0.1524" layer="91"/>
-<pinref part="U$7" gate="G$1" pin="P$2"/>
-<label x="27.94" y="-66.04" size="1.778" layer="95" xref="yes"/>
+<pinref part="U$14" gate="G$1" pin="P$1"/>
+<wire x1="15.24" y1="-38.1" x2="43.18" y2="-38.1" width="0.1524" layer="91"/>
+<junction x="15.24" y="-38.1"/>
 </segment>
 </net>
 <net name="LIVE" class="0">
 <segment>
-<wire x1="10.16" y1="-43.18" x2="7.62" y2="-43.18" width="0.1524" layer="91"/>
 <label x="2.54" y="-43.18" size="1.778" layer="95" rot="MR0" xref="yes"/>
 <pinref part="U$2" gate="G$1" pin="P$7"/>
-<wire x1="7.62" y1="-43.18" x2="2.54" y2="-43.18" width="0.1524" layer="91"/>
-<wire x1="15.24" y1="-43.18" x2="10.16" y2="-43.18" width="0.1524" layer="91"/>
-</segment>
-<segment>
-<wire x1="17.78" y1="-68.58" x2="15.24" y2="-68.58" width="0.1524" layer="91"/>
-<pinref part="U$7" gate="G$1" pin="P$1"/>
-<label x="17.78" y="-68.58" size="1.778" layer="95" xref="yes"/>
+<wire x1="15.24" y1="-43.18" x2="2.54" y2="-43.18" width="0.1524" layer="91"/>
+<pinref part="U$3" gate="G$1" pin="P$1"/>
+<wire x1="43.18" y1="-43.18" x2="15.24" y2="-43.18" width="0.1524" layer="91"/>
+<junction x="15.24" y="-43.18"/>
 </segment>
 </net>
@@
 <wire x1="15.24" y1="-8.89" x2="7.874" y2="-8.89" width="0.1524" layer="91"/>
 <junction x="7.874" y="-8.89"/>
+<pinref part="R2" gate="G$1" pin="1"/>
+<wire x1="15.24" y1="2.54" x2="15.24" y2="-12.7" width="0.1524" layer="91"/>
+<junction x="15.24" y="-12.7"/>
 </segment>
 </net>
@@
 </segment>
 </net>
-<net name="PE" class="0">
-<segment>
-<pinref part="U$2" gate="G$1" pin="P$5"/>
-<pinref part="PE1" gate="M" pin="PE"/>
-<wire x1="15.24" y1="-33.02" x2="45.72" y2="-33.02" width="0.1524" layer="91"/>
-</segment>
-<segment>
-<pinref part="U$8" gate="G$1" pin="P$1"/>
-<wire x1="38.1" y1="124.46" x2="27.94" y2="124.46" width="0.1524" layer="91"/>
-<wire x1="27.94" y1="124.46" x2="27.94" y2="116.84" width="0.1524" layer="91"/>
-<pinref part="U$6" gate="G$1" pin="P$1"/>
-<wire x1="27.94" y1="116.84" x2="27.94" y2="109.22" width="0.1524" layer="91"/>
-<wire x1="27.94" y1="109.22" x2="27.94" y2="101.6" width="0.1524" layer="91"/>
-<wire x1="27.94" y1="101.6" x2="27.94" y2="99.06" width="0.1524" layer="91"/>
-<wire x1="38.1" y1="101.6" x2="27.94" y2="101.6" width="0.1524" layer="91"/>
-<junction x="27.94" y="101.6"/>
-<pinref part="U$4" gate="G$1" pin="P$1"/>
-<wire x1="38.1" y1="116.84" x2="27.94" y2="116.84" width="0.1524" layer="91"/>
-<junction x="27.94" y="116.84"/>
-<pinref part="U$5" gate="G$1" pin="P$1"/>
-<wire x1="38.1" y1="109.22" x2="27.94" y2="109.22" width="0.1524" layer="91"/>
-<junction x="27.94" y="109.22"/>
-<pinref part="PE2" gate="M" pin="PE"/>
-</segment>
-</net>

Commit message: working on os1
Parts:
- removed R1: (no value), adafruit_changed:R-US_0411/15
Connections:
- net +12V: no longer R1.2
- net GND: no longer R1.1
Changed lines of the file:
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@@
 <part name="R2" library="adafruit_changed" deviceset="R-US_" device="0411/15"/>
 <part name="GND3" library="supply1" library_urn="urn:adsk.eagle:library:371" deviceset="GND" device=""/>
-<part name="R1" library="adafruit_changed" deviceset="R-US_" device="0411/15"/>
-<part name="GND5" library="supply1" library_urn="urn:adsk.eagle:library:371" deviceset="GND" device=""/>
 </parts>
 <sheets>
@@
 <attribute name="VALUE" x="38.1" y="-2.54" size="1.778" layer="96" rot="MR0"/>
 </instance>
-<instance part="R1" gate="G$1" x="-15.24" y="-27.94" smashed="yes">
-<attribute name="NAME" x="-19.05" y="-26.4414" size="1.778" layer="95"/>
-<attribute name="VALUE" x="-19.05" y="-31.242" size="1.778" layer="96"/>
-</instance>
-<instance part="GND5" gate="1" x="-25.4" y="-30.48" smashed="yes" rot="MR0">
-<attribute name="VALUE" x="-22.86" y="-33.02" size="1.778" layer="96" rot="MR0"/>
-</instance>
 </instances>
 <busses>
@@
 <wire x1="35.56" y1="2.54" x2="25.4" y2="2.54" width="0.1524" layer="91"/>
 </segment>
-<segment>
-<pinref part="GND5" gate="1" pin="GND"/>
-<pinref part="R1" gate="G$1" pin="1"/>
-<wire x1="-25.4" y1="-27.94" x2="-20.32" y2="-27.94" width="0.1524" layer="91"/>
-</segment>
 </net>
 <net name="+12V" class="0">
@@
 <pinref part="U$2" gate="G$1" pin="P$3"/>
 <pinref part="P+3" gate="1" pin="+12V"/>
-<wire x1="15.24" y1="-22.86" x2="0" y2="-22.86" width="0.1524" layer="91"/>
-<pinref part="R1" gate="G$1" pin="2"/>
-<wire x1="0" y1="-22.86" x2="-5.08" y2="-22.86" width="0.1524" layer="91"/>
-<wire x1="-10.16" y1="-27.94" x2="0" y2="-27.94" width="0.1524" layer="91"/>
-<wire x1="0" y1="-27.94" x2="0" y2="-22.86" width="0.1524" layer="91"/>
-<junction x="0" y="-22.86"/>
+<wire x1="15.24" y1="-22.86" x2="-5.08" y2="-22.86" width="0.1524" layer="91"/>
 </segment>
 <segment>

Commit message: mw os1
Parts:
- removed U$14, U$3: 28FLAG, blade:28FLAG
- U$1: device apricot:MEANWELL_RD50 -> os1:MEANWELL_RD50
- U$2: value TERM9.5 -> TERM_RD50; device os1:TERM9.5 -> os1:TERM_RD50
Connections:
- removed net LIVE: U$2.P$7, U$3.P$1
- removed net NEUTRAL: U$14.P$1, U$2.P$6
- net +12V: now also U$2.+12V; no longer U$2.P$3
- net GND: now also U$1.P$1, U$1.P$2, U$2.EARTH, U$2.GND1, U$2.GND2; no longer U$2.P$2, U$2.P$4, U$2.P$5
- net N$2: now also U$2.+5V; no longer U$2.P$1
Changed lines of the file:
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@@
 </classes>
 <parts>
-<part name="U$1" library="apricot" deviceset="MEANWELL_RD50" device=""/>
-<part name="U$2" library="os1" deviceset="TERM9.5" device=""/>
+<part name="U$1" library="os1" deviceset="MEANWELL_RD50" device=""/>
+<part name="U$2" library="os1" deviceset="TERM_RD50" device=""/>
 <part name="JP2" library="pinhead" library_urn="urn:adsk.eagle:library:325" deviceset="PINHD-1X4" device="/90" package3d_urn="urn:adsk.eagle:package:22404/2"/>
 <part name="JP1" library="pinhead" library_urn="urn:adsk.eagle:library:325" deviceset="PINHD-1X4" device="/90" package3d_urn="urn:adsk.eagle:package:22404/2"/>
@@
 <part name="P+10" library="supply1" library_urn="urn:adsk.eagle:library:371" deviceset="+12V" device=""/>
 <part name="GND1" library="supply1" library_urn="urn:adsk.eagle:library:371" deviceset="GND" device=""/>
-<part name="U$14" library="blade" deviceset="28FLAG" device=""/>
-<part name="U$3" library="blade" deviceset="28FLAG" device=""/>
 <part name="R2" library="adafruit_changed" deviceset="R-US_" device="0411/15"/>
 <part name="GND3" library="supply1" library_urn="urn:adsk.eagle:library:371" deviceset="GND" device=""/>
+<part name="GND5" library="supply1" library_urn="urn:adsk.eagle:library:371" deviceset="GND" device=""/>
 </parts>
 <sheets>
@@
 <attribute name="VALUE" x="30.48" y="96.52" size="1.778" layer="96" rot="MR0"/>
 </instance>
-<instance part="U$14" gate="G$1" x="53.34" y="-38.1" smashed="yes"/>
-<instance part="U$3" gate="G$1" x="53.34" y="-43.18" smashed="yes"/>
 <instance part="R2" gate="G$1" x="20.32" y="2.54" smashed="yes">
 <attribute name="NAME" x="16.51" y="4.0386" size="1.778" layer="95"/>
@@
 <instance part="GND3" gate="1" x="35.56" y="0" smashed="yes" rot="MR0">
 <attribute name="VALUE" x="38.1" y="-2.54" size="1.778" layer="96" rot="MR0"/>
+</instance>
+<instance part="GND5" gate="1" x="0" y="12.7" smashed="yes" rot="MR0">
+<attribute name="VALUE" x="2.54" y="10.16" size="1.778" layer="96" rot="MR0"/>
 </instance>
 </instances>
@@
 <segment>
 <pinref part="GND4" gate="1" pin="GND"/>
-<pinref part="U$2" gate="G$1" pin="P$4"/>
+<pinref part="U$2" gate="G$1" pin="GND2"/>
 <wire x1="15.24" y1="-27.94" x2="48.26" y2="-27.94" width="0.1524" layer="91"/>
 <wire x1="48.26" y1="-27.94" x2="55.88" y2="-27.94" width="0.1524" layer="91"/>
-<pinref part="U$2" gate="G$1" pin="P$2"/>
+<pinref part="U$2" gate="G$1" pin="GND1"/>
 <wire x1="15.24" y1="-17.78" x2="48.26" y2="-17.78" width="0.1524" layer="91"/>
 <wire x1="48.26" y1="-17.78" x2="48.26" y2="-27.94" width="0.1524" layer="91"/>
@@
 <wire x1="5.08" y1="-27.94" x2="5.08" y2="-33.02" width="0.1524" layer="91"/>
 <junction x="15.24" y="-27.94"/>
-<pinref part="U$2" gate="G$1" pin="P$5"/>
+<pinref part="U$2" gate="G$1" pin="EARTH"/>
 <wire x1="5.08" y1="-33.02" x2="15.24" y2="-33.02" width="0.1524" layer="91"/>
 </segment>
@@
 <wire x1="35.56" y1="2.54" x2="25.4" y2="2.54" width="0.1524" layer="91"/>
 </segment>
+<segment>
+<pinref part="U$1" gate="G$1" pin="P$2"/>
+<pinref part="GND5" gate="1" pin="GND"/>
+<wire x1="7.62" y1="15.24" x2="0" y2="15.24" width="0.1524" layer="91"/>
+<pinref part="U$1" gate="G$1" pin="P$1"/>
+<wire x1="7.62" y1="20.32" x2="0" y2="20.32" width="0.1524" layer="91"/>
+<wire x1="0" y1="20.32" x2="0" y2="15.24" width="0.1524" layer="91"/>
+<junction x="0" y="15.24"/>
+</segment>
 </net>
 <net name="+12V" class="0">
 <segment>
-<pinref part="U$2" gate="G$1" pin="P$3"/>
+<pinref part="U$2" gate="G$1" pin="+12V"/>
 <pinref part="P+3" gate="1" pin="+12V"/>
 <wire x1="15.24" y1="-22.86" x2="-5.08" y2="-22.86" width="0.1524" layer="91"/>
@@
 </segment>
 </net>
-<net name="NEUTRAL" class="0">
-<segment>
-<wire x1="2.54" y1="-38.1" x2="15.24" y2="-38.1" width="0.1524" layer="91"/>
-<label x="2.54" y="-38.1" size="1.778" layer="95" rot="MR0" xref="yes"/>
-<pinref part="U$2" gate="G$1" pin="P$6"/>
-<pinref part="U$14" gate="G$1" pin="P$1"/>
-<wire x1="15.24" y1="-38.1" x2="43.18" y2="-38.1" width="0.1524" layer="91"/>
-<junction x="15.24" y="-38.1"/>
-</segment>
-</net>
-<net name="LIVE" class="0">
-<segment>
-<label x="2.54" y="-43.18" size="1.778" layer="95" rot="MR0" xref="yes"/>
-<pinref part="U$2" gate="G$1" pin="P$7"/>
-<wire x1="15.24" y1="-43.18" x2="2.54" y2="-43.18" width="0.1524" layer="91"/>
-<pinref part="U$3" gate="G$1" pin="P$1"/>
-<wire x1="43.18" y1="-43.18" x2="15.24" y2="-43.18" width="0.1524" layer="91"/>
-<junction x="15.24" y="-43.18"/>
-</segment>
-</net>
 <net name="N$2" class="0">
 <segment>
@@
 <pinref part="U$9" gate="G$1" pin="B0"/>
 <wire x1="7.874" y1="-11.43" x2="7.874" y2="-8.89" width="0.1524" layer="91"/>
-<pinref part="U$2" gate="G$1" pin="P$1"/>
+<pinref part="U$2" gate="G$1" pin="+5V"/>
 <wire x1="15.24" y1="-12.7" x2="15.24" y2="-8.89" width="0.1524" layer="91"/>
 <wire x1="15.24" y1="-8.89" x2="7.874" y2="-8.89" width="0.1524" layer="91"/>

Commit message: updated osborne 1 pcb
Parts:
- added U$3: TERM_RD50_MAINS, os1:TERM_RD50_MAINS
- added U$7: CAR_FUSE_HOLDER3IN1, atx_power_control:CAR_FUSE_HOLDER3IN1
- U$2: value TERM_RD50 -> 396_2P_LIVE; device os1:TERM_RD50 -> 396_conn:396_2P_LIVE
Connections:
- new net N$1: U$3.+12V, U$7.B0, U$7.B1
- new net N$3: U$2.P$2, U$3.NEUTRAL
- new net N$4: U$2.P$1, U$3.LIVE
- net +12V: now also U$7.A0, U$7.A1; no longer U$2.+12V
- net GND: now also U$3.EARTH, U$3.GND1, U$3.GND2; no longer U$2.EARTH, U$2.GND1, U$2.GND2
- net N$2: now also U$3.+5V; no longer U$2.+5V
Changed lines of the file:
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@@
 <parts>
 <part name="U$1" library="os1" deviceset="MEANWELL_RD50" device=""/>
-<part name="U$2" library="os1" deviceset="TERM_RD50" device=""/>
 <part name="JP2" library="pinhead" library_urn="urn:adsk.eagle:library:325" deviceset="PINHD-1X4" device="/90" package3d_urn="urn:adsk.eagle:package:22404/2"/>
 <part name="JP1" library="pinhead" library_urn="urn:adsk.eagle:library:325" deviceset="PINHD-1X4" device="/90" package3d_urn="urn:adsk.eagle:package:22404/2"/>
@@
 <part name="GND3" library="supply1" library_urn="urn:adsk.eagle:library:371" deviceset="GND" device=""/>
 <part name="GND5" library="supply1" library_urn="urn:adsk.eagle:library:371" deviceset="GND" device=""/>
+<part name="U$3" library="os1" deviceset="TERM_RD50_MAINS" device=""/>
+<part name="U$2" library="396_conn" deviceset="396_2P_LIVE" device=""/>
+<part name="U$7" library="atx_power_control" deviceset="CAR_FUSE_HOLDER" device="3IN1"/>
 </parts>
 <sheets>
@@
 <instances>
 <instance part="U$1" gate="G$1" x="45.72" y="38.1" smashed="yes"/>
-<instance part="U$2" gate="G$1" x="30.48" y="-25.4" smashed="yes"/>
 <instance part="JP2" gate="A" x="180.34" y="-17.78" smashed="yes">
 <attribute name="NAME" x="173.99" y="-9.525" size="1.778" layer="95"/>
@@
 <attribute name="VALUE" x="-60.96" y="-7.62" size="1.778" layer="96" rot="MR0"/>
 </instance>
-<instance part="P+3" gate="1" x="-7.62" y="-22.86" smashed="yes" rot="MR270">
-<attribute name="VALUE" x="-10.16" y="-22.86" size="1.778" layer="96" rot="MR0"/>
+<instance part="P+3" gate="1" x="-40.64" y="-40.64" smashed="yes" rot="MR270">
+<attribute name="VALUE" x="-43.18" y="-40.64" size="1.778" layer="96" rot="MR0"/>
 </instance>
 <instance part="GND4" gate="1" x="55.88" y="-30.48" smashed="yes" rot="MR0">
@@
 <attribute name="VALUE" x="2.54" y="10.16" size="1.778" layer="96" rot="MR0"/>
 </instance>
+<instance part="U$3" gate="G$1" x="30.48" y="-25.4" smashed="yes"/>
+<instance part="U$2" gate="G$1" x="0" y="-40.64" smashed="yes" rot="R180"/>
+<instance part="U$7" gate="G$1" x="-7.62" y="-22.86" smashed="yes"/>
 </instances>
 <busses>
@@
 <segment>
 <pinref part="GND4" gate="1" pin="GND"/>
-<pinref part="U$2" gate="G$1" pin="GND2"/>
+<wire x1="5.08" y1="-27.94" x2="15.24" y2="-27.94" width="0.1524" layer="91"/>
 <wire x1="15.24" y1="-27.94" x2="48.26" y2="-27.94" width="0.1524" layer="91"/>
 <wire x1="48.26" y1="-27.94" x2="55.88" y2="-27.94" width="0.1524" layer="91"/>
-<pinref part="U$2" gate="G$1" pin="GND1"/>
 <wire x1="15.24" y1="-17.78" x2="48.26" y2="-17.78" width="0.1524" layer="91"/>
 <wire x1="48.26" y1="-17.78" x2="48.26" y2="-27.94" width="0.1524" layer="91"/>
 <junction x="48.26" y="-27.94"/>
-<wire x1="15.24" y1="-27.94" x2="5.08" y2="-27.94" width="0.1524" layer="91"/>
 <wire x1="5.08" y1="-27.94" x2="5.08" y2="-33.02" width="0.1524" layer="91"/>
+<wire x1="5.08" y1="-33.02" x2="15.24" y2="-33.02" width="0.1524" layer="91"/>
+<pinref part="U$3" gate="G$1" pin="GND1"/>
+<pinref part="U$3" gate="G$1" pin="GND2"/>
 <junction x="15.24" y="-27.94"/>
-<pinref part="U$2" gate="G$1" pin="EARTH"/>
-<wire x1="5.08" y1="-33.02" x2="15.24" y2="-33.02" width="0.1524" layer="91"/>
+<pinref part="U$3" gate="G$1" pin="EARTH"/>
 </segment>
 <segment>
@@
 <net name="+12V" class="0">
 <segment>
-<pinref part="U$2" gate="G$1" pin="+12V"/>
-<pinref part="P+3" gate="1" pin="+12V"/>
-<wire x1="15.24" y1="-22.86" x2="-5.08" y2="-22.86" width="0.1524" layer="91"/>
-</segment>
-<segment>
 <pinref part="JP2" gate="A" pin="2"/>
 <pinref part="JP1" gate="A" pin="2"/>
@@
 <wire x1="172.72" y1="22.86" x2="200.66" y2="22.86" width="0.1524" layer="91"/>
 </segment>
+<segment>
+<pinref part="U$7" gate="G$1" pin="A1"/>
+<pinref part="U$7" gate="G$1" pin="A0"/>
+<wire x1="-22.606" y1="-24.13" x2="-22.606" y2="-21.59" width="0.1524" layer="91"/>
+<pinref part="P+3" gate="1" pin="+12V"/>
+<wire x1="-22.606" y1="-24.13" x2="-22.606" y2="-40.64" width="0.1524" layer="91"/>
+<wire x1="-22.606" y1="-40.64" x2="-38.1" y2="-40.64" width="0.1524" layer="91"/>
+<junction x="-22.606" y="-24.13"/>
+</segment>
 </net>
 <net name="N$2" class="0">
@@
 <pinref part="U$9" gate="G$1" pin="B0"/>
 <wire x1="7.874" y1="-11.43" x2="7.874" y2="-8.89" width="0.1524" layer="91"/>
-<pinref part="U$2" gate="G$1" pin="+5V"/>
 <wire x1="15.24" y1="-12.7" x2="15.24" y2="-8.89" width="0.1524" layer="91"/>
 <wire x1="15.24" y1="-8.89" x2="7.874" y2="-8.89" width="0.1524" layer="91"/>
 <junction x="7.874" y="-8.89"/>
 <pinref part="R2" gate="G$1" pin="1"/>
-<wire x1="15.24" y1="2.54" x2="15.24" y2="-12.7" width="0.1524" layer="91"/>
-<junction x="15.24" y="-12.7"/>
+<wire x1="15.24" y1="2.54" x2="15.24" y2="-8.89" width="0.1524" layer="91"/>
+<pinref part="U$3" gate="G$1" pin="+5V"/>
 </segment>
 </net>
@@
 </segment>
 </net>
+<net name="N$1" class="0">
+<segment>
+<pinref part="U$3" gate="G$1" pin="+12V"/>
+<pinref part="U$7" gate="G$1" pin="B0"/>
+<wire x1="15.24" y1="-22.86" x2="7.874" y2="-22.86" width="0.1524" layer="91"/>
+<wire x1="7.874" y1="-22.86" x2="7.874" y2="-21.59" width="0.1524" layer="91"/>
+<pinref part="U$7" gate="G$1" pin="B1"/>
+<wire x1="7.874" y1="-24.13" x2="7.874" y2="-21.59" width="0.1524" layer="91"/>
+<junction x="7.874" y="-21.59"/>
+</segment>
+</net>
+<net name="N$3" class="0">
+<segment>
+<pinref part="U$3" gate="G$1" pin="NEUTRAL"/>
+<pinref part="U$2" gate="G$1" pin="P$2"/>
+<wire x1="15.24" y1="-38.1" x2="5.08" y2="-38.1" width="0.1524" layer="91"/>
+</segment>
+</net>
+<net name="N$4" class="0">
+<segment>
+<pinref part="U$2" gate="G$1" pin="P$1"/>
+<wire x1="5.08" y1="-40.64" x2="5.08" y2="-43.18" width="0.1524" layer="91"/>
+<pinref part="U$3" gate="G$1" pin="LIVE"/>
+<wire x1="5.08" y1="-43.18" x2="15.24" y2="-43.18" width="0.1524" layer="91"/>
+</segment>
+</net>
